File: KiCAD_PCB/Calculator_PCB/Calculator_PCB.kicad_sch (KiCad schematic)
At the start: 106 parts, among them J1 USB_B_Micro, SW1 +, SW10 E, SW11 D, SW12 C, SW13 *, SW14 R, SW15 F, SW16 V, SW17 =, SW18 T, SW19 G, SW2 Q, SW20 B, SW21 SQRT, SW22 Y, SW23 H, SW24 N, SW25 e^x (ln), SW26 U, SW27 J, SW28 M, SW29 10^x (log), SW3 A, SW30 I, SW31 K, SW32 [ ] ({ }), SW33 Symbol's, SW34 O, SW35 L, SW36 ; (:), SW37 Menu, SW38 P, SW39 Trig, SW4 Z, SW40 Greek, SW5 -, SW6 W, SW7 S, SW8 X, SW9 /, U1 W25Q128JVS, U2 RP2040, U3 NCP1117-3.3_SOT223, Y1 ABLS-12.000MHZ-B4-T

Commit message: PCB Updates
Parts:
- added S?: (no value), symbol PTS810SJK250SMTRLFS:PTS810SJK250SMTRLFS
Connections:
- net GND: now also S?.2, S?.4
- net USB_BOOT: now also S?.1, S?.3
Other:
- note added: "BOOTSEL"
Changed lines of the file:
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@@
   (junction (at 97.536 158.496) (diameter 0) (color 0 0 0 0)
   )
+  (junction (at 96.52 84.074) (diameter 0) (color 0 0 0 0)
+  )
   (junction (at 109.22 158.496) (diameter 0) (color 0 0 0 0)
   )
@@
   (junction (at 119.126 193.548) (diameter 0) (color 0 0 0 0)
   )
+  (junction (at 96.52 67.564) (diameter 0) (color 0 0 0 0)
+  )
   (junction (at 37.338 175.26) (diameter 0) (color 0 0 0 0)
   )
@@
     (stroke (width 0) (type default) (color 0 0 0 0))
   )
+  (wire (pts (xy 95.504 67.564) (xy 96.52 67.564))
+    (stroke (width 0) (type default) (color 0 0 0 0))
+  )
+  (wire (pts (xy 96.52 77.216) (xy 99.06 77.216))
+    (stroke (width 0) (type default) (color 0 0 0 0))
+  )
   (wire (pts (xy 63.5 37.338) (xy 63.5 41.656))
     (stroke (width 0) (type default) (color 0 0 0 0))
@@
     (stroke (width 0) (type default) (color 0 0 0 0))
   )
+  (wire (pts (xy 96.52 67.564) (xy 96.52 77.216))
+    (stroke (width 0) (type default) (color 0 0 0 0))
+  )
   (polyline (pts (xy 84.074 59.436) (xy 84.074 115.824))
     (stroke (width 0) (type default) (color 0 0 0 0))
@@
     (stroke (width 0) (type default) (color 0 0 0 0))
   )
+  (wire (pts (xy 121.92 77.216) (xy 121.92 67.564))
+    (stroke (width 0) (type default) (color 0 0 0 0))
+  )
   (wire (pts (xy 54.102 37.338) (xy 50.8 37.338))
     (stroke (width 0) (type default) (color 0 0 0 0))
@@
     (stroke (width 0) (type default) (color 0 0 0 0))
   )
+  (wire (pts (xy 121.92 79.756) (xy 121.92 84.074))
+    (stroke (width 0) (type default) (color 0 0 0 0))
+  )
   (wire (pts (xy 95.758 140.716) (xy 95.758 140.208))
     (stroke (width 0) (type default) (color 0 0 0 0))
@@
     (stroke (width 0) (type default) (color 0 0 0 0))
   )
+  (wire (pts (xy 119.38 77.216) (xy 121.92 77.216))
+    (stroke (width 0) (type default) (color 0 0 0 0))
+  )
   (wire (pts (xy 95.758 193.548) (xy 107.442 193.548))
     (stroke (width 0) (type default) (color 0 0 0 0))
@@
     (stroke (width 0) (type default) (color 0 0 0 0))
   )
+  (wire (pts (xy 119.38 79.756) (xy 121.92 79.756))
+    (stroke (width 0) (type default) (color 0 0 0 0))
+  )
   (wire (pts (xy 130.81 120.142) (xy 132.588 120.142))
     (stroke (width 0) (type default) (color 0 0 0 0))
@@
     (stroke (width 0) (type default) (color 0 0 0 0))
   )
+  (wire (pts (xy 121.92 84.074) (xy 96.52 84.074))
+    (stroke (width 0) (type default) (color 0 0 0 0))
+  )
   (wire (pts (xy 49.022 120.142) (xy 50.8 120.142))
     (stroke (width 0) (type default) (color 0 0 0 0))
@@
     (stroke (width 0) (type default) (color 0 0 0 0))
   )
+  (wire (pts (xy 96.52 84.074) (xy 96.52 86.614))
+    (stroke (width 0) (type default) (color 0 0 0 0))
+  )
   (wire (pts (xy 119.126 138.176) (xy 119.126 139.192))
     (stroke (width 0) (type default) (color 0 0 0 0))
@@
     (stroke (width 0) (type default) (color 0 0 0 0))
   )
+  (wire (pts (xy 121.92 67.564) (xy 96.52 67.564))
+    (stroke (width 0) (type default) (color 0 0 0 0))
+  )
   (wire (pts (xy 85.852 120.142) (xy 85.852 140.208))
     (stroke (width 0) (type default) (color 0 0 0 0))
@@
     (stroke (width 0) (type default) (color 0 0 0 0))
   )
+  (wire (pts (xy 96.52 79.756) (xy 96.52 84.074))
+    (stroke (width 0) (type default) (color 0 0 0 0))
+  )
   (wire (pts (xy 50.8 37.338) (xy 50.8 41.656))
     (stroke (width 0) (type default) (color 0 0 0 0))
@@
     (stroke (width 0) (type default) (color 0 0 0 0))
   )
+  (wire (pts (xy 96.52 79.756) (xy 99.06 79.756))
+    (stroke (width 0) (type default) (color 0 0 0 0))
+  )
   (wire (pts (xy 62.484 120.142) (xy 62.484 140.208))
     (stroke (width 0) (type default) (color 0 0 0 0))
@@
     (effects (font (size 0.8 0.8)) (justify left bottom))
   )
+  (text "BOOTSEL" (at 103.886 67.056 0)
+    (effects (font (size 1.6 1.6)) (justify left bottom))
+  )
   (text "Decoupling Capacitors\n" (at 13.462 15.494 0)
     (effects (font (size 1.6 1.6)) (justify left bottom))
@@
     (effects (font (size 1.27 1.27)) (justify left bottom))
   )
+  (label "USB_BOOT" (at 95.504 67.564 180)
+    (effects (font (size 1.27 1.27)) (justify right bottom))
+  )
   (label "VREG_IOVDD_44" (at 251.714 113.538 0)
     (effects (font (size 1.27 1.27)) (justify left bottom))
@@
     (pin "2")
   )
+  (symbol (lib_id "power:GND") (at 96.52 86.614 0) (unit 1)
+    (in_bom yes) (on_board yes) (fields_autoplaced)
+    (property "Reference" "#PWR?" (id 0) (at 96.52 92.964 0)
+      (effects (font (size 1.27 1.27)) hide)
+    )
+    (property "Value" "GND" (id 1) (at 96.52 91.44 0))
+    (property "Footprint" "" (id 2) (at 96.52 86.614 0)
+      (effects (font (size 1.27 1.27)) hide)
+    )
+    (property "Datasheet" "" (id 3) (at 96.52 86.614 0)
+      (effects (font (size 1.27 1.27)) hide)
+    )
+    (pin "1")
+  )
   (symbol (lib_id "Device:R_Small") (at 273.304 108.458 90) (unit 1)
     (in_bom yes) (on_board yes)
@@
     (pin "1")
   )
+  (symbol (lib_id "PTS810SJK250SMTRLFS:PTS810SJK250SMTRLFS") (at 99.06 77.216 0) (unit 1)
+    (in_bom yes) (on_board yes) (fields_autoplaced)
+    (property "Reference" "S?" (id 0) (at 109.22 69.85 0))
+    (property "Value" "" (id 1) (at 109.22 72.39 0))
+    (property "Footprint" "" (id 2) (at 99.06 77.216 0)
+      (effects (font (size 1.27 1.27)) (justify left bottom) hide)
+    )
+    (property "Datasheet" "" (id 3) (at 99.06 77.216 0)
+      (effects (font (size 1.27 1.27)) (justify left bottom) hide)
+    )
+    (property "RS_PART_NUMBER" "1359396P" (id 4) (at 99.06 77.216 0)
+      (effects (font (size 1.27 1.27)) (justify left bottom) hide)
+    )
+    (property "MANUFACTURER_PART_NUMBER" "PTS810SJK250SMTRLFS" (id 5) (at 99.06 77.216 0)
+      (effects (font (size 1.27 1.27)) (justify left bottom) hide)
+    )
+    (property "MANUFACTURER_NAME" "C & K COMPONENTS" (id 6) (at 99.06 77.216 0)
+      (effects (font (size 1.27 1.27)) (justify left bottom) hide)
+    )
+    (property "HEIGHT" "mm" (id 7) (at 99.06 77.216 0)
+      (effects (font (size 1.27 1.27)) (justify left bottom) hide)
+    )
+    (property "RS_PRICE-STOCK" "http://uk.rs-online.com/web/p/products/1359396P" (id 8) (at 99.06 77.216 0)
+      (effects (font (size 1.27 1.27)) (justify left bottom) hide)
+    )
+    (property "DESCRIPTION" "IP40 Black Button Tactile Switch, SPST-NO 50 mA 3mm Surface Mount" (id 9) (at 99.06 77.216 0)
+      (effects (font (size 1.27 1.27)) (justify left bottom) hide)
+    )
+    (pin "1")
+    (pin "2")
+    (pin "3")
+    (pin "4")
+  )
   (symbol (lib_id "power:GND") (at 179.324 126.238 0) (unit 1)
     (in_bom yes) (on_board yes) (fields_autoplaced)
@@
       (reference "#PWR0118") (unit 1) (value "VBUS") (footprint "")
     )
+    (path "/62895c27-7821-4b9d-b25d-a97a9add18bb"
+      (reference "#PWR?") (unit 1) (value "GND") (footprint "")
+    )
     (path "/243b70e3-a52d-4de2-a3f1-1a84e3d2c44f"
       (reference "C1") (unit 1) (value "100n") (footprint "")
@@
       (reference "R?") (unit 1) (value "10k") (footprint "")
     )
+    (path "/76a4f48d-78a7-4f5a-a517-e4630a35d809"
+      (reference "S?") (unit 1) (value "PTS810SJK250SMTRLFS") (footprint "PTS810SJG250SMTRLFS")
+    )
     (path "/ea86cc11-be9d-452d-87f6-5ce1008e2886"

Commit message: PCB Updates
Parts:
- added R?: (no value), symbol Device:R_Small
- R?: value (none) -> 10k
- S?: value (none) -> PTS810SJK250SMTRLFS; footprint (none) -> PTS810SJG250SMTRLFS
Connections:
- net +1V1: no longer U2.23 (DVDD)
- net +3V3: now also R?.1
- net RUN_26: now reaches U2.26 (RUN)
- net RUN_26: now also R?.2
- net QSPI_SCLK renamed QSPI_SCLK_52
- net QSPI_SD0 renamed QSPI_SD0_53
- net QSPI_SD1 renamed QSPI_SD1_55
- net QSPI_SD2 renamed QSPI_SD2_54
- net QSPI_SD3 renamed QSPI_SD3_51
- net QSPI_SS renamed QSPI_SS_56
Other:
- note added: "Note: If run is not used, tie high Tie into switch if wanting to utilize reset to upload UF2"
- moved on the sheet: R1, U2

Commit message: PCB Updates
Connections:
- net XIN is gone; now on net XIN_20: C15.2, Y1.2
- net QSPI_SCLK_52: now also U2.52 (QSPI_SCLK)
- net QSPI_SD0_53: now also U2.53 (QSPI_SD0)
- net QSPI_SD1_55: now also U2.55 (QSPI_SD1)
- net QSPI_SD2_54: now also U2.54 (QSPI_SD2)
- net QSPI_SD3_51: now also U2.51 (QSPI_SD3)
- net QSPI_SS_56: now also U2.56 (QSPI_SS_N)
- net XIN_20: now reaches U2.20 (XIN)
- net XOUT renamed XOUT_21
Changed lines of the file:
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@@
+    (stroke (width 0) (type default) (color 0 0 0 0))
+  )
+  (wire (pts (xy 190.5 128.778) (xy 191.516 128.778))
     (stroke (width 0) (type default) (color 0 0 0 0))
   )
@@
     (stroke (width 0) (type default) (color 0 0 0 0))
   )
-  (wire (pts (xy 181.102 126.238) (xy 191.516 126.238))
+  (wire (pts (xy 179.578 126.238) (xy 191.516 126.238))
     (stroke (width 0) (type default) (color 0 0 0 0))
   )
@@
     (stroke (width 0) (type default) (color 0 0 0 0))
   )
+  (wire (pts (xy 252.476 85.598) (xy 253.492 85.598))
+    (stroke (width 0) (type default) (color 0 0 0 0))
+  )
   (wire (pts (xy 60.706 140.208) (xy 62.484 140.208))
     (stroke (width 0) (type default) (color 0 0 0 0))
@@
     (stroke (width 0) (type default) (color 0 0 0 0))
   )
+  (wire (pts (xy 252.476 95.758) (xy 253.492 95.758))
+    (stroke (width 0) (type default) (color 0 0 0 0))
+  )
   (wire (pts (xy 173.99 30.48) (xy 181.61 30.48))
     (stroke (width 0) (type default) (color 0 0 0 0))
@@
     (stroke (width 0) (type default) (color 0 0 0 0))
   )
-  (wire (pts (xy 252.476 80.518) (xy 262.89 80.518))
+  (wire (pts (xy 252.476 80.518) (xy 268.224 80.518))
     (stroke (width 0) (type default) (color 0 0 0 0))
   )
@@
     (stroke (width 0) (type default) (color 0 0 0 0))
   )
+  (wire (pts (xy 252.476 90.678) (xy 253.492 90.678))
+    (stroke (width 0) (type default) (color 0 0 0 0))
+  )
   (wire (pts (xy 39.116 140.208) (xy 39.116 158.496))
     (stroke (width 0) (type default) (color 0 0 0 0))
@@
     (stroke (width 0) (type default) (color 0 0 0 0))
   )
+  (wire (pts (xy 252.476 83.058) (xy 253.492 83.058))
+    (stroke (width 0) (type default) (color 0 0 0 0))
+  )
   (wire (pts (xy 72.39 140.208) (xy 74.168 140.208))
     (stroke (width 0) (type default) (color 0 0 0 0))
@@
     (stroke (width 0) (type default) (color 0 0 0 0))
   )
+  (wire (pts (xy 252.476 93.218) (xy 253.492 93.218))
+    (stroke (width 0) (type default) (color 0 0 0 0))
+  )
   (wire (pts (xy 50.8 37.338) (xy 47.752 37.338))
     (stroke (width 0) (type default) (color 0 0 0 0))
@@
   )
   (wire (pts (xy 34.798 156.972) (xy 37.338 156.972))
+    (stroke (width 0) (type default) (color 0 0 0 0))
+  )
+  (wire (pts (xy 252.476 88.138) (xy 253.492 88.138))
     (stroke (width 0) (type default) (color 0 0 0 0))
   )
@@
     (effects (font (size 1.6 1.6)) (justify left bottom))
   )
-  (text "Note:\nUSB Resistors need to be placed near RP2040\n"
-    (at 254.762 95.504 0)
+  (text "Note:\nUSB Resistors need \nto be placed near \nRP2040\n"
+    (at 272.034 102.616 0)
     (effects (font (size 0.8 0.8)) (justify left bottom))
   )
@@
     (effects (font (size 1.27 1.27)) (justify right bottom))
   )
+  (label "QSPI_SS_56" (at 253.492 83.058 0)
+    (effects (font (size 1.27 1.27)) (justify left bottom))
+  )
   (label "Col3" (at 34.798 193.548 180)
     (effects (font (size 1.27 1.27)) (justify right bottom))
@@
     (effects (font (size 1.27 1.27)) (justify left bottom))
   )
+  (label "QSPI_SCLK_52" (at 253.492 93.218 0)
+    (effects (font (size 1.27 1.27)) (justify left bottom))
+  )
   (label "USB_BOOT" (at 95.504 67.564 180)
     (effects (font (size 1.27 1.27)) (justify right bottom))
@@
     (effects (font (size 1.27 1.27)) (justify left bottom))
   )
-  (label "XIN" (at 272.542 29.972 0)
+  (label "XIN_20" (at 272.542 29.972 0)
     (effects (font (size 1.27 1.27)) (justify left bottom))
   )
@@
     (effects (font (size 1.27 1.27)) (justify right bottom))
   )
+  (label "XOUT_21" (at 190.5 131.318 180)
+    (effects (font (size 1.27 1.27)) (justify right bottom))
+  )
+  (label "XIN_20" (at 190.5 128.778 180)
+    (effects (font (size 1.27 1.27)) (justify right bottom))
+  )
   (label "DVDD_50" (at 253.492 98.298 0)
     (effects (font (size 1.27 1.27)) (justify left bottom))
   )
+  (label "QSPI_SD1_55" (at 253.492 85.598 0)
+    (effects (font (size 1.27 1.27)) (justify left bottom))
+  )
   (label "Row1" (at 49.022 120.142 180)
     (effects (font (size 1.27 1.27)) (justify right bottom))
@@
     (effects (font (size 1.27 1.27)) (justify right bottom))
   )
+  (label "QSPI_SD0_53" (at 253.492 90.678 0)
+    (effects (font (size 1.27 1.27)) (justify left bottom))
+  )
+  (label "QSPI_SD3_51" (at 253.492 95.758 0)
+    (effects (font (size 1.27 1.27)) (justify left bottom))
+  )
   (label "DVDD_23" (at 190.5 136.398 180)
     (effects (font (size 1.27 1.27)) (justify right bottom))
   )
+  (label "QSPI_SD2_54" (at 253.492 88.138 0)
+    (effects (font (size 1.27 1.27)) (justify left bottom))
+  )
   (label "IOVDD_1" (at 66.802 41.656 270)
     (effects (font (size 1.27 1.27)) (justify right bottom))
@@
     (effects (font (size 1.27 1.27)) (justify right bottom))
   )
-  (label "XOUT" (at 272.542 37.084 0)
+  (label "XOUT_21" (at 272.542 37.084 0)
     (effects (font (size 1.27 1.27)) (justify left bottom))
   )
@@
     (pin "2")
   )
-  (symbol (lib_id "power:GND") (at 262.89 80.518 0) (unit 1)
-    (in_bom yes) (on_board yes) (fields_autoplaced)
-    (property "Reference" "#PWR0108" (id 0) (at 262.89 86.868 0)
-      (effects (font (size 1.27 1.27)) hide)
-    )
-    (property "Value" "GND" (id 1) (at 262.89 85.598 0))
-    (property "Footprint" "" (id 2) (at 262.89 80.518 0)
-      (effects (font (size 1.27 1.27)) hide)
-    )
-    (property "Datasheet" "" (id 3) (at 262.89 80.518 0)
+  (symbol (lib_id "power:GND") (at 268.224 80.518 0) (unit 1)
+    (in_bom yes) (on_board yes) (fields_autoplaced)
+    (property "Reference" "#PWR0108" (id 0) (at 268.224 86.868 0)
+      (effects (font (size 1.27 1.27)) hide)
+    )
+    (property "Value" "GND" (id 1) (at 268.224 85.598 0))
+    (property "Footprint" "" (id 2) (at 268.224 80.518 0)
+      (effects (font (size 1.27 1.27)) hide)
+    )
+    (property "Datasheet" "" (id 3) (at 268.224 80.518 0)
       (effects (font (size 1.27 1.27)) hide)
     )
@@
     (pin "4")
   )
-  (symbol (lib_id "power:GND") (at 181.102 126.238 0) (unit 1)
-    (in_bom yes) (on_board yes) (fields_autoplaced)
-    (property "Reference" "#PWR0111" (id 0) (at 181.102 132.588 0)
-      (effects (font (size 1.27 1.27)) hide)
-    )
-    (property "Value" "GND" (id 1) (at 181.102 131.064 0))
-    (property "Footprint" "" (id 2) (at 181.102 126.238 0)
-      (effects (font (size 1.27 1.27)) hide)
-    )
-    (property "Datasheet" "" (id 3) (at 181.102 126.238 0)
-      (effects (font (size 1.27 1.27)) hide)
-    )
+  (symbol (lib_id "power:GND") (at 179.578 126.238 0) (unit 1)
+    (in_bom yes) (on_board yes) (fields_autoplaced)
+    (property "Reference" "#PWR0111" (id 0) (at 179.578 132.588 0)
+      (effects (font (size 1.27 1.27)) hide)
+    )
+    (property "Value" "GND" (id 1) (at 179.578 131.064 0))
+    (property "Footprint" "" (id 2) (at 179.578 126.238 0)
+      (effects (font (size 1.27 1.27)) hide)
+    )
+    (property "Datasheet" "" (id 3) (at 179.578 126.238 0)
+      (effects (font (size 1.27 1.27)) hide)
+    )

Commit message: PCB Updates
Parts:
- C1, C10, C11, C12, C13, C14, C15, C16, C2, C3, C4, C5, C6, C7, C8, C9: footprint (none) -> Capacitor_SMD:C_01005_0402Metric_Pad0.57x0.30mm_HandSolder
- D1, D10, D11, D12, D13, D14, D15, D16, D17, D18, D19, D2, D20, D21, D22, D23, D24, D25, D26, D27, D28, D29, D3, D30, D31, D32, D33, D34, D35, D36, D37, D38, D39, D4, D40, D5, D6, D7, D8, D9: footprint (none) -> Diode_SMD:D_0402_1005Metric_Pad0.77x0.64mm_HandSolder
- R6: renamed from R?; value (none) -> 10k
- S1: renamed from S?; footprint PTS810SJG250SMTRLFS -> (none)
- U2: footprint IC57_RP2040 -> (none)
- gave numbers to parts that had none: 1
Other:
- note added: "Buttons"
- moved on the sheet: D1, D10, D11, D12, D13, D14, D15, D16, D17, D18, D19, D2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
