File: KiCAD_PCB/Calculator_PCB/Calculator_PCB.kicad_sch (KiCad schematic)
At the start: 109 parts, among them J1 USB_B_Micro, SW1 SW_SPST, SW10 SW_SPST, SW11 SW_SPST, SW12 SW_SPST, SW13 SW_SPST, SW14 SW_SPST, SW15 SW_SPST, SW16 SW_SPST, SW17 SW_SPST, SW18 SW_SPST, SW19 SW_SPST, SW2 SW_SPST, SW20 SW_SPST, SW21 SW_SPST, SW22 SW_SPST, SW23 SW_SPST, SW24 SW_SPST, SW25 SW_SPST, SW26 SW_SPST, SW27 SW_SPST, SW28 SW_SPST, SW29 SW_SPST, SW3 SW_SPST, SW30 SW_SPST, SW31 SW_SPST, SW32 SW_SPST, SW33 SW_SPST, SW34 SW_SPST, SW35 SW_SPST, SW36 SW_SPST, SW37 SW_SPST, SW38 SW_SPST, SW39 SW_SPST, SW4 SW_SPST, SW40 SW_SPST, SW5 SW_SPST, SW6 SW_SPST, SW7 SW_SPST, SW8 SW_SPST, SW9 SW_SPST, U1 W25Q128JVS, U2 RP2040, U3 NCP1117-3.3_SOT223, Y1 ABLS-12.000MHZ-B4-T

Commit message: PCB Updates
Connections:
- net Col0 is gone; now on net Col3: SW1.2 (B), SW2.2 (B), SW3.2 (B), SW4.2 (B)
- net Col1 is gone; now on net Col4: SW5.2 (B), SW6.2 (B), SW7.2 (B), SW8.2 (B)
- net Col2 is gone; now on net Col5: SW10.2 (B), SW11.2 (B), SW12.2 (B), SW9.2 (B)
- net Row0 is gone; now on net Row2: D1.1 (K), D13.1 (K), D17.1 (K), D21.1 (K), D25.1 (K), D29.1 (K), D33.1 (K), D37.1 (K), D5.1 (K), D9.1 (K)
- net Row1 is gone; now on net Row3: D10.1 (K), D14.1 (K), D18.1 (K), D2.1 (K), D22.1 (K), D26.1 (K), D30.1 (K), D34.1 (K), D38.1 (K), D6.1 (K)
- net Col3: no longer SW13.2 (B), SW14.2 (B), SW15.2 (B), SW16.2 (B)
- net Col4: no longer SW17.2 (B), SW18.2 (B), SW19.2 (B), SW20.2 (B)
- net Col5: no longer SW21.2 (B), SW22.2 (B), SW23.2 (B), SW24.2 (B)
- net Col6: now also SW13.2 (B), SW14.2 (B), SW15.2 (B), SW16.2 (B); no longer SW25.2 (B), SW26.2 (B), SW27.2 (B), SW28.2 (B)
- net Col7: now also SW17.2 (B), SW18.2 (B), SW19.2 (B), SW20.2 (B); no longer SW29.2 (B), SW30.2 (B), SW31.2 (B), SW32.2 (B)
- net Col8: now also SW21.2 (B), SW22.2 (B), SW23.2 (B), SW24.2 (B); no longer SW33.2 (B), SW34.2 (B), SW35.2 (B), SW36.2 (B)
- net Col9: now also SW25.2 (B), SW26.2 (B), SW27.2 (B), SW28.2 (B); no longer SW37.2 (B), SW38.2 (B), SW39.2 (B), SW40.2 (B)
- net Row2: no longer D11.1 (K), D15.1 (K), D19.1 (K), D23.1 (K), D27.1 (K), D3.1 (K), D31.1 (K), D35.1 (K), D39.1 (K), D7.1 (K)
- net Row3: no longer D12.1 (K), D16.1 (K), D20.1 (K), D24.1 (K), D28.1 (K), D32.1 (K), D36.1 (K), D4.1 (K), D40.1 (K), D8.1 (K)
- new net Col10: SW29.2 (B), SW30.2 (B), SW31.2 (B), SW32.2 (B)
- new net Col11: SW33.2 (B), SW34.2 (B), SW35.2 (B), SW36.2 (B)
- new net Col12: SW37.2 (B), SW38.2 (B), SW39.2 (B), SW40.2 (B)
- new net Row4: D11.1 (K), D15.1 (K), D19.1 (K), D23.1 (K), D27.1 (K), D3.1 (K), D31.1 (K), D35.1 (K), D39.1 (K), D7.1 (K)
- new net Row5: D12.1 (K), D16.1 (K), D20.1 (K), D24.1 (K), D28.1 (K), D32.1 (K), D36.1 (K), D4.1 (K), D40.1 (K), D8.1 (K)
Changed lines of the file:
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@@
     (effects (font (size 1.27 1.27)) (justify left bottom))
   )
-  (label "Col0" (at 45.466 135.636 180)
+  (label "Col3" (at 45.466 135.636 180)
     (effects (font (size 1.27 1.27)) (justify right bottom))
   )
-  (label "Row2" (at 25.654 171.958 180)
+  (label "Row4" (at 25.654 171.958 180)
     (effects (font (size 1.27 1.27)) (justify right bottom))
   )
@@
     (effects (font (size 1.27 1.27)) (justify left bottom))
   )
-  (label "Col7" (at 184.15 135.636 180)
+  (label "Col10" (at 184.15 135.636 180)
     (effects (font (size 1.27 1.27)) (justify right bottom))
   )
-  (label "Row0" (at 25.654 148.59 180)
+  (label "Row2" (at 25.654 148.59 180)
     (effects (font (size 1.27 1.27)) (justify right bottom))
   )
@@
     (effects (font (size 1.27 1.27)) (justify right bottom))
   )
-  (label "Col1" (at 65.278 135.636 180)
+  (label "Col4" (at 65.278 135.636 180)
     (effects (font (size 1.27 1.27)) (justify right bottom))
   )
@@
     (effects (font (size 1.27 1.27)) (justify left bottom))
   )
-  (label "Col3" (at 104.902 135.636 180)
+  (label "Col6" (at 104.902 135.636 180)
     (effects (font (size 1.27 1.27)) (justify right bottom))
   )
@@
     (effects (font (size 1.27 1.27)) (justify left bottom))
   )
-  (label "Col5" (at 144.526 135.636 180)
+  (label "Col8" (at 144.526 135.636 180)
     (effects (font (size 1.27 1.27)) (justify right bottom))
   )
@@
     (effects (font (size 1.27 1.27)) (justify left bottom))
   )
-  (label "Col4" (at 124.714 135.636 180)
+  (label "Col7" (at 124.714 135.636 180)
     (effects (font (size 1.27 1.27)) (justify right bottom))
   )
@@
     (effects (font (size 1.27 1.27)) (justify right bottom))
   )
-  (label "Col6" (at 164.338 135.636 180)
+  (label "Col9" (at 164.338 135.636 180)
     (effects (font (size 1.27 1.27)) (justify right bottom))
   )
@@
     (effects (font (size 1.27 1.27)) (justify left bottom))
   )
-  (label "Col8" (at 203.962 135.636 180)
+  (label "Col11" (at 203.962 135.636 180)
     (effects (font (size 1.27 1.27)) (justify right bottom))
   )
@@
     (effects (font (size 1.27 1.27)) (justify left bottom))
   )
-  (label "Row1" (at 25.654 160.274 180)
+  (label "Row3" (at 25.654 160.274 180)
     (effects (font (size 1.27 1.27)) (justify right bottom))
   )
@@
     (effects (font (size 1.27 1.27)) (justify right bottom))
   )
-  (label "Col9" (at 223.774 135.636 180)
+  (label "Col12" (at 223.774 135.636 180)
     (effects (font (size 1.27 1.27)) (justify right bottom))
   )
@@
     (effects (font (size 1.27 1.27)) (justify right bottom))
   )
-  (label "Row3" (at 25.654 183.642 180)
+  (label "Row5" (at 25.654 183.642 180)
     (effects (font (size 1.27 1.27)) (justify right bottom))
   )
@@
     (effects (font (size 1.27 1.27)) (justify right bottom))
   )
-  (label "Col2" (at 85.09 135.636 180)
+  (label "Col5" (at 85.09 135.636 180)
     (effects (font (size 1.27 1.27)) (justify right bottom))
   )

Commit message: PCB Updates
Connections:
- net GND: now also X?.7; no longer X?.10
- net y_out: now reaches X?.1
- net x_out: now reaches X?.2
- net Col0: now reaches X?.3
- net Col1: now reaches X?.4
- net Col2: now reaches X?.5
Other:
- moved on the sheet: X?
Changed lines of the file:
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@@
+    (stroke (width 0) (type default) (color 0 0 0 0))
+  )
+  (wire (pts (xy 35.052 81.026) (xy 36.068 81.026))
     (stroke (width 0) (type default) (color 0 0 0 0))
   )
@@
     (stroke (width 0) (type default) (color 0 0 0 0))
   )
+  (wire (pts (xy 35.052 78.486) (xy 36.068 78.486))
+    (stroke (width 0) (type default) (color 0 0 0 0))
+  )
   (wire (pts (xy 67.818 183.642) (xy 87.63 183.642))
     (stroke (width 0) (type default) (color 0 0 0 0))
@@
     (stroke (width 0) (type default) (color 0 0 0 0))
   )
+  (wire (pts (xy 35.052 88.646) (xy 36.068 88.646))
+    (stroke (width 0) (type default) (color 0 0 0 0))
+  )
   (wire (pts (xy 65.278 181.102) (xy 65.278 169.418))
     (stroke (width 0) (type default) (color 0 0 0 0))
   )
+  (wire (pts (xy 35.052 86.106) (xy 36.068 86.106))
+    (stroke (width 0) (type default) (color 0 0 0 0))
+  )
   (wire (pts (xy 93.726 157.734) (xy 94.742 157.734))
     (stroke (width 0) (type default) (color 0 0 0 0))
@@
     (stroke (width 0) (type default) (color 0 0 0 0))
   )
-  (wire (pts (xy 38.862 91.186) (xy 40.894 91.186))
-    (stroke (width 0) (type default) (color 0 0 0 0))
-  )
   (wire (pts (xy 214.63 69.088) (xy 214.63 70.104))
     (stroke (width 0) (type default) (color 0 0 0 0))
@@
     (stroke (width 0) (type default) (color 0 0 0 0))
   )
+  (wire (pts (xy 35.052 83.566) (xy 36.068 83.566))
+    (stroke (width 0) (type default) (color 0 0 0 0))
+  )
   (wire (pts (xy 19.304 23.368) (xy 19.304 24.384))
     (stroke (width 0) (type default) (color 0 0 0 0))
@@
     (stroke (width 0) (type default) (color 0 0 0 0))
   )
-  (wire (pts (xy 38.862 81.026) (xy 40.894 81.026))
+  (wire (pts (xy 51.308 78.486) (xy 53.34 78.486))
     (stroke (width 0) (type default) (color 0 0 0 0))
   )
@@
     (stroke (width 0) (type default) (color 0 0 0 0))
   )
+  (wire (pts (xy 51.308 81.026) (xy 63.246 81.026))
+    (stroke (width 0) (type default) (color 0 0 0 0))
+  )
   (wire (pts (xy 315.468 108.712) (xy 333.756 108.712))
     (stroke (width 0) (type default) (color 0 0 0 0))
@@
     (stroke (width 0) (type default) (color 0 0 0 0))
   )
-  (wire (pts (xy 40.894 91.186) (xy 40.894 93.726))
+  (wire (pts (xy 63.246 81.026) (xy 63.246 83.566))
     (stroke (width 0) (type default) (color 0 0 0 0))
   )
@@
     (stroke (width 0) (type default) (color 0 0 0 0))
   )
-  (wire (pts (xy 40.894 78.486) (xy 40.894 81.026))
+  (wire (pts (xy 53.34 75.946) (xy 53.34 78.486))
     (stroke (width 0) (type default) (color 0 0 0 0))
   )
@@
     (effects (font (size 1.27 1.27)) (justify right bottom))
   )
+  (label "y_out" (at 35.052 78.486 180)
+    (effects (font (size 1.27 1.27)) (justify right bottom))
+  )
   (label "Row4" (at 25.654 171.958 180)
     (effects (font (size 1.27 1.27)) (justify right bottom))
@@
     (effects (font (size 1.27 1.27)) (justify left bottom))
   )
+  (label "Col2" (at 35.052 88.646 180)
+    (effects (font (size 1.27 1.27)) (justify right bottom))
+  )
   (label "USB_BOOT" (at 166.624 91.694 0)
     (effects (font (size 1.27 1.27)) (justify left bottom))
@@
     (effects (font (size 1.27 1.27)) (justify left bottom))
   )
+  (label "x_out" (at 35.052 81.026 180)
+    (effects (font (size 1.27 1.27)) (justify right bottom))
+  )
   (label "USB_BOOT" (at 307.594 27.686 180)
     (effects (font (size 1.27 1.27)) (justify right bottom))
@@
     (effects (font (size 1.27 1.27)) (justify right bottom))
   )
+  (label "Col0" (at 35.052 83.566 180)
+    (effects (font (size 1.27 1.27)) (justify right bottom))
+  )
   (label "XIN_20" (at 253.492 129.032 180)
     (effects (font (size 1.27 1.27)) (justify right bottom))
@@
   (label "IOVDD_33" (at 316.484 141.732 0)
     (effects (font (size 1.27 1.27)) (justify left bottom))
+  )
+  (label "Col1" (at 35.052 86.106 180)
+    (effects (font (size 1.27 1.27)) (justify right bottom))
   )
   (label "XOUT_21" (at 272.542 37.084 0)
@@
     (pin "2")
   )
-  (symbol (lib_id "power:GND") (at 40.894 93.726 0) (unit 1)
-    (in_bom yes) (on_board yes) (fields_autoplaced)
-    (property "Reference" "#PWR?" (id 0) (at 40.894 100.076 0)
-      (effects (font (size 1.27 1.27)) hide)
-    )
-    (property "Value" "GND" (id 1) (at 40.894 98.552 0))
-    (property "Footprint" "" (id 2) (at 40.894 93.726 0)
-      (effects (font (size 1.27 1.27)) hide)
-    )
-    (property "Datasheet" "" (id 3) (at 40.894 93.726 0)
+  (symbol (lib_id "power:GND") (at 63.246 83.566 0) (unit 1)
+    (in_bom yes) (on_board yes) (fields_autoplaced)
+    (property "Reference" "#PWR?" (id 0) (at 63.246 89.916 0)
+      (effects (font (size 1.27 1.27)) hide)
+    )
+    (property "Value" "GND" (id 1) (at 63.246 88.392 0))
+    (property "Footprint" "" (id 2) (at 63.246 83.566 0)
+      (effects (font (size 1.27 1.27)) hide)
+    )
+    (property "Datasheet" "" (id 3) (at 63.246 83.566 0)
       (effects (font (size 1.27 1.27)) hide)
     )
@@
     (pin "2")
   )
-  (symbol (lib_id "power:+3V3") (at 40.894 78.486 0) (unit 1)
-    (in_bom yes) (on_board yes) (fields_autoplaced)
-    (property "Reference" "#PWR?" (id 0) (at 40.894 82.296 0)
-      (effects (font (size 1.27 1.27)) hide)
-    )
-    (property "Value" "" (id 1) (at 40.894 73.66 0))
-    (property "Footprint" "" (id 2) (at 40.894 78.486 0)
-      (effects (font (size 1.27 1.27)) hide)
-    )
-    (property "Datasheet" "" (id 3) (at 40.894 78.486 0)
+  (symbol (lib_id "power:+3V3") (at 53.34 75.946 0) (unit 1)
+    (in_bom yes) (on_board yes) (fields_autoplaced)
+    (property "Reference" "#PWR?" (id 0) (at 53.34 79.756 0)
+      (effects (font (size 1.27 1.27)) hide)
+    )
+    (property "Value" "+3V3" (id 1) (at 53.34 71.12 0))
+    (property "Footprint" "" (id 2) (at 53.34 75.946 0)
+      (effects (font (size 1.27 1.27)) hide)
+    )
+    (property "Datasheet" "" (id 3) (at 53.34 75.946 0)
       (effects (font (size 1.27 1.27)) hide)
     )
@@
     (pin "2")
   )
-  (symbol (lib_id "SWD 0.05 Pitch Connector - 10 Pin:JTAG-CORTEX") (at 31.242 86.106 0) (unit 1)
-    (in_bom yes) (on_board yes) (fields_autoplaced)
-    (property "Reference" "X?" (id 0) (at 31.242 73.66 0))
-    (property "Value" "JTAG-CORTEX" (id 1) (at 31.242 76.2 0))
-    (property "Footprint" "Adafruit SWD Breakout:2X05_1.27MM_SMT" (id 2) (at 31.115 98.2472 0)
-      (effects (font (size 1.27 1.27)) hide)
-    )
-    (property "Datasheet" "" (id 3) (at 31.242 86.106 0)
+  (symbol (lib_id "SWD 0.05 Pitch Connector - 10 Pin:JTAG-CORTEX") (at 43.688 83.566 0) (unit 1)
+    (in_bom yes) (on_board yes) (fields_autoplaced)
+    (property "Reference" "X?" (id 0) (at 43.688 71.12 0))
+    (property "Value" "JTAG-CORTEX" (id 1) (at 43.688 73.66 0))
+    (property "Footprint" "Adafruit SWD Breakout:2X05_1.27MM_SMT" (id 2) (at 43.561 95.7072 0)
+      (effects (font (size 1.27 1.27)) hide)
+    )
+    (property "Datasheet" "" (id 3) (at 43.688 83.566 0)
       (effects (font (size 1.27 1.27)) hide)
     )
     (pin "1")
     (pin "10")
+    (pin "2")
+    (pin "3")
+    (pin "4")
+    (pin "5")
     (pin "6")
-    (pin "2")
     (pin "7")
-    (pin "3")
     (pin "8")
-    (pin "4")
     (pin "9")
-    (pin "5")
   )
   (symbol (lib_id "Switch:SW_SPST") (at 159.258 181.102 0) (unit 1)

Commit message: PCB Updates
Connections:
- net Row2: now also X?.8
- net Row3: now also X?.9
- net Row4: now also X?.10
Other:
- moved on the sheet: X?
Changed lines of the file:
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@@
     (stroke (width 0) (type default) (color 0 0 0 0))
   )
-  (wire (pts (xy 35.052 81.026) (xy 36.068 81.026))
+  (wire (pts (xy 22.352 77.216) (xy 23.368 77.216))
     (stroke (width 0) (type default) (color 0 0 0 0))
   )
@@
     (stroke (width 0) (type default) (color 0 0 0 0))
   )
-  (wire (pts (xy 35.052 78.486) (xy 36.068 78.486))
+  (wire (pts (xy 22.352 74.676) (xy 23.368 74.676))
     (stroke (width 0) (type default) (color 0 0 0 0))
   )
@@
     (stroke (width 0) (type default) (color 0 0 0 0))
   )
-  (wire (pts (xy 35.052 88.646) (xy 36.068 88.646))
+  (wire (pts (xy 22.352 84.836) (xy 23.368 84.836))
     (stroke (width 0) (type default) (color 0 0 0 0))
   )
@@
     (stroke (width 0) (type default) (color 0 0 0 0))
   )
-  (wire (pts (xy 35.052 86.106) (xy 36.068 86.106))
+  (wire (pts (xy 22.352 82.296) (xy 23.368 82.296))
     (stroke (width 0) (type default) (color 0 0 0 0))
   )
@@
     (stroke (width 0) (type default) (color 0 0 0 0))
   )
+  (wire (pts (xy 38.608 79.756) (xy 39.624 79.756))
+    (stroke (width 0) (type default) (color 0 0 0 0))
+  )
   (wire (pts (xy 67.818 181.102) (xy 67.818 183.642))
     (stroke (width 0) (type default) (color 0 0 0 0))
@@
     (stroke (width 0) (type default) (color 0 0 0 0))
   )
-  (wire (pts (xy 35.052 83.566) (xy 36.068 83.566))
+  (wire (pts (xy 22.352 79.756) (xy 23.368 79.756))
     (stroke (width 0) (type default) (color 0 0 0 0))
   )
@@
     (stroke (width 0) (type default) (color 0 0 0 0))
   )
-  (wire (pts (xy 51.308 78.486) (xy 53.34 78.486))
+  (wire (pts (xy 38.608 74.676) (xy 40.64 74.676))
     (stroke (width 0) (type default) (color 0 0 0 0))
   )
@@
     (stroke (width 0) (type default) (color 0 0 0 0))
   )
+  (wire (pts (xy 38.608 84.836) (xy 39.624 84.836))
+    (stroke (width 0) (type default) (color 0 0 0 0))
+  )
   (wire (pts (xy 48.006 171.958) (xy 67.818 171.958))
     (stroke (width 0) (type default) (color 0 0 0 0))
@@
     (stroke (width 0) (type default) (color 0 0 0 0))
   )
-  (wire (pts (xy 51.308 81.026) (xy 63.246 81.026))
+  (wire (pts (xy 38.608 77.216) (xy 50.546 77.216))
     (stroke (width 0) (type default) (color 0 0 0 0))
   )
@@
     (stroke (width 0) (type default) (color 0 0 0 0))
   )
+  (wire (pts (xy 38.608 82.296) (xy 39.624 82.296))
+    (stroke (width 0) (type default) (color 0 0 0 0))
+  )
   (wire (pts (xy 100.584 30.48) (xy 110.236 30.48))
     (stroke (width 0) (type default) (color 0 0 0 0))
@@
     (stroke (width 0) (type default) (color 0 0 0 0))
   )
-  (wire (pts (xy 63.246 81.026) (xy 63.246 83.566))
+  (wire (pts (xy 50.546 77.216) (xy 50.546 79.756))
     (stroke (width 0) (type default) (color 0 0 0 0))
   )
@@
     (stroke (width 0) (type default) (color 0 0 0 0))
   )
-  (wire (pts (xy 53.34 75.946) (xy 53.34 78.486))
+  (wire (pts (xy 40.64 72.136) (xy 40.64 74.676))
     (stroke (width 0) (type default) (color 0 0 0 0))
   )
@@
     (effects (font (size 1.27 1.27)) (justify right bottom))
   )
-  (label "y_out" (at 35.052 78.486 180)
+  (label "y_out" (at 22.352 74.676 180)
     (effects (font (size 1.27 1.27)) (justify right bottom))
   )
@@
     (effects (font (size 1.27 1.27)) (justify left bottom))
   )
-  (label "Col2" (at 35.052 88.646 180)
+  (label "Col2" (at 22.352 84.836 180)
     (effects (font (size 1.27 1.27)) (justify right bottom))
   )
@@
     (effects (font (size 1.27 1.27)) (justify left bottom))
   )
-  (label "x_out" (at 35.052 81.026 180)
+  (label "x_out" (at 22.352 77.216 180)
     (effects (font (size 1.27 1.27)) (justify right bottom))
   )
@@
     (effects (font (size 1.27 1.27)) (justify right bottom))
   )
-  (label "Col0" (at 35.052 83.566 180)
+  (label "Col0" (at 22.352 79.756 180)
     (effects (font (size 1.27 1.27)) (justify right bottom))
   )
@@
     (effects (font (size 1.27 1.27)) (justify right bottom))
   )
+  (label "Row3" (at 39.624 82.296 0)
+    (effects (font (size 1.27 1.27)) (justify left bottom))
+  )
   (label "QSPI_SD2_54" (at 316.484 88.392 0)
     (effects (font (size 1.27 1.27)) (justify left bottom))
@@
     (effects (font (size 1.27 1.27)) (justify left bottom))
   )
-  (label "Col1" (at 35.052 86.106 180)
-    (effects (font (size 1.27 1.27)) (justify right bottom))
+  (label "Col1" (at 22.352 82.296 180)
+    (effects (font (size 1.27 1.27)) (justify right bottom))
+  )
+  (label "Row4" (at 39.624 84.836 0)
+    (effects (font (size 1.27 1.27)) (justify left bottom))
   )
   (label "XOUT_21" (at 272.542 37.084 0)
+    (effects (font (size 1.27 1.27)) (justify left bottom))
+  )
+  (label "Row2" (at 39.624 79.756 0)
     (effects (font (size 1.27 1.27)) (justify left bottom))
   )
@@
     (pin "2")
   )
-  (symbol (lib_id "power:GND") (at 63.246 83.566 0) (unit 1)
-    (in_bom yes) (on_board yes) (fields_autoplaced)
-    (property "Reference" "#PWR?" (id 0) (at 63.246 89.916 0)
-      (effects (font (size 1.27 1.27)) hide)
-    )
-    (property "Value" "GND" (id 1) (at 63.246 88.392 0))
-    (property "Footprint" "" (id 2) (at 63.246 83.566 0)
-      (effects (font (size 1.27 1.27)) hide)
-    )
-    (property "Datasheet" "" (id 3) (at 63.246 83.566 0)
+  (symbol (lib_id "power:GND") (at 50.546 79.756 0) (unit 1)
+    (in_bom yes) (on_board yes) (fields_autoplaced)
+    (property "Reference" "#PWR?" (id 0) (at 50.546 86.106 0)
+      (effects (font (size 1.27 1.27)) hide)
+    )
+    (property "Value" "GND" (id 1) (at 50.546 84.582 0))
+    (property "Footprint" "" (id 2) (at 50.546 79.756 0)
+      (effects (font (size 1.27 1.27)) hide)
+    )
+    (property "Datasheet" "" (id 3) (at 50.546 79.756 0)
       (effects (font (size 1.27 1.27)) hide)
     )
@@
     (pin "2")
   )
-  (symbol (lib_id "power:+3V3") (at 53.34 75.946 0) (unit 1)
-    (in_bom yes) (on_board yes) (fields_autoplaced)
-    (property "Reference" "#PWR?" (id 0) (at 53.34 79.756 0)
-      (effects (font (size 1.27 1.27)) hide)
-    )
-    (property "Value" "+3V3" (id 1) (at 53.34 71.12 0))
-    (property "Footprint" "" (id 2) (at 53.34 75.946 0)
-      (effects (font (size 1.27 1.27)) hide)
-    )
-    (property "Datasheet" "" (id 3) (at 53.34 75.946 0)
+  (symbol (lib_id "power:+3V3") (at 40.64 72.136 0) (unit 1)
+    (in_bom yes) (on_board yes) (fields_autoplaced)
+    (property "Reference" "#PWR?" (id 0) (at 40.64 75.946 0)
+      (effects (font (size 1.27 1.27)) hide)
+    )
+    (property "Value" "+3V3" (id 1) (at 40.64 67.31 0))
+    (property "Footprint" "" (id 2) (at 40.64 72.136 0)
+      (effects (font (size 1.27 1.27)) hide)
+    )
+    (property "Datasheet" "" (id 3) (at 40.64 72.136 0)
       (effects (font (size 1.27 1.27)) hide)
     )
@@
     (pin "2")
   )
-  (symbol (lib_id "SWD 0.05 Pitch Connector - 10 Pin:JTAG-CORTEX") (at 43.688 83.566 0) (unit 1)
-    (in_bom yes) (on_board yes) (fields_autoplaced)
-    (property "Reference" "X?" (id 0) (at 43.688 71.12 0))
-    (property "Value" "JTAG-CORTEX" (id 1) (at 43.688 73.66 0))
-    (property "Footprint" "Adafruit SWD Breakout:2X05_1.27MM_SMT" (id 2) (at 43.561 95.7072 0)
-      (effects (font (size 1.27 1.27)) hide)
-    )
-    (property "Datasheet" "" (id 3) (at 43.688 83.566 0)
-      (effects (font (size 1.27 1.27)) hide)
-    )
+  (symbol (lib_id "SWD 0.05 Pitch Connector - 10 Pin:JTAG-CORTEX") (at 30.988 79.756 0) (unit 1)
+    (in_bom yes) (on_board yes) (fields_autoplaced)
+    (property "Reference" "X?" (id 0) (at 30.988 67.31 0))
+    (property "Value" "JTAG-CORTEX" (id 1) (at 30.988 69.85 0))
+    (property "Footprint" "Adafruit SWD Breakout:2X05_1.27MM_SMT" (id 2) (at 30.861 91.8972 0)
+      (effects (font (size 1.27 1.27)) hide)
+    )
+    (property "Datasheet" "" (id 3) (at 30.988 79.756 0)
+      (effects (font (size 1.27 1.27)) hide)
+    )

Commit message: PCB Updates
Parts:
- C13, C14: footprint Capacitor_SMD:C_0402_1005Metric_Pad0.74x0.62mm_HandSolder -> (none)
- S1: footprint NCP1117ST33T3G:SOT230P700X180-4N -> (none)
- X1: renamed from X?; footprint Adafruit SWD Breakout:2X05_1.27MM_SMT -> (none)
Connections:
- net Col10: now also U2.14 (GPIO11)
- net Col11: now also U2.15 (GPIO12)
- net Col12: now also U2.16 (GPIO13)
- net Col3: now also U2.6 (GPIO4)
- net Col4: now also U2.7 (GPIO5)
- net Col5: now also U2.8 (GPIO6)
- net Col6: now also U2.9 (GPIO7)
- net Col7: now also U2.11 (GPIO8)
- net Col8: now also U2.12 (GPIO9)
- net Col9: now also U2.13 (GPIO10)
- net Row2: now also U2.2 (GPIO0)
- net Row3: now also U2.3 (GPIO1)
- net Row4: now also U2.4 (GPIO2)
- net Row5: now also U2.5 (GPIO3)
