File: KiCAD_PCB/Calculator_PCB/Calculator_PCB.kicad_sch (KiCad schematic)
At the start: 109 parts, among them J1 USB_B_Micro, SW1 SW_SPST, SW10 SW_SPST, SW11 SW_SPST, SW12 SW_SPST, SW13 SW_SPST, SW14 SW_SPST, SW15 SW_SPST, SW16 SW_SPST, SW17 SW_SPST, SW18 SW_SPST, SW19 SW_SPST, SW2 SW_SPST, SW20 SW_SPST, SW21 SW_SPST, SW22 SW_SPST, SW23 SW_SPST, SW24 SW_SPST, SW25 SW_SPST, SW26 SW_SPST, SW27 SW_SPST, SW28 SW_SPST, SW29 SW_SPST, SW3 SW_SPST, SW30 SW_SPST, SW31 SW_SPST, SW32 SW_SPST, SW33 SW_SPST, SW34 SW_SPST, SW35 SW_SPST, SW36 SW_SPST, SW37 SW_SPST, SW38 SW_SPST, SW39 SW_SPST, SW4 SW_SPST, SW40 SW_SPST, SW5 SW_SPST, SW6 SW_SPST, SW7 SW_SPST, SW8 SW_SPST, SW9 SW_SPST, U1 W25Q128JVS, U2 RP2040, U3 NCP1117-3.3_SOT223, X1 JTAG-CORTEX, Y1 ABLS-12.000MHZ-B4-T

Commit message: PCB Update
Parts:
- C13, C14: footprint (none) -> Capacitor_SMD:C_0805_2012Metric_Pad1.18x1.45mm_HandSolder
- S1: footprint (none) -> PTS810SJK250SMTRLFS:PTS810SJG250SMTRLFS
- X1: footprint (none) -> Adafruit_Connectors:2X05_1.27MM_BOX_POSTS
Connections:
- net Col0: now also U2.27 (GPIO16)
- net Col1: now also U2.18 (GPIO15)
- net Col10: now also U2.8 (GPIO6); no longer U2.14 (GPIO11)
- net Col11: now also U2.7 (GPIO5); no longer U2.15 (GPIO12)
- net Col12: now also U2.6 (GPIO4); no longer U2.16 (GPIO13)
- net Col2: now also U2.17 (GPIO14)
- net Col3: now also U2.16 (GPIO13); no longer U2.6 (GPIO4)
- net Col4: now also U2.15 (GPIO12); no longer U2.7 (GPIO5)
- net Col5: now also U2.14 (GPIO11); no longer U2.8 (GPIO6)
- net Col6: now also U2.13 (GPIO10); no longer U2.9 (GPIO7)
- net Col7: now also U2.12 (GPIO9); no longer U2.11 (GPIO8)
- net Col8: now also U2.11 (GPIO8); no longer U2.12 (GPIO9)
- net Col9: now also U2.9 (GPIO7); no longer U2.13 (GPIO10)
Changed lines of the file:
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@@
     (stroke (width 0) (type default) (color 0 0 0 0))
   )
+  (wire (pts (xy 253.492 146.812) (xy 254.508 146.812))
+    (stroke (width 0) (type default) (color 0 0 0 0))
+  )
   (wire (pts (xy 315.468 101.092) (xy 316.484 101.092))
     (stroke (width 0) (type default) (color 0 0 0 0))
@@
     (stroke (width 0) (type default) (color 0 0 0 0))
   )
+  (wire (pts (xy 253.492 121.412) (xy 254.508 121.412))
+    (stroke (width 0) (type default) (color 0 0 0 0))
+  )
   (wire (pts (xy 73.406 37.338) (xy 73.406 41.656))
     (stroke (width 0) (type default) (color 0 0 0 0))
@@
     (stroke (width 0) (type default) (color 0 0 0 0))
   )
+  (wire (pts (xy 253.492 123.952) (xy 254.508 123.952))
+    (stroke (width 0) (type default) (color 0 0 0 0))
+  )
   (wire (pts (xy 68.834 146.05) (xy 67.818 146.05))
     (stroke (width 0) (type default) (color 0 0 0 0))
@@
     (effects (font (size 1.27 1.27)) (justify left bottom))
   )
-  (label "Col6" (at 253.492 101.092 180)
+  (label "Col9" (at 253.492 101.092 180)
     (effects (font (size 1.27 1.27)) (justify right bottom))
   )
-  (label "Col3" (at 253.492 93.472 180)
+  (label "Col12" (at 253.492 93.472 180)
     (effects (font (size 1.27 1.27)) (justify right bottom))
   )
@@
     (effects (font (size 1.27 1.27)) (justify right bottom))
   )
-  (label "Col11" (at 253.492 116.332 180)
+  (label "Col4" (at 253.492 116.332 180)
     (effects (font (size 1.27 1.27)) (justify right bottom))
   )
@@
     (effects (font (size 1.27 1.27)) (justify left bottom))
   )
+  (label "Col1" (at 253.492 123.952 180)
+    (effects (font (size 1.27 1.27)) (justify right bottom))
+  )
   (label "IOVDD_1" (at 253.492 80.772 180)
     (effects (font (size 1.27 1.27)) (justify right bottom))
@@
     (effects (font (size 1.27 1.27)) (justify right bottom))
   )
-  (label "Col8" (at 253.492 108.712 180)
+  (label "Col7" (at 253.492 108.712 180)
     (effects (font (size 1.27 1.27)) (justify right bottom))
   )
@@
     (effects (font (size 1.27 1.27)) (justify right bottom))
   )
+  (label "Col0" (at 253.492 146.812 180)
+    (effects (font (size 1.27 1.27)) (justify right bottom))
+  )
   (label "USB_BOOT" (at 307.594 27.686 180)
     (effects (font (size 1.27 1.27)) (justify right bottom))
@@
     (effects (font (size 1.27 1.27)) (justify right bottom))
   )
-  (label "Col7" (at 253.492 106.172 180)
+  (label "Col8" (at 253.492 106.172 180)
     (effects (font (size 1.27 1.27)) (justify right bottom))
   )
@@
     (effects (font (size 1.27 1.27)) (justify left bottom))
   )
-  (label "Col9" (at 253.492 111.252 180)
+  (label "Col6" (at 253.492 111.252 180)
     (effects (font (size 1.27 1.27)) (justify right bottom))
   )
@@
     (effects (font (size 1.27 1.27)) (justify right bottom))
   )
-  (label "Col12" (at 253.492 118.872 180)
+  (label "Col2" (at 253.492 121.412 180)
+    (effects (font (size 1.27 1.27)) (justify right bottom))
+  )
+  (label "Col3" (at 253.492 118.872 180)
     (effects (font (size 1.27 1.27)) (justify right bottom))
   )
@@
     (effects (font (size 1.27 1.27)) (justify right bottom))
   )
-  (label "Col4" (at 253.492 96.012 180)
+  (label "Col11" (at 253.492 96.012 180)
     (effects (font (size 1.27 1.27)) (justify right bottom))
   )
@@
     (effects (font (size 1.27 1.27)) (justify right bottom))
   )
-  (label "Col5" (at 253.492 98.552 180)
+  (label "Col10" (at 253.492 98.552 180)
     (effects (font (size 1.27 1.27)) (justify right bottom))
   )
@@
     (effects (font (size 1.27 1.27)) (justify right bottom))
   )
-  (label "Col10" (at 253.492 113.792 180)
+  (label "Col5" (at 253.492 113.792 180)
     (effects (font (size 1.27 1.27)) (justify right bottom))
   )
@@
       (effects (font (size 1.27 1.27)) (justify left))
     )
-    (property "Footprint" "" (id 2) (at 181.61 34.036 0)
+    (property "Footprint" "Capacitor_SMD:C_0805_2012Metric_Pad1.18x1.45mm_HandSolder" (id 2) (at 181.61 34.036 0)
       (effects (font (size 1.27 1.27)) hide)
     )
@@
     (property "Reference" "S1" (id 0) (at 321.31 29.972 0))
     (property "Value" "PTS810SJK250SMTRLFS" (id 1) (at 321.31 32.512 0))
-    (property "Footprint" "" (id 2) (at 311.15 37.338 0)
+    (property "Footprint" "PTS810SJK250SMTRLFS:PTS810SJG250SMTRLFS" (id 2) (at 311.15 37.338 0)
       (effects (font (size 1.27 1.27)) (justify left bottom) hide)
     )
@@
     (property "Reference" "X1" (id 0) (at 30.988 67.31 0))
     (property "Value" "JTAG-CORTEX" (id 1) (at 30.988 69.85 0))
-    (property "Footprint" "" (id 2) (at 30.861 91.8972 0)
+    (property "Footprint" "Adafruit_Connectors:2X05_1.27MM_BOX_POSTS" (id 2) (at 30.861 91.8972 0)
       (effects (font (size 1.27 1.27)) hide)
     )
@@
       (effects (font (size 1.27 1.27)) (justify left))
     )
-    (property "Footprint" "" (id 2) (at 213.614 34.036 0)
+    (property "Footprint" "Capacitor_SMD:C_0805_2012Metric_Pad1.18x1.45mm_HandSolder" (id 2) (at 213.614 34.036 0)
       (effects (font (size 1.27 1.27)) hide)
     )

Commit message: PCB Updates
Parts:
- added X2: JTAG-CORTEX, Adafruit_Connectors:2X05_1.27MM_BOX_POSTS, symbol SWD 0.05 Pitch Connector - 10 Pin:JTAG-CORTEX
Changed lines of the file:
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@@
     (pin "2")
+  )
+  (symbol (lib_id "SWD 0.05 Pitch Connector - 10 Pin:JTAG-CORTEX") (at 75.438 78.994 0) (unit 1)
+    (in_bom yes) (on_board yes) (fields_autoplaced)
+    (property "Reference" "X2" (id 0) (at 75.438 66.548 0))
+    (property "Value" "JTAG-CORTEX" (id 1) (at 75.438 69.088 0))
+    (property "Footprint" "Adafruit_Connectors:2X05_1.27MM_BOX_POSTS" (id 2) (at 75.311 91.1352 0)
+      (effects (font (size 1.27 1.27)) hide)
+    )
+    (property "Datasheet" "" (id 3) (at 75.438 78.994 0)
+      (effects (font (size 1.27 1.27)) hide)
+    )
+    (pin "1")
+    (pin "10")
+    (pin "2")
+    (pin "3")
+    (pin "4")
+    (pin "5")
+    (pin "6")
+    (pin "7")
+    (pin "8")
+    (pin "9")
   )
   (symbol (lib_id "Device:D_Small") (at 51.562 169.418 0) (unit 1)
@@
       (reference "X1") (unit 1) (value "JTAG-CORTEX") (footprint "Adafruit_Connectors:2X05_1.27MM_BOX_POSTS")
     )
+    (path "/a410bf48-ecc7-4ea9-8439-ef92bc056f8c"
+      (reference "X2") (unit 1) (value "JTAG-CORTEX") (footprint "Adafruit_Connectors:2X05_1.27MM_BOX_POSTS")
+    )
     (path "/4e8e0e6c-e85f-4a14-acfd-40545e44f4fc"

Commit message: PCB Updates
Parts:
- removed X1, X2: JTAG-CORTEX, Adafruit_Connectors:2X05_1.27MM_BOX_POSTS, symbol SWD 0.05 Pitch Connector - 10 Pin:JTAG-CORTEX
- added J?: 5034801000, MOLEX_5034801000, symbol 5034801000:5034801000
- added J?: (no value), symbol 5034801000:5034801000
Connections:
- net +3V3: now also J?.1
- net Col0: now also J?.5
- net Col1: now also J?.6
- net Col2: now also J?.7
- net GND: now also J?.4
- net Row2: now also J?.10
- net Row3: now also J?.9
- net Row4: now also J?.8
- net x_out: now also J?.3
- net y_out: now also J?.2
- new net: J?.S1 (SHIELD), J?.S2 (SHIELD) (x2)
- no-connect marks 1 -> 3

Commit message: PCB Udpates
Parts:
- J3: renamed from J?; footprint MOLEX_5034801000 -> (none)
- gave numbers to parts that had none: 1
Changed lines of the file:
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@@
   (symbol (lib_id "5034801000:5034801000") (at 96.266 84.836 0) (unit 1)
     (in_bom yes) (on_board yes) (fields_autoplaced)
-    (property "Reference" "J?" (id 0) (at 102.616 82.2959 0)
+    (property "Reference" "J3" (id 0) (at 102.616 82.2959 0)
       (effects (font (size 1.27 1.27)) (justify left))
     )
@@
       (effects (font (size 1.27 1.27)) (justify left))
     )
-    (property "Footprint" "MOLEX_5034801000" (id 2) (at 96.266 84.836 0)
+    (property "Footprint" "" (id 2) (at 96.266 84.836 0)
       (effects (font (size 1.27 1.27)) (justify left bottom) hide)
     )
@@
   (symbol (lib_id "5034801000:5034801000") (at 41.656 86.106 0) (unit 1)
     (in_bom yes) (on_board yes) (fields_autoplaced)
-    (property "Reference" "J?" (id 0) (at 48.006 83.5659 0)
+    (property "Reference" "J2" (id 0) (at 48.006 83.5659 0)
       (effects (font (size 1.27 1.27)) (justify left))
     )
@@
       (reference "J1") (unit 1) (value "USB_B_Micro") (footprint "Connector_USB:USB_Micro-B_Amphenol_10103594-0001LF_Horizontal")
     )
+    (path "/6b1ec389-895f-4d08-872b-0bc205aa059c"
+      (reference "J2") (unit 1) (value "5034801000") (footprint "5034801000:MOLEX_5034801000")
+    )
     (path "/2fce0416-25ce-42d1-b0da-bfd7a6ca89c1"
-      (reference "J?") (unit 1) (value "5034801000") (footprint "MOLEX_5034801000")
-    )
-    (path "/6b1ec389-895f-4d08-872b-0bc205aa059c"
-      (reference "J?") (unit 1) (value "5034801000") (footprint "MOLEX_5034801000")
+      (reference "J3") (unit 1) (value "5034801000") (footprint "5034801000:MOLEX_5034801000")
     )
     (path "/29f71695-b47c-4fbb-b52b-07876a33a1d5"
