File: KiCAD_PCB/Calculator_PCB/Calculator_PCB.kicad_sch (KiCad schematic)
At the start: 110 parts, among them J1 USB_B_Micro, J3 5034801000, SW1 SW_SPST, SW10 SW_SPST, SW11 SW_SPST, SW12 SW_SPST, SW13 SW_SPST, SW14 SW_SPST, SW15 SW_SPST, SW16 SW_SPST, SW17 SW_SPST, SW18 SW_SPST, SW19 SW_SPST, SW2 SW_SPST, SW20 SW_SPST, SW21 SW_SPST, SW22 SW_SPST, SW23 SW_SPST, SW24 SW_SPST, SW25 SW_SPST, SW26 SW_SPST, SW27 SW_SPST, SW28 SW_SPST, SW29 SW_SPST, SW3 SW_SPST, SW30 SW_SPST, SW31 SW_SPST, SW32 SW_SPST, SW33 SW_SPST, SW34 SW_SPST, SW35 SW_SPST, SW36 SW_SPST, SW37 SW_SPST, SW38 SW_SPST, SW39 SW_SPST, SW4 SW_SPST, SW40 SW_SPST, SW5 SW_SPST, SW6 SW_SPST, SW7 SW_SPST, SW8 SW_SPST, SW9 SW_SPST, U1 W25Q128JVS, U2 RP2040, U3 NCP1117-3.3_SOT223, Y1 ABLS-12.000MHZ-B4-T

Commit message: PCB Updates
Connections:
- net Row2: now also U2.5 (GPIO3); no longer U2.2 (GPIO0)
- net Row3: now also U2.4 (GPIO2); no longer U2.3 (GPIO1)
- net Row4: now also U2.3 (GPIO1); no longer U2.4 (GPIO2)
- net Row5: now also U2.2 (GPIO0); no longer U2.5 (GPIO3)
Changed lines of the file:
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@@
     (effects (font (size 1.27 1.27)) (justify right bottom))
   )
-  (label "Row4" (at 253.492 88.392 180)
+  (label "Row3" (at 253.492 88.392 180)
     (effects (font (size 1.27 1.27)) (justify right bottom))
   )
-  (label "Row5" (at 253.492 90.932 180)
+  (label "Row2" (at 253.492 90.932 180)
     (effects (font (size 1.27 1.27)) (justify right bottom))
   )
@@
     (effects (font (size 1.27 1.27)) (justify right bottom))
   )
-  (label "Row3" (at 253.492 85.852 180)
+  (label "Row4" (at 253.492 85.852 180)
     (effects (font (size 1.27 1.27)) (justify right bottom))
   )
@@
     (effects (font (size 1.27 1.27)) (justify right bottom))
   )
-  (label "Row2" (at 253.492 83.312 180)
+  (label "Row5" (at 253.492 83.312 180)
     (effects (font (size 1.27 1.27)) (justify right bottom))
   )

Commit message: PCB Updates
Parts:
- J2: value (none) -> 5034801000; footprint (none) -> 5034801000:MOLEX_5034801000
- J3: footprint (none) -> 5034801000:MOLEX_5034801000
Connections:
- net Row2: no longer J2.10
- net Row3: now also J2.8; no longer J2.9
- net Row4: now also J2.9; no longer J2.8
- net Row5: now also J2.10
Changed lines of the file:
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@@
     (effects (font (size 1.27 1.27)) (justify right bottom))
   )
-  (label "Row3" (at 30.48 91.186 180)
+  (label "Row4" (at 30.48 91.186 180)
     (effects (font (size 1.27 1.27)) (justify right bottom))
   )
@@
     (effects (font (size 1.27 1.27)) (justify right bottom))
   )
-  (label "Row4" (at 30.48 88.646 180)
+  (label "Row5" (at 30.48 93.726 180)
     (effects (font (size 1.27 1.27)) (justify right bottom))
   )
@@
     (effects (font (size 1.27 1.27)) (justify left bottom))
   )
-  (label "Row2" (at 30.48 93.726 180)
+  (label "Row3" (at 30.48 88.646 180)
     (effects (font (size 1.27 1.27)) (justify right bottom))
   )
@@
       (effects (font (size 1.27 1.27)) (justify left))
     )
-    (property "Footprint" "" (id 2) (at 96.266 84.836 0)
+    (property "Footprint" "5034801000:MOLEX_5034801000" (id 2) (at 96.266 84.836 0)
       (effects (font (size 1.27 1.27)) (justify left bottom) hide)
     )
@@
       (effects (font (size 1.27 1.27)) (justify left))
     )
-    (property "Value" "" (id 1) (at 48.006 86.1059 0)
-      (effects (font (size 1.27 1.27)) (justify left))
-    )
-    (property "Footprint" "" (id 2) (at 41.656 86.106 0)
+    (property "Value" "5034801000" (id 1) (at 48.006 86.1059 0)
+      (effects (font (size 1.27 1.27)) (justify left))
+    )
+    (property "Footprint" "5034801000:MOLEX_5034801000" (id 2) (at 41.656 86.106 0)
       (effects (font (size 1.27 1.27)) (justify left bottom) hide)
     )

Commit message: PCB Updates
Connections:
- net Row3: now also J2.10; no longer J2.8
- net Row5: now also J2.8; no longer J2.10
Changed lines of the file:
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@@
     (effects (font (size 1.27 1.27)) (justify right bottom))
   )
-  (label "Row5" (at 30.48 93.726 180)
+  (label "Row5" (at 30.48 88.646 180)
     (effects (font (size 1.27 1.27)) (justify right bottom))
   )
@@
     (effects (font (size 1.27 1.27)) (justify left bottom))
   )
-  (label "Row3" (at 30.48 88.646 180)
+  (label "Row3" (at 30.48 93.726 180)
     (effects (font (size 1.27 1.27)) (justify right bottom))
   )

Commit message: PCB Updates
Connections:
- net Row2 is gone; now on net Row3: D1.1 (K), D13.1 (K), D17.1 (K), D21.1 (K), D25.1 (K), D29.1 (K), D33.1 (K), D37.1 (K), D5.1 (K), D9.1 (K), U2.5 (GPIO3)
- net +3V3: now also J2.9; no longer J2.1
- net Col0: now also J2.4; no longer J2.5
- net Col1: now also J2.5; no longer J2.6
- net Col2: now also J2.6; no longer J2.7
- net GND: now also J2.10; no longer J2.4
- net Row3: no longer D10.1 (K), D14.1 (K), D18.1 (K), D2.1 (K), D22.1 (K), D26.1 (K), D30.1 (K), D34.1 (K), D38.1 (K), D6.1 (K), J2.10, U2.4 (GPIO2)
- net Row4: now also D10.1 (K), D14.1 (K), D18.1 (K), D2.1 (K), D22.1 (K), D26.1 (K), D30.1 (K), D34.1 (K), D38.1 (K), D6.1 (K), J2.1, U2.4 (GPIO2); no longer D11.1 (K), D15.1 (K), D19.1 (K), D23.1 (K), D27.1 (K), D3.1 (K), D31.1 (K), D35.1 (K), D39.1 (K), D7.1 (K), J2.9, U2.3 (GPIO1)
- net Row5: now also D11.1 (K), D15.1 (K), D19.1 (K), D23.1 (K), D27.1 (K), D3.1 (K), D31.1 (K), D35.1 (K), D39.1 (K), D7.1 (K), J2.2, U2.3 (GPIO1); no longer D12.1 (K), D16.1 (K), D20.1 (K), D24.1 (K), D28.1 (K), D32.1 (K), D36.1 (K), D4.1 (K), D40.1 (K), D8.1 (K), J2.8, U2.2 (GPIO0)
- net x_out: now also J2.7; no longer J2.3
- net y_out: now also J2.8; no longer J2.2
- new net Row6: D12.1 (K), D16.1 (K), D20.1 (K), D24.1 (K), D28.1 (K), D32.1 (K), D36.1 (K), D4.1 (K), D40.1 (K), D8.1 (K), J2.3, U2.2 (GPIO0)

Commit message: PCB Updates
Connections:
- net +3V3: now also J2.4; no longer J2.9
- net Col0: now also J2.9, U2.17 (GPIO14); no longer J2.4, U2.27 (GPIO16)
- net Col1: now also J2.10; no longer J2.5
- net Col2: now also J2.8, U2.27 (GPIO16); no longer J2.6, U2.17 (GPIO14)
- net GND: now also J2.5; no longer J2.10
- net x_out: now also J2.6, U2.40 (GPIO28/ADC2); no longer J2.7
- net y_out: now also J2.7, U2.39 (GPIO27/ADC1); no longer J2.8

Commit message: PCB Updates
Connections:
- net Row3: now also J3.5
- net Row4: now also J3.4
- net Row5: now also J3.3
- net Row6: now also J3.2
- net Row7: now reaches J3.1
- net Col15: now reaches J3.10
- net Row2: now reaches J3.6
- net Row1: now reaches J3.7
- net Col13: now reaches J3.8
- net Col14: now reaches J3.9
Changed lines of the file:
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@@
+    (stroke (width 0) (type default) (color 0 0 0 0))
+  )
+  (wire (pts (xy 85.09 77.216) (xy 86.106 77.216))
     (stroke (width 0) (type default) (color 0 0 0 0))
   )
@@
     (stroke (width 0) (type default) (color 0 0 0 0))
   )
+  (wire (pts (xy 85.09 92.456) (xy 86.106 92.456))
+    (stroke (width 0) (type default) (color 0 0 0 0))
+  )
   (wire (pts (xy 223.774 169.418) (xy 223.774 181.102))
     (stroke (width 0) (type default) (color 0 0 0 0))
@@
     (stroke (width 0) (type default) (color 0 0 0 0))
   )
+  (wire (pts (xy 85.09 74.676) (xy 86.106 74.676))
+    (stroke (width 0) (type default) (color 0 0 0 0))
+  )
   (wire (pts (xy 212.598 169.418) (xy 213.614 169.418))
     (stroke (width 0) (type default) (color 0 0 0 0))
@@
     (stroke (width 0) (type default) (color 0 0 0 0))
   )
+  (wire (pts (xy 85.09 69.596) (xy 86.106 69.596))
+    (stroke (width 0) (type default) (color 0 0 0 0))
+  )
   (wire (pts (xy 315.468 103.632) (xy 316.484 103.632))
     (stroke (width 0) (type default) (color 0 0 0 0))
@@
     (stroke (width 0) (type default) (color 0 0 0 0))
   )
+  (wire (pts (xy 85.09 79.756) (xy 86.106 79.756))
+    (stroke (width 0) (type default) (color 0 0 0 0))
+  )
   (wire (pts (xy 107.442 146.05) (xy 107.442 148.59))
     (stroke (width 0) (type default) (color 0 0 0 0))
@@
     (stroke (width 0) (type default) (color 0 0 0 0))
   )
+  (wire (pts (xy 85.09 72.136) (xy 86.106 72.136))
+    (stroke (width 0) (type default) (color 0 0 0 0))
+  )
   (wire (pts (xy 45.466 157.734) (xy 45.466 169.418))
     (stroke (width 0) (type default) (color 0 0 0 0))
   )
+  (wire (pts (xy 85.09 89.916) (xy 86.106 89.916))
+    (stroke (width 0) (type default) (color 0 0 0 0))
+  )
   (wire (pts (xy 108.458 181.102) (xy 107.442 181.102))
     (stroke (width 0) (type default) (color 0 0 0 0))
@@
     (stroke (width 0) (type default) (color 0 0 0 0))
   )
+  (wire (pts (xy 85.09 84.836) (xy 86.106 84.836))
+    (stroke (width 0) (type default) (color 0 0 0 0))
+  )
   (wire (pts (xy 25.654 160.274) (xy 28.194 160.274))
     (stroke (width 0) (type default) (color 0 0 0 0))
@@
     (stroke (width 0) (type default) (color 0 0 0 0))
   )
+  (wire (pts (xy 85.09 82.296) (xy 86.106 82.296))
+    (stroke (width 0) (type default) (color 0 0 0 0))
+  )
   (wire (pts (xy 253.492 116.332) (xy 254.508 116.332))
     (stroke (width 0) (type default) (color 0 0 0 0))
@@
   )
   (wire (pts (xy 85.09 146.05) (xy 85.09 157.734))
+    (stroke (width 0) (type default) (color 0 0 0 0))
+  )
+  (wire (pts (xy 85.09 87.376) (xy 86.106 87.376))
     (stroke (width 0) (type default) (color 0 0 0 0))
   )
@@
     (effects (font (size 1.27 1.27)) (justify right bottom))
   )
+  (label "Row3" (at 85.09 79.756 180)
+    (effects (font (size 1.27 1.27)) (justify right bottom))
+  )
   (label "IOVDD_49" (at 50.8 41.656 270)
     (effects (font (size 1.27 1.27)) (justify right bottom))
@@
     (effects (font (size 1.27 1.27)) (justify right bottom))
   )
+  (label "Row2" (at 85.09 82.296 180)
+    (effects (font (size 1.27 1.27)) (justify right bottom))
+  )
+  (label "Row5" (at 85.09 74.676 180)
+    (effects (font (size 1.27 1.27)) (justify right bottom))
+  )
   (label "RUN_26" (at 247.904 165.608 180)
     (effects (font (size 1.27 1.27)) (justify right bottom))
@@
     (effects (font (size 1.27 1.27)) (justify left bottom))
   )
+  (label "Col14" (at 85.09 89.916 180)
+    (effects (font (size 1.27 1.27)) (justify right bottom))
+  )
   (label "x_out" (at 30.48 83.566 180)
     (effects (font (size 1.27 1.27)) (justify right bottom))
@@
     (effects (font (size 1.27 1.27)) (justify right bottom))
   )
+  (label "Row7" (at 85.09 69.596 180)
+    (effects (font (size 1.27 1.27)) (justify right bottom))
+  )
   (label "USB_BOOT" (at 307.594 27.686 180)
     (effects (font (size 1.27 1.27)) (justify right bottom))
@@
     (effects (font (size 1.27 1.27)) (justify right bottom))
   )
+  (label "Col15" (at 85.09 92.456 180)
+    (effects (font (size 1.27 1.27)) (justify right bottom))
+  )
   (label "XIN_20" (at 272.542 29.972 0)
     (effects (font (size 1.27 1.27)) (justify left bottom))
   )
+  (label "Row6" (at 85.09 72.136 180)
+    (effects (font (size 1.27 1.27)) (justify right bottom))
+  )
   (label "Col6" (at 253.492 111.252 180)
     (effects (font (size 1.27 1.27)) (justify right bottom))
@@
     (effects (font (size 1.27 1.27)) (justify right bottom))
   )
+  (label "Row1" (at 85.09 84.836 180)
+    (effects (font (size 1.27 1.27)) (justify right bottom))
+  )
   (label "Col0" (at 30.48 91.186 180)
     (effects (font (size 1.27 1.27)) (justify right bottom))
@@
     (effects (font (size 1.27 1.27)) (justify right bottom))
   )
+  (label "Col13" (at 85.09 87.376 180)
+    (effects (font (size 1.27 1.27)) (justify right bottom))
+  )
   (label "Row6" (at 253.492 83.312 180)
     (effects (font (size 1.27 1.27)) (justify right bottom))
@@
     (effects (font (size 1.27 1.27)) (justify left bottom))
   )
+  (label "Row4" (at 85.09 77.216 180)
+    (effects (font (size 1.27 1.27)) (justify right bottom))
+  )
   (symbol (lib_id "Device:D_Small") (at 51.562 157.734 0) (unit 1)

Commit message: PCB Updates
Connections:
- net Col14: now also U2.31 (GPIO20)
- net Col15: now also U2.30 (GPIO19)
- net Row1: now also U2.32 (GPIO21)
- net Row2: now also U2.34 (GPIO22)
- net Row7: now also U2.35 (GPIO23)
- net Col16: now reaches U2.29 (GPIO18)
Changed lines of the file:
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@@
+    (stroke (width 0) (type default) (color 0 0 0 0))
+  )
+  (wire (pts (xy 315.468 136.652) (xy 316.484 136.652))
     (stroke (width 0) (type default) (color 0 0 0 0))
   )
@@
     (stroke (width 0) (type default) (color 0 0 0 0))
   )
+  (wire (pts (xy 315.468 151.892) (xy 316.484 151.892))
+    (stroke (width 0) (type default) (color 0 0 0 0))
+  )
   (wire (pts (xy 331.47 37.338) (xy 334.01 37.338))
     (stroke (width 0) (type default) (color 0 0 0 0))
@@
     (stroke (width 0) (type default) (color 0 0 0 0))
   )
+  (wire (pts (xy 315.468 146.812) (xy 316.484 146.812))
+    (stroke (width 0) (type default) (color 0 0 0 0))
+  )
   (wire (pts (xy 133.35 146.05) (xy 134.366 146.05))
     (stroke (width 0) (type default) (color 0 0 0 0))
@@
     (stroke (width 0) (type default) (color 0 0 0 0))
   )
+  (wire (pts (xy 315.468 139.192) (xy 316.484 139.192))
+    (stroke (width 0) (type default) (color 0 0 0 0))
+  )
   (wire (pts (xy 25.654 148.59) (xy 28.194 148.59))
     (stroke (width 0) (type default) (color 0 0 0 0))
@@
     (stroke (width 0) (type default) (color 0 0 0 0))
   )
+  (wire (pts (xy 315.468 144.272) (xy 316.484 144.272))
+    (stroke (width 0) (type default) (color 0 0 0 0))
+  )
   (wire (pts (xy 37.084 33.02) (xy 37.084 37.338))
     (stroke (width 0) (type default) (color 0 0 0 0))
@@
   )
   (wire (pts (xy 93.726 181.102) (xy 94.742 181.102))
+    (stroke (width 0) (type default) (color 0 0 0 0))
+  )
+  (wire (pts (xy 315.468 149.352) (xy 316.484 149.352))
     (stroke (width 0) (type default) (color 0 0 0 0))
   )
@@
     (effects (font (size 1.27 1.27)) (justify right bottom))
   )
+  (label "Row7" (at 316.484 136.652 0)
+    (effects (font (size 1.27 1.27)) (justify left bottom))
+  )
   (label "QSPI_SS_56" (at 316.484 83.312 0)
     (effects (font (size 1.27 1.27)) (justify left bottom))
@@
     (effects (font (size 1.27 1.27)) (justify left bottom))
   )
+  (label "Row2" (at 316.484 139.192 0)
+    (effects (font (size 1.27 1.27)) (justify left bottom))
+  )
   (label "XIN_20" (at 253.492 129.032 180)
     (effects (font (size 1.27 1.27)) (justify right bottom))
@@
     (effects (font (size 1.27 1.27)) (justify left bottom))
   )
+  (label "Col14" (at 316.484 146.812 0)
+    (effects (font (size 1.27 1.27)) (justify left bottom))
+  )
   (label "DVDD_23" (at 253.492 136.652 180)
     (effects (font (size 1.27 1.27)) (justify right bottom))
@@
     (effects (font (size 1.27 1.27)) (justify right bottom))
   )
+  (label "Row1" (at 316.484 144.272 0)
+    (effects (font (size 1.27 1.27)) (justify left bottom))
+  )
   (label "Row5" (at 30.48 73.406 180)
     (effects (font (size 1.27 1.27)) (justify right bottom))
@@
     (effects (font (size 1.27 1.27)) (justify left bottom))
   )
+  (label "Col16" (at 316.484 151.892 0)
+    (effects (font (size 1.27 1.27)) (justify left bottom))
+  )
   (label "Col1" (at 30.48 93.726 180)
     (effects (font (size 1.27 1.27)) (justify right bottom))
@@
     (effects (font (size 1.27 1.27)) (justify right bottom))
   )
+  (label "Col15" (at 316.484 149.352 0)
+    (effects (font (size 1.27 1.27)) (justify left bottom))
+  )
   (label "XOUT_21" (at 272.542 37.084 0)

Commit message: PCB Updates
Connections:
- net Col16 is gone; now on net Col13: U2.29 (GPIO18)
- net Col14: now also U2.30 (GPIO19); no longer U2.31 (GPIO20)
- net Col15: now also U2.31 (GPIO20); no longer U2.30 (GPIO19)
Changed lines of the file:
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@@
     (effects (font (size 1.27 1.27)) (justify left bottom))
   )
-  (label "Col14" (at 316.484 146.812 0)
+  (label "Col15" (at 316.484 146.812 0)
     (effects (font (size 1.27 1.27)) (justify left bottom))
   )
@@
     (effects (font (size 1.27 1.27)) (justify left bottom))
   )
-  (label "Col16" (at 316.484 151.892 0)
+  (label "Col13" (at 316.484 151.892 0)
     (effects (font (size 1.27 1.27)) (justify left bottom))
   )
@@
     (effects (font (size 1.27 1.27)) (justify right bottom))
   )
-  (label "Col15" (at 316.484 149.352 0)
+  (label "Col14" (at 316.484 149.352 0)
     (effects (font (size 1.27 1.27)) (justify left bottom))
   )
