File: KiCAD_PCB/Calculator_PCB/Calculator_PCB.kicad_pcb (KiCad board)
At the start: 2 copper layers, 108 parts, among them J1 USB_B_Micro, SW1 SW_SPST, SW10 SW_SPST, SW11 SW_SPST, SW12 SW_SPST, SW13 SW_SPST, SW14 SW_SPST, SW15 SW_SPST, SW16 SW_SPST, SW17 SW_SPST, SW18 SW_SPST, SW19 SW_SPST, SW2 SW_SPST, SW20 SW_SPST, SW21 SW_SPST, SW22 SW_SPST, SW23 SW_SPST, SW24 SW_SPST, SW25 SW_SPST, SW26 SW_SPST, SW27 SW_SPST, SW28 SW_SPST, SW29 SW_SPST, SW3 SW_SPST, SW30 SW_SPST, SW31 SW_SPST, SW32 SW_SPST, SW33 SW_SPST, SW34 SW_SPST, SW35 SW_SPST, SW36 SW_SPST, SW37 SW_SPST, SW38 SW_SPST, SW39 SW_SPST, SW4 SW_SPST, SW40 SW_SPST, SW5 SW_SPST, SW6 SW_SPST, SW7 SW_SPST, SW8 SW_SPST, SW9 SW_SPST, U1 W25Q128JVS, U2 RP2040, U3 NCP1117-3.3_SOT223, Y1 ABLS-12.000MHZ-B4-T

Commit message: PCB Updates
Other:
- board text added: "Charging Module"
Changed lines of the file:
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@@
   )
   (gr_line (start 178.1 101.05) (end 178.1 70.55) (layer "B.SilkS") (width 0.15))
+  (gr_line (start 182.9366 63.79) (end 182.9366 106.39) (layer "B.SilkS") (width 0.15))
   (gr_line (start 272.4 55.3) (end 272.4 -4.7) (layer "B.SilkS") (width 0.15))
+  (gr_line (start 182.9366 63.79) (end 199.5366 63.79) (layer "B.SilkS") (width 0.15))
   (gr_line (start 208.2 132.5) (end 238.2 132.5) (layer "B.SilkS") (width 0.15))
   (gr_line (start 170.4 55.3) (end 170.4 -4.7) (layer "B.SilkS") (width 0.15))
@@
   (gr_line (start 112.1 101.05) (end 112.1 70.55) (layer "B.SilkS") (width 0.15))
   (gr_line (start 111.973 101.05) (end 177.973 101.05) (layer "B.SilkS") (width 0.15))
+  (gr_line (start 182.9366 106.39) (end 199.5366 106.39) (layer "B.SilkS") (width 0.15))
+  (gr_line (start 199.5366 63.79) (end 199.5366 106.39) (layer "B.SilkS") (width 0.15))
   (gr_line (start 112.1 70.55) (end 178.1 70.55) (layer "B.SilkS") (width 0.15))
   (gr_line (start 238.2 97.5) (end 238.2 132.5) (layer "B.SilkS") (width 0.15))
@@
   (gr_text "Display" (at 221.4 25.3) (layer "B.SilkS")
     (effects (font (size 6 6) (thickness 0.15)))
+  )
+  (gr_text "Charging Module" (at 191.2366 85.09 270) (layer "B.SilkS")
+    (effects (font (size 3.2 3.2) (thickness 0.15)))
   )
   (gr_text "LIPO Battery" (at 223.2 115 270) (layer "B.SilkS")
@@
       bcbfdb39-441a-41f7-a7ce-19b68bf5d022
       fd313ea1-2c0b-48ad-82be-b04c1bef9db0
+    )
+  )
+  (group "" (id 1b350c19-993f-4432-86a1-4122e950bd0b)
+    (members
+      0f16f15c-d889-430d-bdc7-8ae1f82b9520
+      2ce839a7-ae56-4836-a547-aefa450214ac
+      8cbbddaa-560a-4858-a57e-0d4d594fb21f
+      9b65c9d0-858c-4826-94e3-1e53a6bb86da
     )
   )
@@
     )
   )
+  (group "" (id e721cb39-0cb3-4c17-a648-5ba6edd83876)
+    (members
+      1b350c19-993f-4432-86a1-4122e950bd0b
+      ec9041c6-6700-4963-9711-2f33daa5cfd3
+    )
+  )

Commit message: Update PCB
Parts:
- D2, D6: moved to B.Cu
- moved D2 175.3 mm to (90.1, 124.0)
- moved D6 140.0 mm to (102.0, 124.0)

Commit message: PCB Updates
Parts:
- D10, D14, D18, D22, D26, D30: moved to B.Cu
- moved D26 182.1 mm to (161.5, 124.0)
- moved D30 171.8 mm to (173.4, 124.0)
- moved D18 163.7 mm to (137.7, 124.0)
- moved D22 157.2 mm to (149.6, 124.0)
- moved D10 153.8 mm to (113.9, 124.0)
- moved D14 143.1 mm to (125.8, 124.0)

Commit message: PCB Updates
Parts:
- D11, D12, D15, D16, D19, D20, D23, D24, D27, D28, D3, D31, D32, D34, D35, D36, D38, D39, D4, D40, D7, D8: moved to B.Cu
- moved D40 218.0 mm to (197.2, 140.0)
- moved D19 217.9 mm to (137.7, 132.0)
- moved D39 210.8 mm to (197.2, 132.0)
- moved D7 204.8 mm to (102.0, 132.0)
- moved D36 204.4 mm to (185.3, 140.0)
- moved D38 203.8 mm to (197.2, 124.0)
- moved D32 201.6 mm to (173.4, 140.0)
- moved D34 201.5 mm to (185.3, 124.0)
- moved D27 189.4 mm to (161.5, 132.0)
- moved D15 186.5 mm to (125.8, 132.0)
- moved D4 184.5 mm to (90.1, 140.0)
- moved D23 182.5 mm to (149.6, 132.0)
- moved D28 182.1 mm to (161.5, 140.0)
- moved D24 181.3 mm to (149.6, 140.0)
- moved D12 180.6 mm to (113.9, 140.0)
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
Commit message: PCB Updates
Routing:
- net /Row0: track 17.6 -> 127.3 mm
- net Net-(D29-Pad2): track 0.00 -> 3.55 mm
- net Net-(D9-Pad2): track 0.00 -> 3.55 mm
- net Net-(D37-Pad2): track 0.00 -> 3.55 mm
- net Net-(D33-Pad2): track 0.00 -> 3.55 mm
- net Net-(D21-Pad2): track 0.00 -> 3.55 mm
- net Net-(D17-Pad2): track 0.00 -> 3.55 mm
- net Net-(D13-Pad2): track 0.00 -> 3.55 mm
- net Net-(D2-Pad2): track 0.00 -> 3.55 mm
- net Net-(D5-Pad2): track 0.00 -> 3.55 mm
- net Net-(D25-Pad2): track 0.00 -> 3.55 mm

Commit message: PCB Updates
Routing:
- net /Row3: track 0.00 -> 123.4 mm
- net /Row1: track 0.00 -> 123.4 mm
- net /Row2: track 0.00 -> 123.4 mm
- net Net-(D15-Pad2): track 0.00 -> 3.55 mm
- net Net-(D7-Pad2): track 0.00 -> 3.55 mm
- net Net-(D39-Pad2): track 0.00 -> 3.55 mm
- net Net-(D35-Pad2): track 0.00 -> 3.55 mm
- net Net-(D31-Pad2): track 0.00 -> 3.55 mm
- net Net-(D3-Pad2): track 0.00 -> 3.55 mm
- net Net-(D23-Pad2): track 0.00 -> 3.55 mm
- net Net-(D19-Pad2): track 0.00 -> 3.55 mm
- net Net-(D11-Pad2): track 0.00 -> 3.55 mm
- net Net-(D10-Pad2): track 0.00 -> 3.55 mm
- net Net-(D6-Pad2): track 0.00 -> 3.55 mm
- net Net-(D38-Pad2): track 0.00 -> 3.55 mm
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
Commit message: PCB Updates
Routing:
- net /Col0: track 0.00 -> 31.9 mm
- net /Col2: track 0.00 -> 31.8 mm
- net /Col1: track 0.00 -> 31.8 mm
- net /Col3: track 0.00 -> 31.8 mm

Commit message: PCB Updates
Parts:
- moved J1 129.9 mm to (97.3, 80.0)
Routing:
- net /Col4: track 0.00 -> 31.8 mm
- net /Col9: track 0.00 -> 31.8 mm
- net /Col5: track 0.00 -> 31.8 mm
- net /Col6: track 0.00 -> 31.8 mm
- net /Col7: track 0.00 -> 31.8 mm
- net /Col8: track 0.00 -> 31.8 mm
