File: KiCAD_PCB/Calculator_PCB/Calculator_PCB.kicad_pcb (KiCad board)
At the start: 2 copper layers, 109 parts, among them J1 USB_B_Micro, SW1 SW_SPST, SW10 SW_SPST, SW11 SW_SPST, SW12 SW_SPST, SW13 SW_SPST, SW14 SW_SPST, SW15 SW_SPST, SW16 SW_SPST, SW17 SW_SPST, SW18 SW_SPST, SW19 SW_SPST, SW2 SW_SPST, SW20 SW_SPST, SW21 SW_SPST, SW22 SW_SPST, SW23 SW_SPST, SW24 SW_SPST, SW25 SW_SPST, SW26 SW_SPST, SW27 SW_SPST, SW28 SW_SPST, SW29 SW_SPST, SW3 SW_SPST, SW30 SW_SPST, SW31 SW_SPST, SW32 SW_SPST, SW33 SW_SPST, SW34 SW_SPST, SW35 SW_SPST, SW36 SW_SPST, SW37 SW_SPST, SW38 SW_SPST, SW39 SW_SPST, SW4 SW_SPST, SW40 SW_SPST, SW5 SW_SPST, SW6 SW_SPST, SW7 SW_SPST, SW8 SW_SPST, SW9 SW_SPST, U1 W25Q128JVS, U2 RP2040, U3 NCP1117-3.3_SOT223, X1 JTAG-CORTEX, Y1 ABLS-12.000MHZ-B4-T

Commit message: PCB Updates
Routing:
- net /Col5: track 37.3 -> 80.7 mm, vias 0 -> 2
- net /Col4: track 37.3 -> 77.9 mm, vias 0 -> 2
- net /Col6: track 37.2 -> 63.8 mm, vias 0 -> 2
- net /Col3: track 37.3 -> 61.0 mm
- net /Col7: track 36.5 -> 46.5 mm
- net /Col12: track 32.6 -> 42.5 mm
- net /Col11: track 32.5 -> 42.4 mm
- net /Col9: track 36.2 -> 46.2 mm
- net /Col10: track 36.0 -> 45.9 mm
- net /Col8: track 36.6 -> 46.5 mm

Commit message: PCB Updates
Routing:
- net /Col5: track 80.7 -> 63.8 mm, vias 2 -> 0
- net /Col6: track 63.8 -> 47.2 mm, vias 2 -> 0
- net /Col4: track 77.9 -> 62.9 mm, vias 2 -> 0
- net /Col3: track 61.0 -> 50.7 mm
Changed lines of the file:
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@@
   (segment (start 95.31 133.46) (end 95.504 133.654) (width 0.15) (layer "F.Cu") (net 56))
   (segment (start 95.504 117.475) (end 95.504 117.216) (width 0.15) (layer "F.Cu") (net 56))
-  (segment (start 92.74 126.63) (end 92.68 126.63) (width 0.15) (layer "F.Cu") (net 56))
   (segment (start 95.504 109.728) (end 95.236 109.46) (width 0.15) (layer "F.Cu") (net 56))
   (segment (start 95.504 125.4252) (end 95.504 125.216) (width 0.15) (layer "F.Cu") (net 56))
@@
   (segment (start 95.504 117.856) (end 95.504 117.7544) (width 0.15) (layer "F.Cu") (net 56))
   (segment (start 95.504 125.216) (end 95.504 125.095) (width 0.15) (layer "F.Cu") (net 56))
-  (segment (start 93.91 125.46) (end 92.74 126.63) (width 0.15) (layer "F.Cu") (net 56))
   (segment (start 95.504 117.094) (end 95.504 109.728) (width 0.15) (layer "F.Cu") (net 56))
   (segment (start 95.48 133.46) (end 95.504 133.436) (width 0.15) (layer "F.Cu") (net 56))
@@
   (segment (start 95.504 133.256) (end 95.504 133.186) (width 0.15) (layer "F.Cu") (net 56))
   (segment (start 95.3 133.46) (end 95.48 133.46) (width 0.15) (layer "F.Cu") (net 56))
-  (segment (start 92.68 126.63) (end 84.16 126.63) (width 0.15) (layer "F.Cu") (net 56))
   (segment (start 93.91 125.46) (end 95.1898 125.46) (width 0.15) (layer "F.Cu") (net 56))
   (segment (start 95.1634 117.46) (end 95.489 117.46) (width 0.15) (layer "F.Cu") (net 56))
@@
   (segment (start 107.404 109.728) (end 107.136 109.46) (width 0.15) (layer "F.Cu") (net 59))
   (segment (start 107.404 117.706) (end 107.404 117.475) (width 0.15) (layer "F.Cu") (net 59))
-  (segment (start 91.41048 127.01952) (end 92.54 127.01952) (width 0.15) (layer "F.Cu") (net 59))
   (segment (start 107.16 117.46) (end 107.16 117.462) (width 0.15) (layer "F.Cu") (net 59))
   (segment (start 107.404 140.996) (end 106.06 142.34) (width 0.15) (layer "F.Cu") (net 59))
@@
   (segment (start 107.18 133.46) (end 107.18 133.43) (width 0.15) (layer "F.Cu") (net 59))
   (segment (start 107.0634 117.46) (end 107.389 117.46) (width 0.15) (layer "F.Cu") (net 59))
-  (segment (start 97.26 127.02) (end 104.25 127.02) (width 0.15) (layer "F.Cu") (net 59))
-  (segment (start 94.84952 127.01952) (end 94.85 127.02) (width 0.15) (layer "F.Cu") (net 59))
   (segment (start 107.188 125.46) (end 107.404 125.676) (width 0.15) (layer "F.Cu") (net 59))
   (segment (start 107.18 133.43) (end 107.404 133.206) (width 0.15) (layer "F.Cu") (net 59))
   (segment (start 107.38 133.46) (end 107.404 133.484) (width 0.15) (layer "F.Cu") (net 59))
   (segment (start 107.404 117.856) (end 107.404 117.7544) (width 0.15) (layer "F.Cu") (net 59))
-  (segment (start 92.54 127.01952) (end 94.84952 127.01952) (width 0.15) (layer "F.Cu") (net 59))
   (segment (start 107.404 125.676) (end 107.404 125.4252) (width 0.15) (layer "F.Cu") (net 59))
   (segment (start 107.404 125.216) (end 107.404 125.095) (width 0.15) (layer "F.Cu") (net 59))
   (segment (start 107.404 133.096) (end 107.404 125.7554) (width 0.15) (layer "F.Cu") (net 59))
   (segment (start 107.404 133.096) (end 107.404 133.206) (width 0.15) (layer "F.Cu") (net 59))
-  (segment (start 104.25 127.02) (end 105.81 125.46) (width 0.15) (layer "F.Cu") (net 59))
   (segment (start 107.0898 125.46) (end 107.3692 125.46) (width 0.15) (layer "F.Cu") (net 59))
   (segment (start 91.01048 142.33952) (end 93.83 142.33952) (width 0.15) (layer "F.Cu") (net 59))
@@
   (segment (start 106.03952 142.33952) (end 106.04 142.34) (width 0.15) (layer "F.Cu") (net 59))
   (segment (start 107.3692 125.46) (end 107.404 125.4252) (width 0.15) (layer "F.Cu") (net 59))
-  (via (at 94.85 127.02) (size 0.6) (drill 0.35) (layers "F.Cu" "B.Cu") (free) (net 59))
-  (via (at 97.26 127.02) (size 0.6) (drill 0.35) (layers "F.Cu" "B.Cu") (free) (net 59))
-  (segment (start 94.85 127.02) (end 97.26 127.02) (width 0.15) (layer "B.Cu") (net 59))
   (segment (start 115.8136 122.541) (end 115.5446 122.81) (width 0.15) (layer "B.Cu") (net 60))
   (segment (start 117.787 122.541) (end 115.8136 122.541) (width 0.15) (layer "B.Cu") (net 60))
@@
   (segment (start 93.2825 89.7425) (end 87.5675 89.7425) (width 0.15) (layer "F.Cu") (net 71))
   (segment (start 117.958 142.732) (end 102.40296 142.732) (width 0.15) (layer "F.Cu") (net 71))
-  (segment (start 115.76 127.41) (end 117.71 125.46) (width 0.15) (layer "F.Cu") (net 71))
   (segment (start 117.71 133.46) (end 119.04 133.46) (width 0.15) (layer "F.Cu") (net 71))
   (segment (start 119.304 133.096) (end 119.304 133.246) (width 0.15) (layer "F.Cu") (net 71))
@@
   (segment (start 119.304 117.7544) (end 119.304 117.706) (width 0.15) (layer "F.Cu") (net 71))
   (segment (start 119.304 133.416) (end 119.304 133.664) (width 0.15) (layer "F.Cu") (net 71))
-  (segment (start 103.92 127.40952) (end 106.72952 127.40952) (width 0.15) (layer "F.Cu") (net 71))
   (segment (start 119.06 125.46) (end 119.088 125.46) (width 0.15) (layer "F.Cu") (net 71))
   (segment (start 119.304 133.246) (end 119.304 133.416) (width 0.15) (layer "F.Cu") (net 71))
@@
   (segment (start 119.04 133.46) (end 119.09 133.46) (width 0.15) (layer "F.Cu") (net 71))
   (segment (start 119.302 141.388) (end 117.958 142.732) (width 0.15) (layer "F.Cu") (net 71))
-  (segment (start 109.15 127.41) (end 115.76 127.41) (width 0.15) (layer "F.Cu") (net 71))
   (segment (start 119.26 133.46) (end 119.304 133.416) (width 0.15) (layer "F.Cu") (net 71))
   (segment (start 119.302 141.388) (end 119.302 133.418) (width 0.15) (layer "F.Cu") (net 71))
-  (segment (start 101.60048 127.40952) (end 103.92 127.40952) (width 0.15) (layer "F.Cu") (net 71))
-  (segment (start 106.72952 127.40952) (end 106.73 127.41) (width 0.15) (layer "F.Cu") (net 71))
   (segment (start 117.71 125.46) (end 118.9898 125.46) (width 0.15) (layer "F.Cu") (net 71))
   (segment (start 119.304 117.856) (end 119.304 117.7544) (width 0.15) (layer "F.Cu") (net 71))
-  (via (at 109.15 127.41) (size 0.6) (drill 0.35) (layers "F.Cu" "B.Cu") (free) (net 71))
-  (via (at 106.73 127.41) (size 0.6) (drill 0.35) (layers "F.Cu" "B.Cu") (net 71))
-  (segment (start 106.73 127.41) (end 109.15 127.41) (width 0.15) (layer "B.Cu") (net 71))
   (segment (start 153.4994 122.541) (end 151.526 122.541) (width 0.15) (layer "B.Cu") (net 72))
   (segment (start 151.257 122.81) (end 151.257 124.0028) (width 0.15) (layer "B.Cu") (net 72))
@@
   (segment (start 131.204 133.096) (end 131.204 133.246) (width 0.15) (layer "F.Cu") (net 76))
   (segment (start 131.204 125.676) (end 131.204 125.4252) (width 0.15) (layer "F.Cu") (net 76))
-  (segment (start 113.92048 127.79952) (end 115.64 127.79952) (width 0.15) (layer "F.Cu") (net 76))
   (segment (start 131.16 133.46) (end 131.204 133.416) (width 0.15) (layer "F.Cu") (net 76))
   (segment (start 129.61 117.46) (end 130.8634 117.46) (width 0.15) (layer "F.Cu") (net 76))
@@
   (segment (start 130.96 117.46) (end 130.96 117.462) (width 0.15) (layer "F.Cu") (net 76))
   (segment (start 131.204 117.706) (end 131.204 117.475) (width 0.15) (layer "F.Cu") (net 76))
-  (segment (start 121.05 127.8) (end 127.27 127.8) (width 0.15) (layer "F.Cu") (net 76))
   (segment (start 131.204 133.096) (end 131.204 125.7554) (width 0.15) (layer "F.Cu") (net 76))
   (segment (start 131.204 125.7554) (end 131.204 125.676) (width 0.15) (layer "F.Cu") (net 76))
-  (segment (start 118.64952 127.79952) (end 118.65 127.8) (width 0.15) (layer "F.Cu") (net 76))
   (segment (start 131.204 117.216) (end 131.204 117.094) (width 0.15) (layer "F.Cu") (net 76))
   (segment (start 130.94 133.46) (end 131.16 133.46) (width 0.15) (layer "F.Cu") (net 76))
-  (segment (start 115.64 127.79952) (end 118.64952 127.79952) (width 0.15) (layer "F.Cu") (net 76))
   (segment (start 131.204 125.095) (end 131.204 117.856) (width 0.15) (layer "F.Cu") (net 76))
-  (segment (start 127.27 127.8) (end 129.61 125.46) (width 0.15) (layer "F.Cu") (net 76))
   (segment (start 130.99 133.46) (end 131 133.46) (width 0.15) (layer "F.Cu") (net 76))
   (segment (start 87.6325 90.1425) (end 87.63 90.14) (width 0.15) (layer "F.Cu") (net 76))
@@
   (segment (start 131.204 117.094) (end 131.204 109.728) (width 0.15) (layer "F.Cu") (net 76))
   (segment (start 130.8634 117.46) (end 131.189 117.46) (width 0.15) (layer "F.Cu") (net 76))
-  (via (at 121.05 127.8) (size 0.6) (drill 0.35) (layers "F.Cu" "B.Cu") (net 76))
-  (via (at 118.65 127.8) (size 0.6) (drill 0.35) (layers "F.Cu" "B.Cu") (net 76))
-  (segment (start 118.65 127.8) (end 121.05 127.8) (width 0.15) (layer "B.Cu") (net 76))
   (segment (start 163.4132 122.541) (end 163.1442 122.81) (width 0.15) (layer "B.Cu") (net 77))
   (segment (start 163.1442 122.81) (end 163.1442 124.0028) (width 0.15) (layer "B.Cu") (net 77))

Commit message: PCB Update
Routing:
- net /Col12: track 42.5 -> 159.6 mm
- net /Col11: track 42.4 -> 147.8 mm
- net /Col10: track 45.9 -> 139.5 mm
- net /Col9: track 46.2 -> 127.9 mm
- net /Col8: track 46.5 -> 116.3 mm
- net /Col7: track 46.5 -> 102.2 mm
- net /Col6: track 47.2 -> 91.0 mm
- net /Col5: track 63.8 -> 95.6 mm
- net /Col4: track 62.9 -> 82.8 mm
- net /Col3: track 50.7 -> 59.1 mm
Changed lines of the file:
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@@
   (segment (start 91.706296 92.676296) (end 91.464032 92.91856) (width 0.15) (layer "F.Cu") (net 14))
   (segment (start 178.804 133.664) (end 178.804 142.516) (width 0.15) (layer "F.Cu") (net 14))
+  (segment (start 147.14096 135.58904) (end 84.52 135.58904) (width 0.15) (layer "B.Cu") (net 14))
+  (segment (start 147.14096 135.58904) (end 175.08096 135.58904) (width 0.15) (layer "B.Cu") (net 14))
+  (segment (start 175.08096 135.58904) (end 177.21 133.46) (width 0.15) (layer "B.Cu") (net 14))
   (segment (start 190.704 133.664) (end 190.704 142.516) (width 0.15) (layer "F.Cu") (net 15))
   (segment (start 190.66 133.46) (end 190.704 133.416) (width 0.15) (layer "F.Cu") (net 15))
@@
   (segment (start 190.6692 125.46) (end 190.704 125.4252) (width 0.15) (layer "F.Cu") (net 15))
   (segment (start 189.11 125.46) (end 190.3898 125.46) (width 0.15) (layer "F.Cu") (net 15))
+  (segment (start 147.63144 135.97856) (end 84.83 135.97856) (width 0.15) (layer "B.Cu") (net 15))
+  (segment (start 147.63144 135.97856) (end 186.59144 135.97856) (width 0.15) (layer "B.Cu") (net 15))
+  (segment (start 186.59144 135.97856) (end 189.11 133.46) (width 0.15) (layer "B.Cu") (net 15))
   (segment (start 201.01 133.46) (end 202.34 133.46) (width 0.15) (layer "F.Cu") (net 16))
   (segment (start 202.336 109.46) (end 201.01 109.46) (width 0.15) (layer "F.Cu") (net 16))
@@
   (segment (start 202.36 125.46) (end 202.604 125.216) (width 0.15) (layer "F.Cu") (net 16))
   (segment (start 202.5692 125.46) (end 202.604 125.4252) (width 0.15) (layer "F.Cu") (net 16))
+  (segment (start 148.01192 136.36808) (end 85.22 136.36808) (width 0.15) (layer "B.Cu") (net 16))
+  (segment (start 85.22 136.36808) (end 85.13 136.36808) (width 0.15) (layer "B.Cu") (net 16))
+  (segment (start 198.10192 136.36808) (end 201.01 133.46) (width 0.15) (layer "B.Cu") (net 16))
+  (segment (start 148.01192 136.36808) (end 198.10192 136.36808) (width 0.15) (layer "B.Cu") (net 16))
   (segment (start 94.92 92.98) (end 94.92 94.12) (width 0.15) (layer "F.Cu") (net 22))
   (segment (start 95.32 92.98) (end 95.32 94.19) (width 0.15) (layer "F.Cu") (net 23))
@@
   (segment (start 95.504 140.606) (end 94.16 141.95) (width 0.15) (layer "F.Cu") (net 56))
   (segment (start 95.3 133.46) (end 95.504 133.256) (width 0.15) (layer "F.Cu") (net 56))
+  (segment (start 93.91 125.46) (end 92.55 126.82) (width 0.15) (layer "B.Cu") (net 56))
+  (segment (start 92.55 126.82) (end 86.11 126.82) (width 0.15) (layer "B.Cu") (net 56))
   (segment (start 141.5868 122.541) (end 139.6134 122.541) (width 0.15) (layer "B.Cu") (net 58))
   (segment (start 139.6134 122.541) (end 139.3444 122.81) (width 0.15) (layer "B.Cu") (net 58))
@@
   (segment (start 106.03952 142.33952) (end 106.04 142.34) (width 0.15) (layer "F.Cu") (net 59))
   (segment (start 107.3692 125.46) (end 107.404 125.4252) (width 0.15) (layer "F.Cu") (net 59))
+  (segment (start 86.60048 127.20952) (end 104.06048 127.20952) (width 0.15) (layer "B.Cu") (net 59))
+  (segment (start 104.06048 127.20952) (end 105.81 125.46) (width 0.15) (layer "B.Cu") (net 59))
   (segment (start 115.8136 122.541) (end 115.5446 122.81) (width 0.15) (layer "B.Cu") (net 60))
   (segment (start 117.787 122.541) (end 115.8136 122.541) (width 0.15) (layer "B.Cu") (net 60))
@@
   (segment (start 117.71 125.46) (end 118.9898 125.46) (width 0.15) (layer "F.Cu") (net 71))
   (segment (start 119.304 117.856) (end 119.304 117.7544) (width 0.15) (layer "F.Cu") (net 71))
+  (segment (start 115.57096 127.59904) (end 117.71 125.46) (width 0.15) (layer "B.Cu") (net 71))
+  (segment (start 86.76096 127.59904) (end 115.57096 127.59904) (width 0.15) (layer "B.Cu") (net 71))
   (segment (start 153.4994 122.541) (end 151.526 122.541) (width 0.15) (layer "B.Cu") (net 72))
   (segment (start 151.257 122.81) (end 151.257 124.0028) (width 0.15) (layer "B.Cu") (net 72))
@@
   (segment (start 131.204 117.094) (end 131.204 109.728) (width 0.15) (layer "F.Cu") (net 76))
   (segment (start 130.8634 117.46) (end 131.189 117.46) (width 0.15) (layer "F.Cu") (net 76))
+  (segment (start 87.72856 127.98856) (end 87.73 127.99) (width 0.15) (layer "B.Cu") (net 76))
+  (segment (start 87.73 127.99) (end 127.08 127.99) (width 0.15) (layer "B.Cu") (net 76))
+  (segment (start 86.85144 127.98856) (end 87.72856 127.98856) (width 0.15) (layer "B.Cu") (net 76))
+  (segment (start 127.08 127.99) (end 129.61 125.46) (width 0.15) (layer "B.Cu") (net 76))
   (segment (start 163.4132 122.541) (end 163.1442 122.81) (width 0.15) (layer "B.Cu") (net 77))
   (segment (start 163.1442 122.81) (end 163.1442 124.0028) (width 0.15) (layer "B.Cu") (net 77))
@@
   (segment (start 143.104 142.516) (end 143.1 142.52) (width 0.15) (layer "F.Cu") (net 81))
   (segment (start 143.104 133.096) (end 143.104 133.246) (width 0.15) (layer "F.Cu") (net 81))
+  (segment (start 91.13 128.37952) (end 138.59048 128.37952) (width 0.15) (layer "B.Cu") (net 81))
+  (segment (start 138.59048 128.37952) (end 141.51 125.46) (width 0.15) (layer "B.Cu") (net 81))
+  (segment (start 86.94048 128.37952) (end 91.13 128.37952) (width 0.15) (layer "B.Cu") (net 81))
   (segment (start 175.3004 122.541) (end 175.0314 122.81) (width 0.15) (layer "B.Cu") (net 82))
   (segment (start 175.0314 122.81) (end 175.0314 124.0028) (width 0.15) (layer "B.Cu") (net 82))
@@
   (segment (start 154.8 133.46) (end 155.004 133.664) (width 0.15) (layer "F.Cu") (net 85))
   (segment (start 155.004 142.516) (end 155 142.52) (width 0.15) (layer "F.Cu") (net 85))
+  (segment (start 145.68 134.81) (end 84.18 134.81) (width 0.15) (layer "B.Cu") (net 85))
+  (segment (start 152.06 134.81) (end 145.68 134.81) (width 0.15) (layer "B.Cu") (net 85))
+  (segment (start 153.41 133.46) (end 152.06 134.81) (width 0.15) (layer "B.Cu") (net 85))
   (segment (start 186.944 122.81) (end 186.944 124.0028) (width 0.15) (layer "B.Cu") (net 86))
   (segment (start 187.213 122.541) (end 186.944 122.81) (width 0.15) (layer "B.Cu") (net 86))
@@
   (segment (start 166.889 117.46) (end 166.904 117.475) (width 0.15) (layer "F.Cu") (net 90))
   (segment (start 166.69 133.46) (end 166.7 133.46) (width 0.15) (layer "F.Cu") (net 90))
+  (segment (start 146.43048 135.19952) (end 84.33 135.19952) (width 0.15) (layer "B.Cu") (net 90))
+  (segment (start 146.43048 135.19952) (end 163.57048 135.19952) (width 0.15) (layer "B.Cu") (net 90))
+  (segment (start 163.57048 135.19952) (end 165.31 133.46) (width 0.15) (layer "B.Cu") (net 90))
   (segment (start 201.0736 122.541) (end 199.1002 122.541) (width 0.15) (layer "B.Cu") (net 91))
   (segment (start 199.1002 122.541) (end 198.8312 122.81) (width 0.15) (layer "B.Cu") (net 91))

Commit message: PCB Updates
Routing:
- net /Col12: track 159.6 -> 172.3 mm
- net /Col11: track 147.8 -> 160.1 mm
- net /Col10: track 139.5 -> 151.3 mm
- net /Col9: track 127.9 -> 139.2 mm
- net /Col8: track 116.3 -> 127.5 mm
- net /Col5: track 95.6 -> 104.6 mm
- net /Col7: track 102.2 -> 109.9 mm
- net /Col6: track 91.0 -> 97.8 mm
- net /Col4: track 82.8 -> 89.2 mm
- net /Col3: track 59.1 -> 64.5 mm

Commit message: PCB Updates
Routing:
- net /Col6: track 97.8 -> 112.4 mm, vias 0 -> 1
- net /Col4: track 89.2 -> 103.4 mm, vias 0 -> 1
- net /Col3: track 64.5 -> 78.6 mm, vias 0 -> 1
- net /Col7: track 109.9 -> 123.8 mm, vias 0 -> 1
- net /Col11: track 160.1 -> 146.5 mm, vias 0 -> 1
- net /Col10: track 151.3 -> 137.9 mm, vias 0 -> 1
- net /Col9: track 139.2 -> 126.2 mm, vias 0 -> 1
- net /Col8: track 127.5 -> 114.5 mm, vias 0 -> 1
- net /Col12: track 172.3 -> 159.5 mm, vias 0 -> 1
- net /Col5: track 104.6 -> 116.7 mm, vias 0 -> 1

Commit message: PCB Updates
Routing:
- net /Col11: track 146.5 -> 172.9 mm
- net /Col12: track 159.5 -> 185.6 mm
- net /Col10: track 137.9 -> 163.8 mm
- net /Col9: track 126.2 -> 151.5 mm
- net /Col8: track 114.5 -> 139.6 mm

Commit message: PCB Updates
Routing:
- net /Col5: track 116.7 -> 90.3 mm
- net /Col4: track 103.4 -> 77.9 mm
- net /Col3: track 78.6 -> 65.3 mm
- net /Col8: track 139.6 -> 129.8 mm
- net /Col6: track 112.4 -> 102.6 mm
- net /Col12: track 185.6 -> 175.7 mm
- net /Col11: track 172.9 -> 163.1 mm
- net /Col10: track 163.8 -> 154.0 mm
- net /Col7: track 123.8 -> 114.0 mm
- net /Col9: track 151.5 -> 141.7 mm

Commit message: PCB Updates
Parts:
- moved X1 1.14 mm to (76.3, 91.4)
Routing:
- net /Col10: track 154.0 -> 169.9 mm
- net /Col9: track 141.7 -> 157.5 mm
- net /Col11: track 163.1 -> 178.8 mm
- net /Col12: track 175.7 -> 191.3 mm
- net /Col8: track 129.8 -> 145.3 mm
- net /Col7: track 114.0 -> 129.2 mm
- net /Col6: track 102.6 -> 117.3 mm
- net /Col5: track 90.3 -> 104.8 mm
- net /Col4: track 77.9 -> 92.3 mm
- net /Col3: track 65.3 -> 79.6 mm
- net /Row2: track 133.1 -> 136.8 mm, vias 0 -> 1
