File: KiCAD_PCB/Calculator_PCB/Calculator_PCB.kicad_pcb (KiCad board)
At the start: 2 copper layers, 132 x 78 mm, 110 parts, among them J1 USB_B_Micro, J2 5034801000, J3 5034801000, SW1 SW_SPST, SW10 SW_SPST, SW11 SW_SPST, SW12 SW_SPST, SW13 SW_SPST, SW14 SW_SPST, SW15 SW_SPST, SW16 SW_SPST, SW17 SW_SPST, SW18 SW_SPST, SW19 SW_SPST, SW2 SW_SPST, SW20 SW_SPST, SW21 SW_SPST, SW22 SW_SPST, SW23 SW_SPST, SW24 SW_SPST, SW25 SW_SPST, SW26 SW_SPST, SW27 SW_SPST, SW28 SW_SPST, SW29 SW_SPST, SW3 SW_SPST, SW30 SW_SPST, SW31 SW_SPST, SW32 SW_SPST, SW33 SW_SPST, SW34 SW_SPST, SW35 SW_SPST, SW36 SW_SPST, SW37 SW_SPST, SW38 SW_SPST, SW39 SW_SPST, SW4 SW_SPST, SW40 SW_SPST, SW5 SW_SPST, SW6 SW_SPST, SW7 SW_SPST, SW8 SW_SPST, SW9 SW_SPST, U1 W25Q128JVS, U2 RP2040, U3 NCP1117-3.3_SOT223, Y1 ABLS-12.000MHZ-B4-T

Commit message: PCB updates
Routing:
- net /x_out: track 40.0 -> 69.1 mm, vias 1 -> 4
- net /y_out: track 38.2 -> 64.9 mm, vias 1 -> 4
- net /Col2: track 32.4 -> 57.9 mm, vias 1 -> 2

Commit message: PCB Updates
Parts:
- moved C14 0.45 mm to (106.1, 81.8)
- moved C13 0.45 mm to (104.9, 69.3)
- moved U3 0.45 mm to (105.0, 75.6)
Changed lines of the file:
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@@
   )
   (footprint "Capacitor_SMD:C_0805_2012Metric_Pad1.18x1.45mm_HandSolder" (layer "F.Cu")
-    (at 105.32 69.32)
+    (at 104.87 69.31)
     (descr "Capacitor SMD 0805 (2012 Metric), square (rectangular) end terminal, IPC_7351 nominal with elongated pad for handsoldering. (Body size source: IPC-SM-782 page 76, https://www.pcb-3d.com/wordpress/wp-content/uploads/ipc-sm-782a_amendment_1_and_2.pdf, https://docs.google.com/spreadsheets/d/1BsfQQcO9C6DZCsRaXUlFlo91Tg2WpOkGARC1WS5S8t0/edit?usp=sharing), generated with kicad-footprint-generator")
     (tags "capacitor handsolder")
@@
   )
   (footprint "Capacitor_SMD:C_0805_2012Metric_Pad1.18x1.45mm_HandSolder" (layer "F.Cu")
-    (at 106.55 81.84)
+    (at 106.1 81.83)
     (descr "Capacitor SMD 0805 (2012 Metric), square (rectangular) end terminal, IPC_7351 nominal with elongated pad for handsoldering. (Body size source: IPC-SM-782 page 76, https://www.pcb-3d.com/wordpress/wp-content/uploads/ipc-sm-782a_amendment_1_and_2.pdf, https://docs.google.com/spreadsheets/d/1BsfQQcO9C6DZCsRaXUlFlo91Tg2WpOkGARC1WS5S8t0/edit?usp=sharing), generated with kicad-footprint-generator")
     (tags "capacitor handsolder")
@@
   )
   (footprint "Package_TO_SOT_SMD:SOT-223-3_TabPin2" (layer "F.Cu")
-    (at 105.49 75.6 -90)
+    (at 105.04 75.59 -90)
     (descr "module CMS SOT223 4 pins")
     (tags "CMS SOT")
@@
   (segment (start 95.515 66.525) (end 95.785 66.255) (width 0.2) (layer "F.Cu") (net 11))
   (segment (start 97.975 66.525) (end 97.705 66.255) (width 0.2) (layer "F.Cu") (net 11))
-  (segment (start 106.3575 69.32) (end 106.63 69.32) (width 0.2) (layer "F.Cu") (net 11))
-  (segment (start 107.5875 81.84) (end 109.12 81.84) (width 0.2) (layer "F.Cu") (net 11))
+  (segment (start 105.9075 69.31) (end 106.18 69.31) (width 0.2) (layer "F.Cu") (net 11))
+  (segment (start 107.1375 81.83) (end 108.67 81.83) (width 0.2) (layer "F.Cu") (net 11))
   (segment (start 97.005 99.21) (end 98.04 99.21) (width 0.2) (layer "F.Cu") (net 11))
-  (segment (start 106.63 69.32) (end 107.465 70.155) (width 0.2) (layer "F.Cu") (net 11))
-  (segment (start 107.465 70.155) (end 107.66 70.35) (width 0.2) (layer "F.Cu") (net 11))
+  (segment (start 106.18 69.31) (end 107.015 70.145) (width 0.2) (layer "F.Cu") (net 11))
+  (segment (start 107.015 70.145) (end 107.21 70.34) (width 0.2) (layer "F.Cu") (net 11))
   (segment (start 89.4 90.8075) (end 88.365 90.8075) (width 0.2) (layer "F.Cu") (net 11))
   (segment (start 99.76 82.19) (end 99.76 81.155) (width 0.2) (layer "F.Cu") (net 11))
   (segment (start 92.58 99.21) (end 91.545 99.21) (width 0.2) (layer "F.Cu") (net 11))
-  (segment (start 107.66 70.35) (end 107.79 70.48) (width 0.2) (layer "F.Cu") (net 11))
+  (segment (start 107.21 70.34) (end 107.34 70.47) (width 0.2) (layer "F.Cu") (net 11))
   (segment (start 95.72 92.98) (end 95.72 94.52) (width 0.2) (layer "F.Cu") (net 11))
   (segment (start 88.74 73.18) (end 88.74 74.215) (width 0.2) (layer "F.Cu") (net 11))
@@
   (segment (start 94.015 66.525) (end 95.515 66.525) (width 0.2) (layer "F.Cu") (net 11))
   (segment (start 95.45 69.41) (end 95.45 70.9425) (width 0.2) (layer "F.Cu") (net 11))
-  (segment (start 107.79 70.48) (end 107.79 72.45) (width 0.2) (layer "F.Cu") (net 11))
+  (segment (start 107.34 70.47) (end 107.34 72.44) (width 0.2) (layer "F.Cu") (net 11))
   (segment (start 104.03 90.81) (end 105.065 90.81) (width 0.2) (layer "F.Cu") (net 11))
   (segment (start 97.19 96.85) (end 97.19 97.885) (width 0.2) (layer "F.Cu") (net 11))
@@
   (via (at 105.055 85.57) (size 0.6) (drill 0.35) (layers "F.Cu" "B.Cu") (net 11))
   (via (at 105.065 83.91) (size 0.6) (drill 0.35) (layers "F.Cu" "B.Cu") (net 11))
-  (via (at 109.12 81.84) (size 0.6) (drill 0.35) (layers "F.Cu" "B.Cu") (net 11))
+  (via (at 108.67 81.83) (size 0.6) (drill 0.35) (layers "F.Cu" "B.Cu") (net 11))
   (via (at 97.19 97.885) (size 0.6) (drill 0.35) (layers "F.Cu" "B.Cu") (net 11))
   (via (at 98.04 99.21) (size 0.6) (drill 0.35) (layers "F.Cu" "B.Cu") (net 11))
@@
   (via (at 95.45 70.9425) (size 0.6) (drill 0.35) (layers "F.Cu" "B.Cu") (net 11))
   (via (at 88.74 74.215) (size 0.6) (drill 0.35) (layers "F.Cu" "B.Cu") (net 11))
-  (via (at 107.465 70.155) (size 0.6) (drill 0.35) (layers "F.Cu" "B.Cu") (net 11))
+  (via (at 107.015 70.145) (size 0.6) (drill 0.35) (layers "F.Cu" "B.Cu") (net 11))
   (segment (start 80.71 112.859616) (end 80.26243 113.307186) (width 0.15) (layer "F.Cu") (net 12))
   (segment (start 204.960864 111.83) (end 204.10952 112.681344) (width 0.15) (layer "F.Cu") (net 12))

Commit message: PCB Updates
Routing:
- added copper zone on F.Cu, net GND
Changed lines of the file:
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@@
   (segment (start 112.3193 140.0048) (end 105.4603 140.0048) (width 0.15) (layer "B.Cu") (net 94))
   (segment (start 171.7548 141.1214) (end 171.7548 140.0048) (width 0.15) (layer "B.Cu") (net 94))
+  (zone (net 11) (net_name "GND") (layer "F.Cu") (hatch edge 0.508)
+    (priority 1)
+    (connect_pads (clearance 0.25))
+    (min_thickness 0.254) (filled_areas_thickness no)
+    (fill yes (thermal_gap 0.5) (thermal_bridge_width 0.5))
+    (polygon
+      (pts
+        (xy 96.67 98.48)
+        (xy 103.02 98.47)
+        (xy 103 106.17)
+        (xy 86.7 106.2)
+        (xy 86.7 101.08)
+        (xy 91.3 96.39)
+        (xy 93.57 96.39)
+        (xy 95.51 94.42)
+        (xy 96.67 94.42)
+      )
+    )
+  )
   (group "" (id 03c52c21-9f81-4a19-9890-eb9cfb396402)
     (members

Commit message: PCB Updates
Parts:
- moved R2 0.15 mm to (95.4, 97.0)
Routing:
- net GND: track 27.8 -> 29.1 mm, vias 18 -> 19
- net (no net): vias 1 -> 0
Changed lines of the file:
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@@
   )
   (footprint "Resistor_SMD:R_0402_1005Metric_Pad0.72x0.64mm_HandSolder" (layer "F.Cu")
-    (at 95.55 96.97 90)
+    (at 95.4 96.97 90)
     (descr "Resistor SMD 0402 (1005 Metric), square (rectangular) end terminal, IPC_7351 nominal with elongated pad for handsoldering. (Body size source: IPC-SM-782 page 72, https://www.pcb-3d.com/wordpress/wp-content/uploads/ipc-sm-782a_amendment_1_and_2.pdf), generated with kicad-footprint-generator")
     (tags "resistor handsolder")
@@
     (effects (font (size 3.6 3.6) (thickness 0.15)))
   )
-  (via (at 96.35 96.85) (size 0.6) (drill 0.35) (layers "F.Cu" "B.Cu") (free) (net 0))
   (segment (start 98.74 84.1825) (end 98.74 83.3675) (width 0.2) (layer "F.Cu") (net 1))
   (segment (start 98.12 86.105) (end 98.12 84.8025) (width 0.2) (layer "F.Cu") (net 1))
@@
   (segment (start 95.71 81.025) (end 95.71 79.99) (width 0.2) (layer "F.Cu") (net 11))
   (segment (start 95.515 66.525) (end 95.785 66.255) (width 0.2) (layer "F.Cu") (net 11))
+  (segment (start 97.0075 99.21) (end 97.0075 98.7175) (width 0.15) (layer "F.Cu") (net 11))
   (segment (start 97.975 66.525) (end 97.705 66.255) (width 0.2) (layer "F.Cu") (net 11))
   (segment (start 105.9075 69.31) (end 106.18 69.31) (width 0.2) (layer "F.Cu") (net 11))
@@
   (segment (start 107.21 70.34) (end 107.34 70.47) (width 0.2) (layer "F.Cu") (net 11))
   (segment (start 95.72 92.98) (end 95.72 94.52) (width 0.2) (layer "F.Cu") (net 11))
+  (segment (start 97.0075 98.7175) (end 96.43 98.14) (width 0.15) (layer "F.Cu") (net 11))
   (segment (start 88.74 73.18) (end 88.74 74.215) (width 0.2) (layer "F.Cu") (net 11))
   (segment (start 104.03 83.91) (end 105.065 83.91) (width 0.2) (layer "F.Cu") (net 11))
@@
   (via (at 88.74 74.215) (size 0.6) (drill 0.35) (layers "F.Cu" "B.Cu") (net 11))
   (via (at 107.015 70.145) (size 0.6) (drill 0.35) (layers "F.Cu" "B.Cu") (net 11))
+  (via (at 96.35 96.85) (size 0.6) (drill 0.35) (layers "F.Cu" "B.Cu") (free) (net 11))
   (segment (start 80.71 112.859616) (end 80.26243 113.307186) (width 0.15) (layer "F.Cu") (net 12))
   (segment (start 204.960864 111.83) (end 204.10952 112.681344) (width 0.15) (layer "F.Cu") (net 12))
@@
     (polygon
       (pts
-        (xy 96.67 98.48)
+        (xy 96.83 98.48)
         (xy 103.02 98.47)
         (xy 103 106.17)
@@
         (xy 93.57 96.39)
         (xy 95.51 94.42)
-        (xy 96.67 94.42)
+        (xy 96.83 94.42)
       )
     )

Commit message: PCB Updates
Routing:
- net GND: track 29.1 -> 32.3 mm, vias 19 -> 20
Changed lines of the file:
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@@
   (segment (start 97.005 99.21) (end 98.04 99.21) (width 0.2) (layer "F.Cu") (net 11))
   (segment (start 106.18 69.31) (end 107.015 70.145) (width 0.2) (layer "F.Cu") (net 11))
+  (segment (start 95.72 94.52) (end 93.94 96.3) (width 0.2) (layer "F.Cu") (net 11))
   (segment (start 107.015 70.145) (end 107.21 70.34) (width 0.2) (layer "F.Cu") (net 11))
   (segment (start 89.4 90.8075) (end 88.365 90.8075) (width 0.2) (layer "F.Cu") (net 11))
@@
   (segment (start 104.03 83.91) (end 105.065 83.91) (width 0.2) (layer "F.Cu") (net 11))
   (segment (start 96.71 81.025) (end 96.71 79.99) (width 0.2) (layer "F.Cu") (net 11))
+  (segment (start 93.94 96.3) (end 93.94 97.02) (width 0.2) (layer "F.Cu") (net 11))
   (segment (start 98.35 96.86) (end 98.35 97.895) (width 0.2) (layer "F.Cu") (net 11))
   (segment (start 100.76 82.19) (end 100.76 81.155) (width 0.2) (layer "F.Cu") (net 11))
@@
   (via (at 105.055 85.57) (size 0.6) (drill 0.35) (layers "F.Cu" "B.Cu") (net 11))
   (via (at 105.065 83.91) (size 0.6) (drill 0.35) (layers "F.Cu" "B.Cu") (net 11))
+  (via (at 93.94 97.02) (size 0.6) (drill 0.35) (layers "F.Cu" "B.Cu") (net 11))
   (via (at 108.67 81.83) (size 0.6) (drill 0.35) (layers "F.Cu" "B.Cu") (net 11))
   (via (at 97.19 97.885) (size 0.6) (drill 0.35) (layers "F.Cu" "B.Cu") (net 11))

Commit message: PCB Updates
Routing:
- net GND: track 32.3 -> 34.3 mm, vias 20 -> 21
- added copper zone on B.Cu, net GND
Changed lines of the file:
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@@
   (segment (start 89.4 90.8075) (end 88.365 90.8075) (width 0.2) (layer "F.Cu") (net 11))
   (segment (start 99.76 82.19) (end 99.76 81.155) (width 0.2) (layer "F.Cu") (net 11))
+  (segment (start 85.245 82.425) (end 86.15 83.33) (width 0.15) (layer "F.Cu") (net 11))
   (segment (start 92.58 99.21) (end 91.545 99.21) (width 0.2) (layer "F.Cu") (net 11))
   (segment (start 107.21 70.34) (end 107.34 70.47) (width 0.2) (layer "F.Cu") (net 11))
@@
   (segment (start 104.02 85.57) (end 105.055 85.57) (width 0.2) (layer "F.Cu") (net 11))
   (segment (start 94.015 66.525) (end 95.515 66.525) (width 0.2) (layer "F.Cu") (net 11))
+  (segment (start 84.57 82.425) (end 85.245 82.425) (width 0.15) (layer "F.Cu") (net 11))
   (segment (start 95.45 69.41) (end 95.45 70.9425) (width 0.2) (layer "F.Cu") (net 11))
   (segment (start 107.34 70.47) (end 107.34 72.44) (width 0.2) (layer "F.Cu") (net 11))
@@
   (via (at 95.45 70.9425) (size 0.6) (drill 0.35) (layers "F.Cu" "B.Cu") (net 11))
   (via (at 88.74 74.215) (size 0.6) (drill 0.35) (layers "F.Cu" "B.Cu") (net 11))
+  (via (at 86.15 83.33) (size 0.6) (drill 0.35) (layers "F.Cu" "B.Cu") (net 11))
   (via (at 107.015 70.145) (size 0.6) (drill 0.35) (layers "F.Cu" "B.Cu") (net 11))
   (via (at 96.35 96.85) (size 0.6) (drill 0.35) (layers "F.Cu" "B.Cu") (free) (net 11))
@@
       )
     )
+  )
+  (zone (net 11) (net_name "GND") (layer "B.Cu") (hatch edge 0.508)
+    (connect_pads (clearance 0.2))
+    (min_thickness 0.2) (filled_areas_thickness no)
+    (fill yes (thermal_gap 0.3) (thermal_bridge_width 0.3))
+    (polygon
+      (pts
+        (xy 109.68 108.19)
+        (xy 77.66 108.2)
+        (xy 77.65 64.22)
+        (xy 109.65 64.19)
+      )
+    )

Commit message: PCB Updates
Routing:
- net +3V3: track 16.2 -> 18.8 mm
- net GND: track 34.3 -> 35.4 mm, vias 21 -> 22
- added copper zone on F.Cu, net +1V1
- added copper zone on F.Cu, net +3V3
Changed lines of the file:
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@@
   (segment (start 95.55 95.89) (end 95.55 96.3725) (width 0.15) (layer "F.Cu") (net 6))
   (segment (start 90.8075 90.5425) (end 90.54 90.81) (width 0.2) (layer "F.Cu") (net 7))
+  (segment (start 100.1575 86.9425) (end 99.3325 86.9425) (width 0.2) (layer "F.Cu") (net 7))
   (segment (start 99.32 85.6525) (end 99.68 85.2925) (width 0.2) (layer "F.Cu") (net 7))
   (segment (start 93.2825 90.5425) (end 90.8075 90.5425) (width 0.2) (layer "F.Cu") (net 7))
   (segment (start 102.6325 90.5425) (end 102.9 90.81) (width 0.2) (layer "F.Cu") (net 7))
   (segment (start 97.07 85.0325) (end 97.07 83.5525) (width 0.2) (layer "F.Cu") (net 7))
+  (segment (start 98.92 86.82) (end 99.1 87) (width 0.2) (layer "F.Cu") (net 7))
   (segment (start 97.19 95.36) (end 96.92 95.09) (width 0.2) (layer "F.Cu") (net 7))
+  (segment (start 99.32 86.93) (end 99.32 86.105) (width 0.2) (layer "F.Cu") (net 7))
+  (segment (start 98.92 86.105) (end 98.92 86.82) (width 0.2) (layer "F.Cu") (net 7))
   (segment (start 97.07 85.0525) (end 97.07 85.0325) (width 0.2) (layer "F.Cu") (net 7))
   (segment (start 97.32 86.105) (end 97.32 85.2825) (width 0.2) (layer "F.Cu") (net 7))
@@
   (segment (start 97.32 85.2825) (end 97.07 85.0325) (width 0.2) (layer "F.Cu") (net 7))
   (segment (start 97.19 95.72) (end 97.19 95.36) (width 0.2) (layer "F.Cu") (net 7))
+  (segment (start 99.3325 86.9425) (end 99.32 86.93) (width 0.2) (layer "F.Cu") (net 7))
   (segment (start 97.07 83.5525) (end 96.71 83.1925) (width 0.2) (layer "F.Cu") (net 7))
   (segment (start 98.92 85.396796) (end 99.347148 84.969648) (width 0.2) (layer "F.Cu") (net 7))
@@
   (segment (start 84.57 75.3925) (end 84.585 75.3775) (width 0.15) (layer "F.Cu") (net 10))
   (segment (start 84.585 75.3775) (end 84.585 73.165) (width 0.15) (layer "F.Cu") (net 10))
+  (segment (start 83.23 92.38) (end 83.37 92.52) (width 0.15) (layer "F.Cu") (net 11))
   (segment (start 90.63 76.63) (end 89.595 76.63) (width 0.2) (layer "F.Cu") (net 11))
   (segment (start 99.475 66.525) (end 97.975 66.525) (width 0.2) (layer "F.Cu") (net 11))
@@
   (segment (start 97.0075 98.7175) (end 96.43 98.14) (width 0.15) (layer "F.Cu") (net 11))
   (segment (start 88.74 73.18) (end 88.74 74.215) (width 0.2) (layer "F.Cu") (net 11))
+  (segment (start 82.289568 92.38) (end 83.23 92.38) (width 0.15) (layer "F.Cu") (net 11))
   (segment (start 104.03 83.91) (end 105.065 83.91) (width 0.2) (layer "F.Cu") (net 11))
   (segment (start 96.71 81.025) (end 96.71 79.99) (width 0.2) (layer "F.Cu") (net 11))
@@
   (via (at 105.065 83.91) (size 0.6) (drill 0.35) (layers "F.Cu" "B.Cu") (net 11))
   (via (at 93.94 97.02) (size 0.6) (drill 0.35) (layers "F.Cu" "B.Cu") (net 11))
+  (via (at 83.37 92.52) (size 0.6) (drill 0.35) (layers "F.Cu" "B.Cu") (net 11))
   (via (at 108.67 81.83) (size 0.6) (drill 0.35) (layers "F.Cu" "B.Cu") (net 11))
   (via (at 97.19 97.885) (size 0.6) (drill 0.35) (layers "F.Cu" "B.Cu") (net 11))
@@
   (segment (start 112.3193 140.0048) (end 105.4603 140.0048) (width 0.15) (layer "B.Cu") (net 94))
   (segment (start 171.7548 141.1214) (end 171.7548 140.0048) (width 0.15) (layer "B.Cu") (net 94))
+  (zone (net 30) (net_name "+1V1") (layer "F.Cu") (hatch edge 0.508)
+    (priority 1)
+    (connect_pads (clearance 0.15))
+    (min_thickness 0.1) (filled_areas_thickness no)
+    (fill yes (thermal_gap 0.11) (thermal_bridge_width 0.11))
+    (polygon
+      (pts
+        (xy 98.72 87.76)
+        (xy 95.12 87.76)
+        (xy 95.12 91.13)
+        (xy 97.69 91.13)
+        (xy 97.69 92.08)
+        (xy 96.91 92.08)
+        (xy 96.91 91.92)
+        (xy 94.4 91.92)
+        (xy 94.4 87.2)
+        (xy 97.31 87.2)
+        (xy 97.31 87.07)
+        (xy 97.72 87.07)
+        (xy 97.72 86.73)
+        (xy 98.72 86.73)
+      )
+    )
+  )
   (zone (net 11) (net_name "GND") (layer "F.Cu") (hatch edge 0.508)
     (priority 1)
@@
       )
     )
+  )
+  (zone (net 7) (net_name "+3V3") (layer "F.Cu") (hatch edge 0.508)
+    (connect_pads (clearance 0.18))
+    (min_thickness 0.15) (filled_areas_thickness no)
+    (fill yes (thermal_gap 0.25) (thermal_bridge_width 0.25))
+    (polygon
+      (pts
+        (xy 100.84 93.66)
+        (xy 92.6 93.66)
+        (xy 92.6 85.42)
+        (xy 100.84 85.42)
+      )
+    )

Commit message: PCB Updates
Routing:
- net +1V1: track 10.7 -> 11.6 mm
Changed lines of the file:
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@@
   (segment (start 97.32 94.43) (end 97.58 94.69) (width 0.2) (layer "F.Cu") (net 30))
   (segment (start 96.52 84.7625) (end 96.52 86.105) (width 0.2) (layer "F.Cu") (net 30))
+  (segment (start 98.52 86.105) (end 98.52 86.98) (width 0.2) (layer "F.Cu") (net 30))
   (segment (start 98.52 86.105) (end 98.52 85.3025) (width 0.2) (layer "F.Cu") (net 30))
   (segment (start 99.75 84.0725) (end 99.75 83.33) (width 0.2) (layer "F.Cu") (net 30))
@@
         (xy 97.69 92.08)
         (xy 96.91 92.08)
-        (xy 96.91 91.92)
-        (xy 94.4 91.92)
-        (xy 94.4 87.2)
-        (xy 97.31 87.2)
+        (xy 96.91 91.75)
+        (xy 94.51 91.75)
+        (xy 94.51 87.33)
+        (xy 97.31 87.33)
         (xy 97.31 87.07)
         (xy 97.72 87.07)
