File: KiCAD_PCB/Calculator_PCB/Shit.kicad_pcb (KiCad board)
At the start: 2 copper layers, 110 parts, among them J1 USB_B_Micro, J2 5034801000, J3 5034801000, SW1 SW_SPST, SW10 SW_SPST, SW11 SW_SPST, SW12 SW_SPST, SW13 SW_SPST, SW14 SW_SPST, SW15 SW_SPST, SW16 SW_SPST, SW17 SW_SPST, SW18 SW_SPST, SW19 SW_SPST, SW2 SW_SPST, SW20 SW_SPST, SW21 SW_SPST, SW22 SW_SPST, SW23 SW_SPST, SW24 SW_SPST, SW25 SW_SPST, SW26 SW_SPST, SW27 SW_SPST, SW28 SW_SPST, SW29 SW_SPST, SW3 SW_SPST, SW30 SW_SPST, SW31 SW_SPST, SW32 SW_SPST, SW33 SW_SPST, SW34 SW_SPST, SW35 SW_SPST, SW36 SW_SPST, SW37 SW_SPST, SW38 SW_SPST, SW39 SW_SPST, SW4 SW_SPST, SW40 SW_SPST, SW5 SW_SPST, SW6 SW_SPST, SW7 SW_SPST, SW8 SW_SPST, SW9 SW_SPST, U1 W25Q128JVS, U2 RP2040, U3 NCP1117-3.3_SOT223, Y1 ABLS-12.000MHZ-B4-T

Commit message: PCB Updates
Parts:
- moved J2 2.80 mm to (80.2, 92.4), turned to 90 degrees
Connections:
- D1 pad 1: /Row3 -> /Row2
- D10 pad 1: /Row4 -> /Row3
- D11 pad 1: /Row5 -> /Row4
- D12 pad 1: /Row6 -> /Row5
- D13 pad 1: /Row3 -> /Row2
- D14 pad 1: /Row4 -> /Row3
- D15 pad 1: /Row5 -> /Row4
- D16 pad 1: /Row6 -> /Row5
- D17 pad 1: /Row3 -> /Row2
- D18 pad 1: /Row4 -> /Row3
- D19 pad 1: /Row5 -> /Row4
- D2 pad 1: /Row4 -> /Row3
- D20 pad 1: /Row6 -> /Row5
- D21 pad 1: /Row3 -> /Row2
- D22 pad 1: /Row4 -> /Row3
- D23 pad 1: /Row5 -> /Row4
- D24 pad 1: /Row6 -> /Row5
- D25 pad 1: /Row3 -> /Row2
- D26 pad 1: /Row4 -> /Row3
- D27 pad 1: /Row5 -> /Row4
- D28 pad 1: /Row6 -> /Row5
- D29 pad 1: /Row3 -> /Row2
- D3 pad 1: /Row5 -> /Row4
- D30 pad 1: /Row4 -> /Row3
- D31 pad 1: /Row5 -> /Row4
- D32 pad 1: /Row6 -> /Row5
- D33 pad 1: /Row3 -> /Row2
- D34 pad 1: /Row4 -> /Row3
- D35 pad 1: /Row5 -> /Row4
- D36 pad 1: /Row6 -> /Row5
- D37 pad 1: /Row3 -> /Row2
- D38 pad 1: /Row4 -> /Row3
- D39 pad 1: /Row5 -> /Row4
- D4 pad 1: /Row6 -> /Row5
- D40 pad 1: /Row6 -> /Row5
- D5 pad 1: /Row3 -> /Row2
- D6 pad 1: /Row4 -> /Row3
- D7 pad 1: /Row5 -> /Row4
- D8 pad 1: /Row6 -> /Row5
- D9 pad 1: /Row3 -> /Row2
- J2 pad 1: /Row4 -> +3V3
- J2 pad 10: GND -> /Row3
- J2 pad 2: /Row5 -> /y_out
- J2 pad 3: /Row6 -> /x_out
- J2 pad 4: /Col0 -> GND
- J2 pad 5: /Col1 -> /Col0
- J2 pad 6: /Col2 -> /Col1
- J2 pad 7: /x_out -> /Col2
- J2 pad 8: /y_out -> /Row5
- J2 pad 9: +3V3 -> /Row4
- U2 pad 2: /Row6 -> /Row5
- U2 pad 3: /Row5 -> /Row4
- U2 pad 4: /Row4 -> /Row3
- U2 pad 5: /Row3 -> /Row2
Routing:
- net /Row6: track 197.7 -> 0.00 mm, vias 1 -> 0
- net /Row2: track 0.00 -> 165.9 mm, vias 0 -> 1
- net /Row3: track 165.9 -> 184.3 mm
- net /Row4: track 180.3 -> 193.4 mm
- net /Row5: track 190.0 -> 201.6 mm
- net /Col1: track 10.9 -> 2.82 mm, vias 1 -> 0
- net /Col2: track 9.92 -> 3.52 mm, vias 1 -> 0
- net GND: track 27.8 -> 29.4 mm
- net /y_out: track 0.68 -> 0.00 mm
- net +3V3: track 16.8 -> 16.2 mm
