File: KiCAD_PCB/Calculator_PCB _V2/Calculator_PCB _V2.kicad_pcb (KiCad board)
At the start: 2 copper layers, 132 x 78 mm, 110 parts, among them J1 USB_B_Micro, J2 5034801000, J3 5034801000, SW1 SW_SPST, SW10 SW_SPST, SW11 SW_SPST, SW12 SW_SPST, SW13 SW_SPST, SW14 SW_SPST, SW15 SW_SPST, SW16 SW_SPST, SW17 SW_SPST, SW18 SW_SPST, SW19 SW_SPST, SW2 SW_SPST, SW20 SW_SPST, SW21 SW_SPST, SW22 SW_SPST, SW23 SW_SPST, SW24 SW_SPST, SW25 SW_SPST, SW26 SW_SPST, SW27 SW_SPST, SW28 SW_SPST, SW29 SW_SPST, SW3 SW_SPST, SW30 SW_SPST, SW31 SW_SPST, SW32 SW_SPST, SW33 SW_SPST, SW34 SW_SPST, SW35 SW_SPST, SW36 SW_SPST, SW37 SW_SPST, SW38 SW_SPST, SW39 SW_SPST, SW4 SW_SPST, SW40 SW_SPST, SW5 SW_SPST, SW6 SW_SPST, SW7 SW_SPST, SW8 SW_SPST, SW9 SW_SPST, U1 W25Q128JVS, U2 RP2040, U3 NCP1117-3.3_SOT223, Y1 ABLS-12.000MHZ-B4-T

Commit message: PCB V2 Updates
Parts:
- removed C1, C10, C11, C12, C2, C4, C5, C7, C8, C9: 100n, Capacitor_SMD:C_0402_1005Metric_Pad0.74x0.62mm_HandSolder
- removed C13, C14: 10u, Capacitor_SMD:C_0805_2012Metric_Pad1.18x1.45mm_HandSolder
- removed C15, C16: 27p, Capacitor_SMD:C_0402_1005Metric_Pad0.74x0.62mm_HandSolder
- removed C3, C6: 1u, Capacitor_SMD:C_0402_1005Metric_Pad0.74x0.62mm_HandSolder
- removed J2: 5034801000, 5034801000:MOLEX_5034801000
- removed R1, R2: 1k, Resistor_SMD:R_0402_1005Metric_Pad0.72x0.64mm_HandSolder
- removed R3, R4: 27.4, Resistor_SMD:R_0402_1005Metric_Pad0.72x0.64mm_HandSolder
- removed R5, R6: 10k, Resistor_SMD:R_0402_1005Metric_Pad0.72x0.64mm_HandSolder
- removed U2: RP2040, RP2040_minimal:RP2040-QFN-56
- removed U3: NCP1117-3.3_SOT223, Package_TO_SOT_SMD:SOT-223-3_TabPin2
- removed Y1: ABLS-12.000MHZ-B4-T, RP2040_minimal:Crystal_SMD_HC49-US
- J1: moved to B.Cu
- U1: value W25Q128JVS -> RP2040_Stamp; footprint Package_SO:SOIC-8_5.23x5.23mm_P1.27mm -> RP2040_Stamp:RP2040_Stamp_SMD; moved to B.Cu
- moved S1 18.4 mm to (105.0, 70.4)
- moved U1 8.48 mm to (93.7, 87.0), turned to 180 degrees
- moved J1 3.14 mm to (93.6, 67.0), turned to 0 degrees
Connections:
- U1 pad 1: /QSPI_SS_56 -> unconnected-(U1-Pad1)
- U1 pad 2: /QSPI_SD1_55 -> unconnected-(U1-Pad2)
- U1 pad 3: /QSPI_SD2_54 -> unconnected-(U1-Pad3)
- U1 pad 4: GND -> unconnected-(U1-Pad4)
- U1 pad 5: /QSPI_SD0_53 -> unconnected-(U1-Pad5)
- U1 pad 6: /QSPI_SCLK_52 -> unconnected-(U1-Pad6)
- U1 pad 7: /QSPI_SD3_51 -> unconnected-(U1-Pad7)
- U1 pad 8: +3V3 -> unconnected-(U1-Pad8)
Routing:
- net /x_out: track 69.1 -> 0.00 mm, vias 4 -> 0
- net /y_out: track 64.9 -> 0.00 mm, vias 4 -> 0
- net /Col2: track 57.9 -> 0.00 mm, vias 2 -> 0
- net +3V3: track 36.4 -> 0.00 mm, vias 2 -> 0
- net GND: track 35.4 -> 0.00 mm, vias 22 -> 0
- net /Row6: track 234.7 -> 203.5 mm
- net /Row5: track 219.0 -> 188.3 mm
- net /Row4: track 203.1 -> 173.1 mm
- net /Row1: track 125.0 -> 100.0 mm
- net /Row7: track 129.4 -> 104.6 mm
- net /Row2: track 126.1 -> 101.4 mm
- net /Col15: track 119.7 -> 96.3 mm
- net /QSPI_SS_56: track 23.3 -> 0.00 mm
- net /Col14: track 119.7 -> 96.5 mm
- net /Col13: track 119.8 -> 96.7 mm
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- removed copper zone on F.Cu, net +1V1
- removed copper zone on F.Cu, net +3V3
- removed copper zone on F.Cu, net GND
- removed copper zone on F.Cu, net VBUS

Commit message: PCB V2 Updates
Parts:
- added J2: 5034801000, 5034801000:MOLEX_5034801000, B.Cu at (81.4, 110.6)
- J3: moved to B.Cu
- moved S1 3.47 mm to (102.2, 68.3), turned to 90 degrees
- moved J3 0.48 mm to (205.9, 110.6), turned to -90 degrees
Routing:
- net /Row7: track 104.6 -> 0.00 mm
- net /Row2: track 101.4 -> 0.00 mm
- net /Row1: track 100.0 -> 0.00 mm
- net /Col13: track 96.7 -> 0.00 mm
- net /Col14: track 96.5 -> 0.00 mm
- net /Col15: track 96.3 -> 0.00 mm
- net /Col12: track 185.2 -> 160.7 mm
- net /Col11: track 171.8 -> 147.9 mm
- net /Col10: track 158.7 -> 135.2 mm
- net /Col9: track 145.6 -> 122.7 mm
- net /Col6: track 102.6 -> 79.7 mm
- net /Col7: track 116.0 -> 93.7 mm
- net /Col4: track 76.5 -> 54.2 mm
- net /Col8: track 132.4 -> 110.4 mm
- net /Col3: track 63.3 -> 41.4 mm
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- added copper zone on F.Cu, net GND
- removed copper zone on B.Cu, net GND

Commit message: PCB V2 Updates
Routing:
- net /Row5: track 167.4 -> 154.3 mm, vias 2 -> 1
- net /Row6: track 183.0 -> 172.5 mm
- net /Row4: track 151.2 -> 148.8 mm, vias 2 -> 1
Changed lines of the file:
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@@
   (segment (start 93.61 70.035) (end 93.90452 70.32952) (width 0.4) (layer "B.Cu") (net 2))
   (segment (start 93.90452 77.741228) (end 93.90452 70.645) (width 0.8) (layer "B.Cu") (net 2))
-  (segment (start 80.87 121.743844) (end 80.87 122.15) (width 0.15) (layer "F.Cu") (net 5))
   (segment (start 204.10952 112.681344) (end 204.10952 120.15718) (width 0.15) (layer "F.Cu") (net 5))
-  (segment (start 81.101922 121.511922) (end 80.87 121.743844) (width 0.15) (layer "F.Cu") (net 5))
   (segment (start 204.10952 120.15718) (end 203.2685 120.9982) (width 0.15) (layer "F.Cu") (net 5))
   (via (at 203.2685 120.9982) (size 0.6) (drill 0.35) (layers "F.Cu" "B.Cu") (net 5))
-  (via (at 80.87 122.15) (size 0.6) (drill 0.35) (layers "F.Cu" "B.Cu") (net 5))
   (segment (start 112.2934 124.0028) (end 105.4344 124.0028) (width 0.15) (layer "B.Cu") (net 5))
   (segment (start 148.1318 125.3236) (end 147.9286 125.1204) (width 0.15) (layer "B.Cu") (net 5))
@@
   (segment (start 196.29 121.3482) (end 196.64 120.9982) (width 0.15) (layer "B.Cu") (net 5))
   (segment (start 171.7294 125.1194) (end 171.7294 124.0028) (width 0.15) (layer "B.Cu") (net 5))
-  (segment (start 82.069519 123.349519) (end 80.87 122.15) (width 0.15) (layer "B.Cu") (net 5))
   (segment (start 93.5482 124.0028) (end 92.2274 125.3236) (width 0.15) (layer "B.Cu") (net 5))
   (segment (start 88.646 125.3236) (end 88.4428 125.1204) (width 0.15) (layer "B.Cu") (net 5))
@@
   (segment (start 129.2596 124.0033) (end 127.9388 125.3241) (width 0.15) (layer "B.Cu") (net 5))
   (segment (start 141.1468 124.0028) (end 139.826 125.3236) (width 0.15) (layer "B.Cu") (net 5))
-  (segment (start 80.84 126.73) (end 80.84 126.33) (width 0.15) (layer "F.Cu") (net 6))
-  (segment (start 80.255489 121.806913) (end 80.712402 121.35) (width 0.15) (layer "F.Cu") (net 6))
-  (segment (start 81.101922 126.068078) (end 81.101922 123.250973) (width 0.15) (layer "F.Cu") (net 6))
-  (segment (start 80.712402 120.98) (end 80.71048 120.978078) (width 0.15) (layer "F.Cu") (net 6))
   (segment (start 204.49904 112.842688) (end 204.49904 127.79766) (width 0.15) (layer "F.Cu") (net 6))
-  (segment (start 80.712402 121.35) (end 80.712402 120.98) (width 0.15) (layer "F.Cu") (net 6))
-  (segment (start 80.84 126.33) (end 81.101922 126.068078) (width 0.15) (layer "F.Cu") (net 6))
   (segment (start 204.49904 127.79766) (end 203.2985 128.9982) (width 0.15) (layer "F.Cu") (net 6))
-  (segment (start 80.255489 122.40454) (end 80.255489 121.806913) (width 0.15) (layer "F.Cu") (net 6))
-  (segment (start 81.101922 123.250973) (end 80.255489 122.40454) (width 0.15) (layer "F.Cu") (net 6))
   (via (at 203.2985 128.9982) (size 0.6) (drill 0.35) (layers "F.Cu" "B.Cu") (net 6))
-  (via (at 80.84 126.73) (size 0.6) (drill 0.35) (layers "F.Cu" "B.Cu") (net 6))
   (segment (start 92.2264 133.3246) (end 88.645 133.3246) (width 0.15) (layer "B.Cu") (net 6))
   (segment (start 153.0599 132.0038) (end 151.7391 133.3246) (width 0.15) (layer "B.Cu") (net 6))
@@
   (segment (start 112.2934 132.0038) (end 105.4344 132.0038) (width 0.15) (layer "B.Cu") (net 6))
   (segment (start 127.9134 133.3246) (end 124.332 133.3246) (width 0.15) (layer "B.Cu") (net 6))
-  (segment (start 81.680481 127.520481) (end 83.62 129.46) (width 0.15) (layer "B.Cu") (net 6))
   (segment (start 164.9466 132.0038) (end 163.6258 133.3246) (width 0.15) (layer "B.Cu") (net 6))
   (segment (start 105.4344 132.0038) (end 104.1136 133.3246) (width 0.15) (layer "B.Cu") (net 6))
@@
   (segment (start 148.1577 133.3246) (end 147.9545 133.1214) (width 0.15) (layer "B.Cu") (net 6))
   (segment (start 183.642 133.1204) (end 183.642 132.0038) (width 0.15) (layer "B.Cu") (net 6))
-  (segment (start 81.680481 127.520481) (end 80.89 126.73) (width 0.15) (layer "B.Cu") (net 6))
   (segment (start 104.1136 133.3246) (end 100.5322 133.3246) (width 0.15) (layer "B.Cu") (net 6))
   (segment (start 171.7294 133.1204) (end 171.7294 132.0038) (width 0.15) (layer "B.Cu") (net 6))
   (segment (start 116.0262 133.3246) (end 112.4448 133.3246) (width 0.15) (layer "B.Cu") (net 6))
-  (segment (start 83.62 131.3176) (end 84.3062 132.0038) (width 0.15) (layer "B.Cu") (net 6))
-  (segment (start 83.62 129.46) (end 83.62 131.3176) (width 0.15) (layer "B.Cu") (net 6))
   (segment (start 196.32 129.3482) (end 196.67 128.9982) (width 0.15) (layer "B.Cu") (net 6))
   (segment (start 141.1468 132.0038) (end 139.826 133.3246) (width 0.15) (layer "B.Cu") (net 6))
@@
   (segment (start 171.9316 133.3246) (end 171.7284 133.1214) (width 0.15) (layer "B.Cu") (net 6))
   (segment (start 100.4062 132.0038) (end 93.5472 132.0038) (width 0.15) (layer "B.Cu") (net 6))
-  (segment (start 80.89 126.73) (end 80.84 126.73) (width 0.15) (layer "B.Cu") (net 6))
   (segment (start 82.283362 127.28941) (end 82.283363 126.6) (width 0.15) (layer "F.Cu") (net 7))
   (segment (start 178.54 133.46) (end 178.59 133.46) (width 0.15) (layer "F.Cu") (net 7))
@@
   (segment (start 177.2738 130.542) (end 175.3004 130.542) (width 0.15) (layer "B.Cu") (net 59))
   (segment (start 205.062592 112.83) (end 204.88856 113.004032) (width 0.15) (layer "F.Cu") (net 67))
-  (segment (start 79.86597 122.565885) (end 80.712402 123.412317) (width 0.15) (layer "F.Cu") (net 67))
   (segment (start 204.88856 135.40964) (end 203.29 137.0082) (width 0.15) (layer "F.Cu") (net 67))
   (segment (start 83.042334 134.951423) (end 84.81 136.719089) (width 0.15) (layer "F.Cu") (net 67))
-  (segment (start 80.712402 125.906734) (end 80.225489 126.393647) (width 0.15) (layer "F.Cu") (net 67))
   (segment (start 83.042334 129.801385) (end 83.042334 134.951423) (width 0.15) (layer "F.Cu") (net 67))
-  (segment (start 80.225489 126.98454) (end 83.042334 129.801385) (width 0.15) (layer "F.Cu") (net 67))
-  (segment (start 80.32096 121.190578) (end 79.865969 121.645569) (width 0.15) (layer "F.Cu") (net 67))
   (segment (start 204.88856 113.004032) (end 204.88856 135.40964) (width 0.15) (layer "F.Cu") (net 67))
-  (segment (start 80.712402 123.412317) (end 80.712402 125.906734) (width 0.15) (layer "F.Cu") (net 67))
-  (segment (start 79.865969 121.645569) (end 79.86597 122.565885) (width 0.15) (layer "F.Cu") (net 67))
   (segment (start 84.81 136.719089) (end 84.81 139.22) (width 0.15) (layer "F.Cu") (net 67))
-  (segment (start 80.225489 126.393647) (end 80.225489 126.98454) (width 0.15) (layer "F.Cu") (net 67))
   (via (at 84.81 139.22) (size 0.6) (drill 0.35) (layers "F.Cu" "B.Cu") (net 67))
   (via (at 203.29 137.0082) (size 0.6) (drill 0.35) (layers "F.Cu" "B.Cu") (net 67))

Commit message: V2 PCB Updates
Connections:
- U1 pad 11: unconnected-(U1-Pad11) -> /Col12
- U1 pad 12: unconnected-(U1-Pad12) -> /Col11
- U1 pad 13: unconnected-(U1-Pad13) -> /Col10
- U1 pad 14: unconnected-(U1-Pad14) -> /Col9
- U1 pad 15: unconnected-(U1-Pad15) -> /Col8
- U1 pad 16: unconnected-(U1-Pad16) -> /Col7
- U1 pad 17: unconnected-(U1-Pad17) -> /Col6
- U1 pad 18: unconnected-(U1-Pad18) -> /Col5
- U1 pad 19: unconnected-(U1-Pad19) -> /Col4
- U1 pad 20: unconnected-(U1-Pad20) -> /Col3
Routing:
- net /Row5: track 154.3 -> 179.1 mm
- net /Row4: track 148.8 -> 166.9 mm
- net /Row3: track 138.8 -> 150.1 mm
- net /Col8: track 110.4 -> 100.9 mm
- net /Col9: track 122.7 -> 113.7 mm
- net /Col11: track 147.9 -> 139.3 mm
- net /Col12: track 160.7 -> 152.1 mm
- net /Col10: track 135.2 -> 126.8 mm
- net /Col5: track 69.2 -> 63.3 mm
- net /Col7: track 93.7 -> 88.3 mm
- net /Row6: track 172.5 -> 167.3 mm
- net /Col6: track 79.7 -> 75.8 mm
- net /Col3: track 41.4 -> 37.9 mm
- net /Col4: track 54.2 -> 50.9 mm
- net unconnected-(U1-Pad23): track 0.00 -> 2.24 mm, vias 0 -> 1
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
Commit message: V2 PCB Updates
Routing:
- net /Col10: track 126.8 -> 34.7 mm, vias 1 -> 0
- net /Col9: track 113.7 -> 34.1 mm, vias 1 -> 0
- net /Col8: track 100.9 -> 39.9 mm, vias 1 -> 0
- net /Row6: track 167.3 -> 198.1 mm, vias 2 -> 1
- net /Col12: track 152.1 -> 140.7 mm, vias 1 -> 0
- net /Col11: track 139.3 -> 129.7 mm, vias 1 -> 0
- net /Row5: track 179.1 -> 182.7 mm

Commit message: V2 PCB updates
Connections:
- J2 pad 1: /Row4 -> unconnected-(J2-Pad1)
- J2 pad 10: /Col1 -> unconnected-(J2-Pad10)
- J2 pad 2: /Row5 -> unconnected-(J2-Pad2)
- J2 pad 3: /Row6 -> unconnected-(J2-Pad3)
- J2 pad 4: +3V3 -> unconnected-(J2-Pad4)
- J2 pad 5: GND -> unconnected-(J2-Pad5)
- J2 pad 6: /x_out -> unconnected-(J2-Pad6)
- J2 pad 7: /y_out -> unconnected-(J2-Pad7)
- J2 pad 8: /Col2 -> unconnected-(J2-Pad8)
- J2 pad 9: /Col0 -> unconnected-(J2-Pad9)
- J2 pad S1: unconnected-(J2-PadS1) -> GND
- J2 pad S2: unconnected-(J2-PadS1) -> GND
- J3 pad S1: unconnected-(J3-PadS1) -> GND
- J3 pad S2: unconnected-(J3-PadS1) -> GND
- U1 pad 21: unconnected-(U1-Pad21) -> /Row3
- U1 pad 22: unconnected-(U1-Pad22) -> /Row4
- U1 pad 23: unconnected-(U1-Pad23) -> /Row5
- U1 pad 24: unconnected-(U1-Pad24) -> /Row6
- U1 pad 25: unconnected-(U1-Pad25) -> /y_out
- U1 pad 26: unconnected-(U1-Pad26) -> /x_out
- U1 pad 34: unconnected-(U1-Pad34) -> +3V3
Routing:
- net /Col12: track 140.7 -> 31.7 mm
- net /Col11: track 129.7 -> 31.7 mm
- net /Col7: track 88.3 -> 31.7 mm, vias 1 -> 0
- net /Col6: track 75.8 -> 31.7 mm, vias 1 -> 0
- net /Col5: track 63.3 -> 31.7 mm, vias 1 -> 0
- net /Row5: track 182.7 -> 208.5 mm, vias 1 -> 2
- net /Row4: track 166.9 -> 191.5 mm, vias 1 -> 2
- net /Row3: track 150.1 -> 173.5 mm, vias 1 -> 2
- net /Col4: track 50.9 -> 31.6 mm, vias 1 -> 0
- net /Row6: track 198.1 -> 208.6 mm
- net /Col8: track 39.9 -> 31.7 mm
- net /Col3: track 37.9 -> 31.7 mm, vias 1 -> 0
- net /Col10: track 34.7 -> 31.7 mm
- net /Col9: track 34.1 -> 31.7 mm
- net unconnected-(U1-Pad23): track 2.24 -> 0.00 mm, vias 1 -> 0
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
Commit message: V2 PCB Updates
Connections:
- J2 pad 10: unconnected-(J2-Pad10) -> /Row3
- J2 pad 3: unconnected-(J2-Pad3) -> /Col2
- J2 pad 4: unconnected-(J2-Pad4) -> /Col1
- J2 pad 5: unconnected-(J2-Pad5) -> /Col0
- J2 pad 6: unconnected-(J2-Pad6) -> /x_out
- J2 pad 7: unconnected-(J2-Pad7) -> /y_out
- J2 pad 8: unconnected-(J2-Pad8) -> /Row5
- J2 pad 9: unconnected-(J2-Pad9) -> /Row4
- U1 pad 24: /Row6 -> /y_out
- U1 pad 25: /y_out -> /x_out
- U1 pad 26: /x_out -> /Row6
- U1 pad 27: unconnected-(U1-Pad27) -> /Col2
- U1 pad 28: unconnected-(U1-Pad28) -> /Col1
- U1 pad 29: unconnected-(U1-Pad29) -> /Col0
Routing:
- net /Col0: track 0.00 -> 36.6 mm
- net /Col1: track 0.00 -> 35.3 mm
- net /Col2: track 0.00 -> 34.1 mm
- net /Row6: track 208.6 -> 220.4 mm
- net /x_out: track 0.00 -> 9.31 mm, vias 0 -> 1
- net /y_out: track 0.00 -> 8.81 mm, vias 0 -> 1
- net /Row3: track 173.5 -> 165.1 mm
- net /Row4: track 191.5 -> 187.2 mm
- net /Row5: track 208.5 -> 205.9 mm

Commit message: V2 Updates
Connections:
- U1 pad 24: /y_out -> /Row6
- U1 pad 25: /x_out -> /Col0
- U1 pad 26: /Row6 -> /Col1
- U1 pad 28: /Col1 -> /y_out
- U1 pad 29: /Col0 -> /x_out
Routing:
- net /Col6: track 31.7 -> 114.5 mm
- net /Col7: track 31.7 -> 112.5 mm
- net /Col8: track 31.7 -> 110.5 mm
- net /Col15: track 0.00 -> 77.5 mm
- net /Row2: track 0.00 -> 77.5 mm
- net /Col14: track 0.00 -> 77.3 mm
- net /Row7: track 0.00 -> 77.3 mm
- net /Row1: track 0.00 -> 77.2 mm
- net /Col9: track 31.7 -> 108.5 mm
- net /Col10: track 31.7 -> 106.4 mm
- net /Col11: track 31.7 -> 104.4 mm
- net /Col12: track 31.7 -> 102.2 mm
- net /Col13: track 0.00 -> 68.8 mm
- net /Col5: track 31.7 -> 88.0 mm
- net /Col1: track 35.3 -> 0.00 mm
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