File: KiCAD_PCB/Calculator_PCB _V2/Calculator_PCB _V2.kicad_pcb (KiCad board)
At the start: 2 copper layers, 132 x 78 mm, 85 parts, among them J1 USB_B_Micro, J2 5034801000, J3 5034801000, SW1 SW_SPST, SW10 SW_SPST, SW11 SW_SPST, SW12 SW_SPST, SW13 SW_SPST, SW14 SW_SPST, SW15 SW_SPST, SW16 SW_SPST, SW17 SW_SPST, SW18 SW_SPST, SW19 SW_SPST, SW2 SW_SPST, SW20 SW_SPST, SW21 SW_SPST, SW22 SW_SPST, SW23 SW_SPST, SW24 SW_SPST, SW25 SW_SPST, SW26 SW_SPST, SW27 SW_SPST, SW28 SW_SPST, SW29 SW_SPST, SW3 SW_SPST, SW30 SW_SPST, SW31 SW_SPST, SW32 SW_SPST, SW33 SW_SPST, SW34 SW_SPST, SW35 SW_SPST, SW36 SW_SPST, SW37 SW_SPST, SW38 SW_SPST, SW39 SW_SPST, SW4 SW_SPST, SW40 SW_SPST, SW5 SW_SPST, SW6 SW_SPST, SW7 SW_SPST, SW8 SW_SPST, SW9 SW_SPST, U1 RP2040_Stamp

Commit message: V2 Updates
Routing:
- net /Col6: track 114.5 -> 77.2 mm
- net /Col12: track 102.2 -> 136.4 mm
- net /Col13: track 68.8 -> 97.0 mm
- net /Col14: track 77.3 -> 105.4 mm
- net /Col15: track 77.5 -> 105.4 mm
- net /Row1: track 77.2 -> 104.9 mm
- net /Row7: track 77.3 -> 104.8 mm
- net /Row2: track 77.5 -> 104.9 mm
- net /Col4: track 31.6 -> 58.9 mm
- net /Col7: track 112.5 -> 87.1 mm
- net /Col11: track 104.4 -> 126.6 mm
- net /Col5: track 88.0 -> 67.2 mm
- net /Col3: track 31.7 -> 49.5 mm
- net /Col8: track 110.5 -> 96.9 mm
- net /Col10: track 106.4 -> 116.7 mm
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
Commit message: V2 Updates
Connections:
- J2 pad 3: /Col2 -> /Col0
- J2 pad 5: /Col0 -> /Col2
Routing:
- net /x_out: track 36.6 -> 0.00 mm
- net /y_out: track 35.3 -> 0.00 mm
- net /Col1: track 0.00 -> 31.3 mm
- net /Col0: track 5.90 -> 30.0 mm, vias 1 -> 0
- net /Row6: track 225.8 -> 216.4 mm, vias 2 -> 1
- net /Col2: track 34.1 -> 32.6 mm

Commit message: V2 PCB Updates
Parts:
- moved J1 32.0 mm to (70.0, 45.5)
Connections:
- J2 pad 10: /Row3 -> /y_out
- J2 pad 3: /Col0 -> /Row5
- J2 pad 4: /Col1 -> /Row4
- J2 pad 5: /Col2 -> /Row3
- J2 pad 6: /x_out -> /Col0
- J2 pad 7: /y_out -> /Col1
- J2 pad 8: /Row5 -> /Col2
- J2 pad 9: /Row4 -> /x_out
Routing:
- net /x_out: track 0.00 -> 34.6 mm, vias 0 -> 2
- net /y_out: track 0.00 -> 30.9 mm, vias 0 -> 2
- net /Row5: track 202.5 -> 224.5 mm, vias 2 -> 3
- net /Row4: track 183.7 -> 198.3 mm, vias 2 -> 3
- net /Row3: track 161.6 -> 168.7 mm, vias 2 -> 3
- net /Col2: track 32.6 -> 31.1 mm
- net /Col0: track 30.0 -> 28.5 mm
- net /Col1: track 31.3 -> 29.8 mm

Commit message: Updating Version 2
Parts:
- removed J1: USB_B_Micro, Connector_USB:USB_Micro-B_Amphenol_10103594-0001LF_Horizontal
- added JP1: HEADER-1X570MIL, USB_B_Micro_Breakout:USB_B_Micro_Headers, B.Cu at (92.3, 68.3)
- added REF**: MountingHole_2.2mm_M2_DIN965, MountingHole:MountingHole_2.2mm_M2_DIN965, F.Cu at (79.7, 140.2)
- added REF**: MountingHole_2.2mm_M2_DIN965, MountingHole:MountingHole_2.2mm_M2_DIN965, F.Cu at (207.7, 140.2)
- added REF**: MountingHole_2.2mm_M2_DIN965, MountingHole:MountingHole_2.2mm_M2_DIN965, F.Cu at (79.6, 66.2)
- added REF**: MountingHole_2.2mm_M2_DIN965, MountingHole:MountingHole_2.2mm_M2_DIN965, F.Cu at (107.7, 66.2)
- added REF**: MountingHole_2.2mm_M2_DIN965, MountingHole:MountingHole_2.2mm_M2_DIN965, F.Cu at (207.7, 104.7)
- added REF**: PinHeader_1x01_P2.00mm_Vertical, Connector_PinHeader_2.00mm:PinHeader_1x01_P2.00mm_Vertical, B.Cu at (79.3, 75.0)
- added REF**: PinHeader_1x02_P2.00mm_Vertical, Connector_PinHeader_2.00mm:PinHeader_1x02_P2.00mm_Vertical, B.Cu at (79.3, 72.0)
Connections:
- J3 pad 1: /Row7 -> /Col15
- J3 pad 10: /Col15 -> /Row7
- J3 pad 2: /Row6 -> /Col14
- J3 pad 3: /Row5 -> /Col13
- J3 pad 4: /Row4 -> /Row1
- J3 pad 5: /Row3 -> /Row2
- J3 pad 6: /Row2 -> /Row3
- J3 pad 7: /Row1 -> /Row4
- J3 pad 8: /Col13 -> /Row5
- J3 pad 9: /Col14 -> /Row6
- S1 pad 1: /USB_BOOT -> GND
- S1 pad 4: GND -> /USB_BOOT
- U1 pad 10: unconnected-(U1-Pad10) -> /Col13
- U1 pad 30: unconnected-(U1-Pad30) -> /Row0
- U1 pad 5: unconnected-(U1-Pad5) -> /Row7
- U1 pad 6: unconnected-(U1-Pad6) -> /Row2
- U1 pad 7: unconnected-(U1-Pad7) -> /Row1
- U1 pad 8: unconnected-(U1-Pad8) -> /Col15
- U1 pad 9: unconnected-(U1-Pad9) -> /Col14
Routing:
- net /Row7: track 104.8 -> 126.0 mm
- net +3V3: track 0.00 -> 20.3 mm
- net /Row2: track 104.9 -> 120.8 mm
- net /Row1: track 104.9 -> 118.0 mm
- net /Col13: track 97.0 -> 109.8 mm
- net GND: track 0.00 -> 12.4 mm, vias 0 -> 7
- net /USB_BOOT: track 0.00 -> 9.36 mm, vias 0 -> 1
- net /Col15: track 105.4 -> 112.8 mm
- net VBUS: track 1.10 -> 7.57 mm
- net /Col14: track 105.4 -> 111.4 mm
- net /Row0: track 0.00 -> 5.24 mm
- net /Row3: track 168.7 -> 173.0 mm, vias 3 -> 2
- net /Row4: track 198.3 -> 201.1 mm, vias 3 -> 2
- net /Row5: track 224.5 -> 226.8 mm, vias 3 -> 2
- net Net-(D39-Pad2): track 5.76 -> 3.55 mm, vias 1 -> 0
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Other:
- outline, holes or cut-outs redrawn
- board text added: "+3V3"
- board text added: "+5V"
- board text added: "Col1"
- board text added: "Col2"
- board text added: "Col3"
- board text added: "Col5"
- board text added: "Col6"
- board text added: "Col7"
- board text added: "Col8"
- board text added: "Col9"
- board text added: "D+"
- board text added: "D-"
- board text added: "GND"
- board text added: "MATH"
- board text added: "MATHilda"
- board text added: "Powered by ilda"
- board text added: "Row3"
- board text added: "Row4"
- board text added: "Row5"
- board text added: "Row6"
- board text added: "x_out"
- board text added: "y_out"

Commit message: V2 Updates
Other:
- board text added: "Col10"
- board text added: "Col11"
- board text added: "Col12"
- board text added: "Col13"
- board text added: "Col14"
- board text added: "Col15"
- board text added: "Row0"
- board text added: "Row1"
- board text added: "Row2"
- board text added: "Row7"
- board text removed: "MATHilda"
Changed lines of the file:
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@@
   (gr_line (start 208.68 99.945) (end 208.68 64.395) (layer "User.9") (width 0.15))
   (gr_line (start 305.79 3.3) (end 407.79 3.3) (layer "User.9") (width 0.15))
+  (gr_text "Row0" (at 79.29 77.99) (layer "B.SilkS")
+    (effects (font (size 0.4 0.4) (thickness 0.1)) (justify mirror))
+  )
+  (gr_text "Row1" (at 108.03 89.99) (layer "B.SilkS")
+    (effects (font (size 0.4 0.4) (thickness 0.1)) (justify mirror))
+  )
   (gr_text "GND\n" (at 82.32 72.05) (layer "B.SilkS")
     (effects (font (size 0.6 0.6) (thickness 0.15)) (justify mirror))
   )
-  (gr_text "Col3" (at 86.65 101.39 90) (layer "B.SilkS")
+  (gr_text "Col3" (at 86.65 101.27 90) (layer "B.SilkS")
     (effects (font (size 0.4 0.4) (thickness 0.1)) (justify mirror))
   )
-  (gr_text "Col5" (at 88.65 101.39 90) (layer "B.SilkS")
+  (gr_text "Row7" (at 108.03 85.99) (layer "B.SilkS")
+    (effects (font (size 0.4 0.4) (thickness 0.1)) (justify mirror))
+  )
+  (gr_text "Col5" (at 88.65 101.27 90) (layer "B.SilkS")
     (effects (font (size 0.4 0.4) (thickness 0.1)) (justify mirror))
   )
@@
     (effects (font (size 0.6 0.6) (thickness 0.15)) (justify mirror))
   )
-  (gr_text "Col3" (at 84.65 101.39 90) (layer "B.SilkS")
+  (gr_text "Col10" (at 98.65 101.45 90) (layer "B.SilkS")
     (effects (font (size 0.4 0.4) (thickness 0.1)) (justify mirror))
   )
-  (gr_text "Col9\n" (at 96.65 101.39 90) (layer "B.SilkS")
+  (gr_text "Col3" (at 84.65 101.27 90) (layer "B.SilkS")
     (effects (font (size 0.4 0.4) (thickness 0.1)) (justify mirror))
   )
-  (gr_text "Col6" (at 90.65 101.39 90) (layer "B.SilkS")
+  (gr_text "Col9\n" (at 96.65 101.27 90) (layer "B.SilkS")
     (effects (font (size 0.4 0.4) (thickness 0.1)) (justify mirror))
   )
-  (gr_text "Row5" (at 79.24 91.99) (layer "B.SilkS")
+  (gr_text "Col6" (at 90.65 101.27 90) (layer "B.SilkS")
+    (effects (font (size 0.4 0.4) (thickness 0.1)) (justify mirror))
+  )
+  (gr_text "Row5" (at 79.29 91.99) (layer "B.SilkS")
     (effects (font (size 0.4 0.4) (thickness 0.1)) (justify mirror))
   )
@@
     (effects (font (size 0.4 0.4) (thickness 0.1)) (justify mirror))
   )
-  (gr_text "Col3" (at 79.24 87.99) (layer "B.SilkS")
+  (gr_text "Col3" (at 79.38 87.99) (layer "B.SilkS")
     (effects (font (size 0.4 0.4) (thickness 0.1)) (justify mirror))
   )
-  (gr_text "Row4" (at 79.24 93.99) (layer "B.SilkS")
+  (gr_text "Row4" (at 79.29 93.99) (layer "B.SilkS")
+    (effects (font (size 0.4 0.4) (thickness 0.1)) (justify mirror))
+  )
+  (gr_text "Col14\n" (at 108.11 94.16) (layer "B.SilkS")
     (effects (font (size 0.4 0.4) (thickness 0.1)) (justify mirror))
   )
@@
     (effects (font (size 0.6 0.6) (thickness 0.15)) (justify mirror))
   )
-  (gr_text "Row3" (at 79.24 95.99) (layer "B.SilkS")
+  (gr_text "Col15" (at 108.11 91.99) (layer "B.SilkS")
     (effects (font (size 0.4 0.4) (thickness 0.1)) (justify mirror))
   )
-  (gr_text "Col7" (at 92.65 101.39 90) (layer "B.SilkS")
+  (gr_text "Row3" (at 79.29 95.99) (layer "B.SilkS")
     (effects (font (size 0.4 0.4) (thickness 0.1)) (justify mirror))
   )
-  (gr_text "Row6" (at 79.24 89.99) (layer "B.SilkS")
+  (gr_text "Col12\n" (at 102.65 101.45 90) (layer "B.SilkS")
+    (effects (font (size 0.4 0.4) (thickness 0.1)) (justify mirror))
+  )
+  (gr_text "Row2" (at 108.03 87.99) (layer "B.SilkS")
+    (effects (font (size 0.4 0.4) (thickness 0.1)) (justify mirror))
+  )
+  (gr_text "Col13\n" (at 108.11 95.99) (layer "B.SilkS")
+    (effects (font (size 0.4 0.4) (thickness 0.1)) (justify mirror))
+  )
+  (gr_text "Col7" (at 92.65 101.27 90) (layer "B.SilkS")
+    (effects (font (size 0.4 0.4) (thickness 0.1)) (justify mirror))
+  )
+  (gr_text "Row6" (at 79.29 89.99) (layer "B.SilkS")
     (effects (font (size 0.4 0.4) (thickness 0.1)) (justify mirror))
   )
@@
     (effects (font (size 0.6 0.6) (thickness 0.15)) (justify mirror))
   )
-  (gr_text "Col2" (at 79.24 83.99) (layer "B.SilkS")
+  (gr_text "Col2" (at 79.38 83.99) (layer "B.SilkS")
     (effects (font (size 0.4 0.4) (thickness 0.1)) (justify mirror))
   )
-  (gr_text "Col1" (at 79.24 85.99) (layer "B.SilkS")
+  (gr_text "Col1" (at 79.38 85.99) (layer "B.SilkS")
     (effects (font (size 0.4 0.4) (thickness 0.1)) (justify mirror))
   )
-  (gr_text "Col8" (at 94.65 101.39 90) (layer "B.SilkS")
+  (gr_text "Col8" (at 94.65 101.27 90) (layer "B.SilkS")
+    (effects (font (size 0.4 0.4) (thickness 0.1)) (justify mirror))
+  )
+  (gr_text "Col11" (at 100.65 101.45 90) (layer "B.SilkS")
     (effects (font (size 0.4 0.4) (thickness 0.1)) (justify mirror))
   )
@@
     (effects (font (size 0.6 0.6) (thickness 0.15)) (justify mirror))
   )
-  (gr_text "MATHilda" (at 56.4 61.64) (layer "F.SilkS")
-    (effects (font (size 4 4) (thickness 1)))
-  )
   (gr_text "Powered by      ilda" (at 93.55 95.33) (layer "F.SilkS")

Commit message: V2 Updates
Other:
- board text removed: "Charging Module"
- board text removed: "LIPO Battery"
- board text removed: "Raspberry Pi Zero"
Changed lines of the file:
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@@
       (drillshape 0)
       (scaleselection 1)
-      (outputdirectory "../../../../403_Pres/Images/")
+      (outputdirectory "Gerber/")
     )
   )
@@
   (gr_line (start 79.65 64.21) (end 107.65 64.21) (layer "Edge.Cuts") (width 0.2))
   (gr_line (start 209.65 106.21) (end 209.65 108.21) (layer "Edge.Cuts") (width 0.2))
-  (gr_arc (start 251.21 133.59) (mid 250.624227 135.004245) (end 249.21 135.59) (layer "User.9") (width 0.2))
-  (gr_line (start 177.49 94.91) (end 177.49 64.41) (layer "User.9") (width 0.15))
-  (gr_circle (center 213.21 133.59) (end 214.21 133.59) (layer "User.9") (width 0.2) (fill none))
-  (gr_circle (center 37.76 75.21) (end 38.76 75.21) (layer "User.9") (width 0.2) (fill none))
-  (gr_line (start 37.76 133.21) (end 73.76 133.21) (layer "User.9") (width 0.2))
-  (gr_line (start 75.76 131.21) (end 75.76 75.21) (layer "User.9") (width 0.2))
-  (gr_line (start 180.28 64.395) (end 180.28 99.895) (layer "User.9") (width 0.15))
   (gr_line (start 407.79 63.3) (end 407.79 3.3) (layer "User.9") (width 0.15))
-  (gr_arc (start 73.76 73.21) (mid 75.174214 73.795786) (end 75.76 75.21) (layer "User.9") (width 0.2))
-  (gr_circle (center 73.76 75.21) (end 74.76 75.21) (layer "User.9") (width 0.2) (fill none))
-  (gr_arc (start 37.76 133.21) (mid 36.345786 132.624214) (end 35.76 131.21) (layer "User.9") (width 0.2))
-  (gr_line (start 211.21 77.59) (end 211.21 133.59) (layer "User.9") (width 0.2))
-  (gr_line (start 217.86 131.13) (end 247.86 131.13) (layer "User.9") (width 0.15))
-  (gr_arc (start 35.76 75.21) (mid 36.345816 73.795816) (end 37.76 73.21) (layer "User.9") (width 0.2))
   (gr_line (start 305.79 63.3) (end 305.79 3.3) (layer "User.9") (width 0.15))
-  (gr_line (start 213.21 135.59) (end 249.21 135.59) (layer "User.9") (width 0.2))
-  (gr_line (start 217.86 96.13) (end 247.86 96.13) (layer "User.9") (width 0.15))
   (gr_line (start 305.79 63.3) (end 407.79 63.3) (layer "User.9") (width 0.15))
-  (gr_arc (start 213.21 135.59) (mid 211.795783 135.00422) (end 211.21 133.59) (layer "User.9") (width 0.2))
-  (gr_arc (start 249.21 75.59) (mid 250.62421 76.175793) (end 251.21 77.59) (layer "User.9") (width 0.2))
-  (gr_circle (center 213.21 77.59) (end 214.21 77.59) (layer "User.9") (width 0.2) (fill none))
-  (gr_line (start 111.49 94.91) (end 111.49 64.41) (layer "User.9") (width 0.15))
-  (gr_line (start 73.76 73.21) (end 37.76 73.21) (layer "User.9") (width 0.2))
-  (gr_line (start 111.363 94.91) (end 177.363 94.91) (layer "User.9") (width 0.15))
-  (gr_arc (start 75.76 131.21) (mid 75.174243 132.624243) (end 73.76 133.21) (layer "User.9") (width 0.2))
-  (gr_arc (start 211.21 77.59) (mid 211.7958 76.175818) (end 213.21 75.59) (layer "User.9") (width 0.2))
-  (gr_circle (center 37.76 131.21) (end 38.76 131.21) (layer "User.9") (width 0.2) (fill none))
-  (gr_line (start 249.21 75.59) (end 213.21 75.59) (layer "User.9") (width 0.2))
-  (gr_line (start 35.76 75.21) (end 35.76 131.21) (layer "User.9") (width 0.2))
-  (gr_circle (center 73.76 131.21) (end 74.76 131.21) (layer "User.9") (width 0.2) (fill none))
-  (gr_line (start 180.28 99.945) (end 208.68 99.945) (layer "User.9") (width 0.15))
-  (gr_line (start 111.49 64.41) (end 177.49 64.41) (layer "User.9") (width 0.15))
-  (gr_line (start 247.86 96.13) (end 247.86 131.13) (layer "User.9") (width 0.15))
-  (gr_line (start 180.28 64.405) (end 208.68 64.395) (layer "User.9") (width 0.15))
-  (gr_line (start 217.86 96.13) (end 217.86 131.13) (layer "User.9") (width 0.15))
-  (gr_circle (center 249.21 133.59) (end 250.21 133.59) (layer "User.9") (width 0.2) (fill none))
-  (gr_line (start 251.21 133.59) (end 251.21 77.59) (layer "User.9") (width 0.2))
-  (gr_circle (center 249.21 77.59) (end 250.21 77.59) (layer "User.9") (width 0.2) (fill none))
-  (gr_line (start 208.68 99.945) (end 208.68 64.395) (layer "User.9") (width 0.15))
   (gr_line (start 305.79 3.3) (end 407.79 3.3) (layer "User.9") (width 0.15))
   (gr_text "Row0" (at 79.29 77.99) (layer "B.SilkS")
@@
     (effects (font (size 1 1) (thickness 0.15)))
   )
-  (gr_text "Raspberry Pi Zero" (at 144.4265 79.66) (layer "User.9")
-    (effects (font (size 4 4) (thickness 0.15)))
-  )
   (gr_text "Display" (at 356.79 33.3) (layer "User.9")
     (effects (font (size 6 6) (thickness 0.15)))
   )
-  (gr_text "Charging Module\n" (at 194.14 82.145 90) (layer "User.9")
-    (effects (font (size 2 2) (thickness 0.15)))
-  )
-  (gr_text "LIPO Battery" (at 232.86 113.63 270) (layer "User.9")
-    (effects (font (size 3.6 3.6) (thickness 0.15)))
-  )
   (segment (start 92.65 73.325) (end 93.145 72.83) (width 0.8) (layer "B.Cu") (net 1))
   (segment (start 92.35 68.34) (end 93.145 69.135) (width 0.8) (layer "B.Cu") (net 1))
@@
     )
   )
-  (group "" (id 2f294de1-352a-42fc-943f-6793c56e77f0)
-    (members
-      3c398f38-0d9a-4978-b0a3-bd2faaea9705
-      5dfb8f93-e4f6-47ec-b627-4e5b0e548ab4
-      db4eca14-2b11-4a86-a337-7c2c951e01de
-      df1dfced-018d-4945-a3a7-025f4b9800ea
-      fd313ea1-2c0b-48ad-82be-b04c1bef9db0
-    )
-  )
   (group "" (id 66c97e6e-49ff-48b7-938e-a4ee6251c17f)
     (members
@@
     )
   )
-  (group "" (id 6cdd37b1-3c6e-4bec-bf59-dbe20cb30a7e)
-    (members
-      013fa9f5-22df-4088-a5bf-a097e13fea35
-      0732c0f8-6283-4114-8dd3-feb637718bd7
-      37775d30-1156-40d6-8928-8924d50621ce
-      5d55b0c1-668a-4e06-8ee8-e378f0fc7743
-      66e27fc5-0860-4dd5-aebc-90b3df6b29fe
-      680b8d24-be2e-4ddf-8ec2-9463efd7a4ae
-      74d73936-9928-415a-9d9b-1eacf862e9ee
-      a7e049f8-3a2b-41cb-bdfb-3b2d403cc30d
-      ab07eea8-f921-444e-bf62-92cca940224d
-      e1ea9f5f-d748-41b3-b2b6-0bc6f6dab8fe
-      e51b5a42-8d8a-4e65-877e-da0990738977
-      e703904b-8a61-42a3-bf23-c3181570f7db
-    )
-  )
-  (group "" (id 7a56d729-369d-4ee3-9fc8-868106ccc5d8)
-    (members
-      099ef8bf-b49f-4a03-af86-1e3a529a6537
-      0a2c1709-7040-4dd5-b7d8-dcfbed282d1d
-      0d3b6537-52c9-4aaa-b886-bdb03e85f690
-      1780692f-b7e9-43b1-b28c-d49ad6524cc6
-      1be3218b-78a4-4a32-b203-7fb265557b76
-      2bb9f075-7376-4f69-b3d1-9028b05c5ed8
-      4a915a64-ba9f-4153-9401-06593582af85
-      78fc91ae-c143-4d31-9cb8-5f20cceea8e4
-      934b1bdf-6c7e-4438-bd5f-f2dffe789710
-      a924d3d2-4d80-453c-8615-2c9f999dfdc7
-      ad297327-5038-46de-8991-437406beeafb
-      bb0bb8f5-2d61-44ba-9191-490bf9ea268c
-    )
-  )
-  (group "" (id aa0e1af7-2545-4753-91f3-6632eb9058c8)
-    (members
-      0f7d0ac4-220d-45c7-90c0-94acd25b5c7b
-      d02fd31a-b3c1-4bd4-a1d1-c4c9363c89da
-      d48878b7-9cc6-440a-b392-f0dc0056b3b5
-      dd7c40a7-1fa8-4d8e-a27a-8c410219cf11
-      e746b6b4-1244-4830-bb75-442261c64091
-    )
-  )
-  (group "" (id d089ab1c-04dd-4db4-9e6c-f6b4641af526)
-    (members
-      04623b2c-141f-45d5-b606-ca93697b2487
-      13dfcd3b-0f2c-4213-9f4e-8f701fa294b3
-      77579cb8-2a2a-4b3b-b46a-2d485cbe99fc
-      800ae900-e504-44d1-9915-4a39b31fd276
-      d7745b46-711a-4d08-adf4-5420ad94e1d9
-    )
-  )

Commit message: V2 Updates
Other:
- board text removed: "Display"
Changed lines of the file:
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@@
       (sketchpadsonfab false)
       (subtractmaskfromsilk false)
-      (outputformat 4)
+      (outputformat 1)
       (mirror false)
       (drillshape 0)
@@
   (gr_line (start 79.65 64.21) (end 107.65 64.21) (layer "Edge.Cuts") (width 0.2))
   (gr_line (start 209.65 106.21) (end 209.65 108.21) (layer "Edge.Cuts") (width 0.2))
-  (gr_line (start 407.79 63.3) (end 407.79 3.3) (layer "User.9") (width 0.15))
-  (gr_line (start 305.79 63.3) (end 305.79 3.3) (layer "User.9") (width 0.15))
-  (gr_line (start 305.79 63.3) (end 407.79 63.3) (layer "User.9") (width 0.15))
-  (gr_line (start 305.79 3.3) (end 407.79 3.3) (layer "User.9") (width 0.15))
   (gr_text "Row0" (at 79.29 77.99) (layer "B.SilkS")
     (effects (font (size 0.4 0.4) (thickness 0.1)) (justify mirror))
@@
     (effects (font (size 0.6 0.6) (thickness 0.15)) (justify mirror))
   )
+  (gr_text "Row5" (at 79.29 91.99) (layer "B.SilkS")
+    (effects (font (size 0.4 0.4) (thickness 0.1)) (justify mirror))
+  )
   (gr_text "Col10" (at 98.65 101.45 90) (layer "B.SilkS")
     (effects (font (size 0.4 0.4) (thickness 0.1)) (justify mirror))
@@
     (effects (font (size 0.4 0.4) (thickness 0.1)) (justify mirror))
   )
-  (gr_text "Row5" (at 79.29 91.99) (layer "B.SilkS")
-    (effects (font (size 0.4 0.4) (thickness 0.1)) (justify mirror))
-  )
   (gr_text "y_out" (at 79.24 81.99) (layer "B.SilkS")
     (effects (font (size 0.4 0.4) (thickness 0.1)) (justify mirror))
@@
     (effects (font (size 1 1) (thickness 0.15)))
   )
-  (gr_text "Display" (at 356.79 33.3) (layer "User.9")
-    (effects (font (size 6 6) (thickness 0.15)))
-  )
   (segment (start 92.65 73.325) (end 93.145 72.83) (width 0.8) (layer "B.Cu") (net 1))
   (segment (start 92.35 68.34) (end 93.145 69.135) (width 0.8) (layer "B.Cu") (net 1))
@@
     )
   )
-  (group "" (id 66c97e6e-49ff-48b7-938e-a4ee6251c17f)
-    (members
-      1584c8fa-3039-4079-bc47-1b5b80c5367b
-      51a43830-14f6-4a46-bf85-57c9e1423de5
-      5ea7a41f-f860-4daa-a540-9fbd6ef6f536
-      66038996-a46c-4850-9f62-775499845652
-      ffb50673-07e1-4205-90a4-093bb79a93ea
-    )
-  )
