File: KiCAD_PCB/Calculator_KeyPad_PCB/KeyPad/KeyPad.kicad_pcb (KiCad board)
At the start: 2 copper layers, 45 x 60 mm, 43 parts, among them J1 5034801000, SW1 SW_SPST, SW10 SW_SPST, SW11 SW_SPST, SW12 SW_SPST, SW13 SW_SPST, SW14 SW_SPST, SW15 SW_SPST, SW16 SW_SPST, SW17 SW_SPST, SW18 SW_SPST, SW19 SW_SPST, SW2 SW_SPST, SW20 SW_SPST, SW21 SW_SPST, SW3 SW_SPST, SW4 SW_SPST, SW5 SW_SPST, SW6 SW_SPST, SW7 SW_SPST, SW8 SW_SPST, SW9 SW_SPST

Commit message: V2 Updates
Parts:
- J1: moved to B.Cu
- moved J1 26.3 mm to (135.9, 103.5), turned to 90 degrees
Connections:
- J1 pad 1: /Col15 -> /Row7
- J1 pad 10: /Row7 -> /Col15
- J1 pad 2: /Col14 -> /Row6
- J1 pad 3: /Col13 -> /Row5
- J1 pad 4: /Row1 -> /Row4
- J1 pad 5: /Row2 -> /Row3
- J1 pad 6: /Row3 -> /Row2
- J1 pad 7: /Row4 -> /Row1
- J1 pad 8: /Row5 -> /Col13
- J1 pad 9: /Row6 -> /Col14
Routing:
- net /Col15: track 62.2 -> 99.9 mm
- net /Row1: track 27.4 -> 59.1 mm
- net /Row2: track 27.4 -> 51.4 mm
- net /Col14: track 62.2 -> 86.2 mm
- net /Row3: track 27.4 -> 43.7 mm
- net /Col13: track 62.2 -> 73.7 mm
- net /Row4: track 27.4 -> 36.7 mm

Commit message: V2 Updates
Routing:
- net /Col15: track 99.9 -> 130.1 mm
- net /Col13: track 73.7 -> 99.0 mm
- net /Row7: track 27.4 -> 50.6 mm
- net /Row6: track 27.4 -> 42.9 mm
- net /Col14: track 86.2 -> 98.0 mm
- net /Row5: track 27.4 -> 35.3 mm
Changed lines of the file:
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@@
   (segment (start 144.9336 117.3208) (end 141.3522 117.3208) (width 0.15) (layer "B.Cu") (net 1))
   (segment (start 153.1134 116) (end 146.2544 116) (width 0.15) (layer "B.Cu") (net 1))
+  (segment (start 137.63 116) (end 141.15 116) (width 0.15) (layer "B.Cu") (net 1))
   (segment (start 146.2544 116) (end 144.9336 117.3208) (width 0.15) (layer "B.Cu") (net 1))
   (segment (start 165.0134 116.01) (end 158.1544 116.01) (width 0.15) (layer "B.Cu") (net 1))
@@
   (segment (start 156.8336 117.3308) (end 153.2522 117.3308) (width 0.15) (layer "B.Cu") (net 1))
   (segment (start 153.05 117.1266) (end 153.05 116.01) (width 0.15) (layer "B.Cu") (net 1))
+  (segment (start 136.77 105.27) (end 137.39 105.89) (width 0.15) (layer "B.Cu") (net 1))
+  (segment (start 137.39 115.76) (end 137.63 116) (width 0.15) (layer "B.Cu") (net 1))
+  (segment (start 135.92 105.27) (end 136.77 105.27) (width 0.15) (layer "B.Cu") (net 1))
+  (segment (start 137.39 105.89) (end 137.39 115.76) (width 0.15) (layer "B.Cu") (net 1))
   (segment (start 141.15 117.1166) (end 141.15 116) (width 0.15) (layer "B.Cu") (net 1))
   (segment (start 135.92 102.77) (end 136.58 102.77) (width 0.15) (layer "B.Cu") (net 3))
@@
   (segment (start 146.6924 98.5382) (end 144.719 98.5382) (width 0.15) (layer "B.Cu") (net 10))
   (segment (start 146.2544 108) (end 144.9336 109.3208) (width 0.15) (layer "B.Cu") (net 11))
+  (segment (start 137.75 107.68) (end 138.07 108) (width 0.15) (layer "B.Cu") (net 11))
   (segment (start 141.15 109.1166) (end 141.15 108) (width 0.15) (layer "B.Cu") (net 11))
   (segment (start 153.05 109.1266) (end 153.05 108.01) (width 0.15) (layer "B.Cu") (net 11))
   (segment (start 158.1544 108.01) (end 156.8336 109.3308) (width 0.15) (layer "B.Cu") (net 11))
   (segment (start 156.8336 109.3308) (end 153.2522 109.3308) (width 0.15) (layer "B.Cu") (net 11))
+  (segment (start 137.05 104.77) (end 137.75 105.47) (width 0.15) (layer "B.Cu") (net 11))
+  (segment (start 138.07 108) (end 141.15 108) (width 0.15) (layer "B.Cu") (net 11))
   (segment (start 144.9336 109.3208) (end 141.3522 109.3208) (width 0.15) (layer "B.Cu") (net 11))
   (segment (start 153.1134 108) (end 146.2544 108) (width 0.15) (layer "B.Cu") (net 11))
   (segment (start 141.3522 109.3208) (end 141.149 109.1176) (width 0.15) (layer "B.Cu") (net 11))
+  (segment (start 135.92 104.77) (end 137.05 104.77) (width 0.15) (layer "B.Cu") (net 11))
   (segment (start 153.2522 109.3308) (end 153.049 109.1276) (width 0.15) (layer "B.Cu") (net 11))
   (segment (start 165.0134 108.01) (end 158.1544 108.01) (width 0.15) (layer "B.Cu") (net 11))
+  (segment (start 137.75 105.47) (end 137.75 107.68) (width 0.15) (layer "B.Cu") (net 11))
   (segment (start 156.8336 125.3308) (end 153.2522 125.3308) (width 0.15) (layer "B.Cu") (net 13))
   (segment (start 141.15 125.1166) (end 141.15 124) (width 0.15) (layer "B.Cu") (net 13))
   (segment (start 153.1134 124) (end 146.2544 124) (width 0.15) (layer "B.Cu") (net 13))
   (segment (start 158.1544 124.01) (end 156.8336 125.3308) (width 0.15) (layer "B.Cu") (net 13))
+  (segment (start 137.04048 106.034776) (end 137.04048 123.75048) (width 0.15) (layer "B.Cu") (net 13))
+  (segment (start 137.29 124) (end 141.15 124) (width 0.15) (layer "B.Cu") (net 13))
   (segment (start 165.0134 124.01) (end 158.1544 124.01) (width 0.15) (layer "B.Cu") (net 13))
   (segment (start 153.05 125.1266) (end 153.05 124.01) (width 0.15) (layer "B.Cu") (net 13))
+  (segment (start 136.775704 105.77) (end 137.04048 106.034776) (width 0.15) (layer "B.Cu") (net 13))
+  (segment (start 137.04048 123.75048) (end 137.29 124) (width 0.15) (layer "B.Cu") (net 13))
   (segment (start 144.9336 125.3208) (end 141.3522 125.3208) (width 0.15) (layer "B.Cu") (net 13))
   (segment (start 141.3522 125.3208) (end 141.149 125.1176) (width 0.15) (layer "B.Cu") (net 13))
+  (segment (start 135.92 105.77) (end 136.775704 105.77) (width 0.15) (layer "B.Cu") (net 13))
   (segment (start 146.2544 124) (end 144.9336 125.3208) (width 0.15) (layer "B.Cu") (net 13))
   (segment (start 153.2522 125.3308) (end 153.049 125.1276) (width 0.15) (layer "B.Cu") (net 13))
@@
   (segment (start 148.204 101.706) (end 148.204 101.475) (width 0.15) (layer "F.Cu") (net 29))
   (segment (start 147.96 85.46) (end 148.204 85.216) (width 0.15) (layer "F.Cu") (net 29))
-  (segment (start 138.59 67.87) (end 137.17 69.29) (width 0.15) (layer "B.Cu") (net 29))
-  (segment (start 146.61 68.14) (end 146.34 67.87) (width 0.15) (layer "B.Cu") (net 29))
-  (segment (start 146.34 67.87) (end 138.59 67.87) (width 0.15) (layer "B.Cu") (net 29))
-  (segment (start 146.61 69.46) (end 146.61 68.14) (width 0.15) (layer "B.Cu") (net 29))
+  (segment (start 135.07 102.27) (end 134.640481 101.840481) (width 0.15) (layer "B.Cu") (net 29))
+  (segment (start 134.640481 101.840481) (end 134.640481 101.475223) (width 0.15) (layer "B.Cu") (net 29))
+  (segment (start 134.900481 100.395223) (end 135.727852 99.567852) (width 0.15) (layer "B.Cu") (net 29))
+  (segment (start 134.845225 100.45048) (end 134.900481 100.395223) (width 0.15) (layer "B.Cu") (net 29))
+  (segment (start 135.92 102.27) (end 135.07 102.27) (width 0.15) (layer "B.Cu") (net 29))
+  (segment (start 135.727852 99.567852) (end 135.727852 69.333558) (width 0.15) (layer "B.Cu") (net 29))
+  (segment (start 134.640481 100.655223) (end 134.845225 100.45048) (width 0.15) (layer "B.Cu") (net 29))
+  (segment (start 134.640481 101.475223) (end 134.640481 100.655223) (width 0.15) (layer "B.Cu") (net 29))
+  (segment (start 135.727852 69.333558) (end 137.350704 67.710705) (width 0.15) (layer "B.Cu") (net 29))
   (segment (start 171.6634 109.46) (end 171.989 109.46) (width 0.15) (layer "F.Cu") (net 30))
   (segment (start 171.736 69.46) (end 170.41 69.46) (width 0.15) (layer "F.Cu") (net 30))
@@
   (segment (start 172.004 93.216) (end 172.004 85.676) (width 0.15) (layer "F.Cu") (net 30))
   (segment (start 171.6634 101.46) (end 171.989 101.46) (width 0.15) (layer "F.Cu") (net 30))
-  (segment (start 170.41 68.14) (end 169.44 67.17) (width 0.15) (layer "B.Cu") (net 30))
-  (segment (start 170.41 69.46) (end 170.41 68.14) (width 0.15) (layer "B.Cu") (net 30))
-  (segment (start 135.92 100.3) (end 135.92 101.27) (width 0.15) (layer "B.Cu") (net 30))
-  (segment (start 138.301408 67.17) (end 136.47096 69.00045) (width 0.15) (layer "B.Cu") (net 30))
-  (segment (start 136.47096 69.00045) (end 136.470961 69.290002) (width 0.15) (layer "B.Cu") (net 30))
-  (segment (start 169.44 67.17) (end 138.301408 67.17) (width 0.15) (layer "B.Cu") (net 30))
+  (segment (start 170.41 68.14) (end 170.41 69.46) (width 0.15) (layer "B.Cu") (net 30))
+  (segment (start 136.45048 69.59952) (end 138.06 67.99) (width 0.15) (layer "B.Cu") (net 30))
+  (segment (start 135.92 100.364296) (end 136.45048 99.833816) (width 0.15) (layer "B.Cu") (net 30))
+  (segment (start 138.06 67.99) (end 170.26 67.99) (width 0.15) (layer "B.Cu") (net 30))
+  (segment (start 170.26 67.99) (end 170.41 68.14) (width 0.15) (layer "B.Cu") (net 30))
+  (segment (start 135.92 101.27) (end 135.92 100.364296) (width 0.15) (layer "B.Cu") (net 30))
+  (segment (start 136.45048 99.833816) (end 136.45048 69.59952) (width 0.15) (layer "B.Cu") (net 30))
   (segment (start 159.86 85.46) (end 160.104 85.216) (width 0.15) (layer "F.Cu") (net 31))
   (segment (start 160.104 117.216) (end 159.86 117.46) (width 0.15) (layer "F.Cu") (net 31))
@@
   (segment (start 159.836 69.46) (end 158.51 69.46) (width 0.15) (layer "F.Cu") (net 31))
   (segment (start 159.86 77.46) (end 160.104 77.216) (width 0.15) (layer "F.Cu") (net 31))
-  (segment (start 158.51 69.46) (end 158.51 68.13) (width 0.15) (layer "B.Cu") (net 31))
-  (segment (start 157.900481 67.520481) (end 138.445223 67.520481) (width 0.15) (layer "B.Cu") (net 31))
-  (segment (start 138.445223 67.520481) (end 136.82048 69.145225) (width 0.15) (layer "B.Cu") (net 31))
-  (segment (start 158.51 68.13) (end 157.900481 67.520481) (width 0.15) (layer "B.Cu") (net 31))
+  (segment (start 136.305705 69.25) (end 137.64 67.915705) (width 0.15) (layer "B.Cu") (net 31))
+  (segment (start 135.92 101.77) (end 135.14 101.77) (width 0.15) (layer "B.Cu") (net 31))
+  (segment (start 136.10096 99.55) (end 136.100961 69.454743) (width 0.15) (layer "B.Cu") (net 31))
+  (segment (start 136.100961 69.454743) (end 136.305705 69.25) (width 0.15) (layer "B.Cu") (net 31))
+  (segment (start 134.99 100.8) (end 135.25 100.54) (width 0.15) (layer "B.Cu") (net 31))
+  (segment (start 137.64 67.915705) (end 137.64 67.91) (width 0.15) (layer "B.Cu") (net 31))
+  (segment (start 136.10096 99.55) (end 136.100481 99.549521) (width 0.15) (layer "B.Cu") (net 31))
+  (segment (start 135.71 100.08) (end 136.10096 99.68904) (width 0.15) (layer "B.Cu") (net 31))
+  (segment (start 136.10096 99.68904) (end 136.10096 99.55) (width 0.15) (layer "B.Cu") (net 31))
+  (segment (start 134.99 101.62) (end 134.99 100.97) (width 0.15) (layer "B.Cu") (net 31))
+  (segment (start 135.14 101.77) (end 134.99 101.62) (width 0.15) (layer "B.Cu") (net 31))
+  (segment (start 135.25 100.54) (end 135.71 100.08) (width 0.15) (layer "B.Cu") (net 31))
+  (segment (start 134.99 100.97) (end 134.99 100.8) (width 0.15) (layer "B.Cu") (net 31))
   (group "" (id 175babef-1062-40f1-b84d-974a7c04386b)
     (members
