File: KiCAD_PCB/Calculator_KeyPad_PCB/KeyPad/KeyPad.kicad_pcb (KiCad board)
At the start: 2 copper layers, 45 x 60 mm, 43 parts, among them J1 5034801000, SW1 SW_SPST, SW10 SW_SPST, SW11 SW_SPST, SW12 SW_SPST, SW13 SW_SPST, SW14 SW_SPST, SW15 SW_SPST, SW16 SW_SPST, SW17 SW_SPST, SW18 SW_SPST, SW19 SW_SPST, SW2 SW_SPST, SW20 SW_SPST, SW21 SW_SPST, SW3 SW_SPST, SW4 SW_SPST, SW5 SW_SPST, SW6 SW_SPST, SW7 SW_SPST, SW8 SW_SPST, SW9 SW_SPST

Commit message: V2 Updates
Routing:
- net Net-(D15-Pad2): track 0.00 -> 3.55 mm
- net Net-(D8-Pad2): track 0.00 -> 3.55 mm
- net Net-(D1-Pad2): track 0.00 -> 3.55 mm

Commit message: V2 Updates
Connections:
- net Net-(J1-PadS1) renamed GND
Routing:
- net /Col14: track 98.0 -> 121.1 mm, vias 0 -> 1
- net /Col13: track 99.0 -> 110.6 mm, vias 0 -> 1
- net GND: track 0.00 -> 1.46 mm, vias 0 -> 2
- added copper zone on F.Cu, net GND
Changed lines of the file:
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@@
   (net 30 "/Col15")
   (net 31 "/Col14")
-  (net 32 "Net-(J1-PadS1)")
+  (net 32 "GND")
   (footprint "KSA_Switch:KSA1M331LFT" (layer "F.Cu")
     (at 154.7 88 90)
@@
       (net 30 "/Col15") (pinfunction "10") (pintype "passive"))
     (pad "S1" smd rect locked (at -3.04 -2.65 90) (size 0.3 1) (layers "B.Cu" "B.Paste" "B.Mask")
-      (net 32 "Net-(J1-PadS1)") (pinfunction "SHIELD") (pintype "passive"))
+      (net 32 "GND") (pinfunction "SHIELD") (pintype "passive"))
     (pad "S2" smd rect locked (at 3.04 -2.65 90) (size 0.3 1) (layers "B.Cu" "B.Paste" "B.Mask")
-      (net 32 "Net-(J1-PadS1)") (pinfunction "SHIELD") (pintype "passive"))
+      (net 32 "GND") (pinfunction "SHIELD") (pintype "passive"))
     (model "C:/Users/natha/Documents/GitHub/Design/KiCAD_PCB/Calculator_PCB_Components/3D_Models/130094464-659-503480-1000/503480-1000.stp"
       (offset (xyz 0 -3.3 0))
@@
   (segment (start 148.204 77.856) (end 148.204 77.7544) (width 0.15) (layer "F.Cu") (net 29))
   (segment (start 148.204 85.095) (end 148.204 77.856) (width 0.15) (layer "F.Cu") (net 29))
+  (segment (start 146.61 67.99) (end 146.61 69.46) (width 0.15) (layer "F.Cu") (net 29))
   (segment (start 148.204 69.728) (end 147.936 69.46) (width 0.15) (layer "F.Cu") (net 29))
+  (segment (start 145.43 66.81) (end 146.61 67.99) (width 0.15) (layer "F.Cu") (net 29))
   (segment (start 147.96 77.462) (end 148.204 77.706) (width 0.15) (layer "F.Cu") (net 29))
   (segment (start 146.61 77.46) (end 147.8634 77.46) (width 0.15) (layer "F.Cu") (net 29))
@@
   (segment (start 148.204 93.475) (end 148.204 93.216) (width 0.15) (layer "F.Cu") (net 29))
   (segment (start 147.8634 77.46) (end 148.189 77.46) (width 0.15) (layer "F.Cu") (net 29))
+  (segment (start 144.885 66.81) (end 145.43 66.81) (width 0.15) (layer "F.Cu") (net 29))
   (segment (start 148.204 101.216) (end 148.204 93.706) (width 0.15) (layer "F.Cu") (net 29))
   (segment (start 148.204 101.706) (end 148.204 101.475) (width 0.15) (layer "F.Cu") (net 29))
   (segment (start 147.96 85.46) (end 148.204 85.216) (width 0.15) (layer "F.Cu") (net 29))
+  (via (at 144.885 66.81) (size 0.8) (drill 0.4) (layers "F.Cu" "B.Cu") (net 29))
+  (segment (start 143.814038 67.290962) (end 144.295 66.81) (width 0.15) (layer "B.Cu") (net 29))
+  (segment (start 134.640481 101.840481) (end 134.640481 100.655223) (width 0.15) (layer "B.Cu") (net 29))
   (segment (start 135.07 102.27) (end 134.640481 101.840481) (width 0.15) (layer "B.Cu") (net 29))
-  (segment (start 134.640481 101.840481) (end 134.640481 101.475223) (width 0.15) (layer "B.Cu") (net 29))
+  (segment (start 138.06 67.290962) (end 143.814038 67.290962) (width 0.15) (layer "B.Cu") (net 29))
+  (segment (start 135.727852 69.333558) (end 137.350704 67.710705) (width 0.15) (layer "B.Cu") (net 29))
+  (segment (start 137.350704 67.710705) (end 137.350704 67.699296) (width 0.15) (layer "B.Cu") (net 29))
+  (segment (start 135.727852 99.567852) (end 135.727852 69.333558) (width 0.15) (layer "B.Cu") (net 29))
+  (segment (start 137.759039 67.290961) (end 138.06 67.290962) (width 0.15) (layer "B.Cu") (net 29))
+  (segment (start 144.295 66.81) (end 144.885 66.81) (width 0.15) (layer "B.Cu") (net 29))
+  (segment (start 135.92 102.27) (end 135.07 102.27) (width 0.15) (layer "B.Cu") (net 29))
   (segment (start 134.900481 100.395223) (end 135.727852 99.567852) (width 0.15) (layer "B.Cu") (net 29))
-  (segment (start 134.845225 100.45048) (end 134.900481 100.395223) (width 0.15) (layer "B.Cu") (net 29))
-  (segment (start 135.92 102.27) (end 135.07 102.27) (width 0.15) (layer "B.Cu") (net 29))
-  (segment (start 135.727852 99.567852) (end 135.727852 69.333558) (width 0.15) (layer "B.Cu") (net 29))
-  (segment (start 134.640481 100.655223) (end 134.845225 100.45048) (width 0.15) (layer "B.Cu") (net 29))
-  (segment (start 134.640481 101.475223) (end 134.640481 100.655223) (width 0.15) (layer "B.Cu") (net 29))
-  (segment (start 135.727852 69.333558) (end 137.350704 67.710705) (width 0.15) (layer "B.Cu") (net 29))
+  (segment (start 137.350704 67.699296) (end 137.759039 67.290961) (width 0.15) (layer "B.Cu") (net 29))
+  (segment (start 134.640481 100.655223) (end 134.900481 100.395223) (width 0.15) (layer "B.Cu") (net 29))
   (segment (start 171.6634 109.46) (end 171.989 109.46) (width 0.15) (layer "F.Cu") (net 30))
   (segment (start 171.736 69.46) (end 170.41 69.46) (width 0.15) (layer "F.Cu") (net 30))
@@
   (segment (start 160.104 93.706) (end 160.104 93.475) (width 0.15) (layer "F.Cu") (net 31))
   (segment (start 159.7634 109.46) (end 160.089 109.46) (width 0.15) (layer "F.Cu") (net 31))
+  (segment (start 157.68 67.16) (end 157.17 67.16) (width 0.15) (layer "F.Cu") (net 31))
   (segment (start 160.104 101.475) (end 160.104 101.216) (width 0.15) (layer "F.Cu") (net 31))
   (segment (start 158.51 109.46) (end 159.7634 109.46) (width 0.15) (layer "F.Cu") (net 31))
@@
   (segment (start 158.51 101.46) (end 159.7634 101.46) (width 0.15) (layer "F.Cu") (net 31))
   (segment (start 159.7634 93.46) (end 160.089 93.46) (width 0.15) (layer "F.Cu") (net 31))
+  (segment (start 158.51 69.46) (end 158.51 67.99) (width 0.15) (layer "F.Cu") (net 31))
   (segment (start 159.7898 85.46) (end 160.0692 85.46) (width 0.15) (layer "F.Cu") (net 31))
   (segment (start 159.86 77.462) (end 160.104 77.706) (width 0.15) (layer "F.Cu") (net 31))
@@
   (segment (start 159.86 101.46) (end 160.104 101.216) (width 0.15) (layer "F.Cu") (net 31))
   (segment (start 159.86 93.462) (end 160.104 93.706) (width 0.15) (layer "F.Cu") (net 31))
+  (segment (start 158.51 67.99) (end 157.68 67.16) (width 0.15) (layer "F.Cu") (net 31))
   (segment (start 160.104 109.706) (end 160.104 109.475) (width 0.15) (layer "F.Cu") (net 31))
   (segment (start 159.836 69.46) (end 158.51 69.46) (width 0.15) (layer "F.Cu") (net 31))
   (segment (start 159.86 77.46) (end 160.104 77.216) (width 0.15) (layer "F.Cu") (net 31))
-  (segment (start 136.305705 69.25) (end 137.64 67.915705) (width 0.15) (layer "B.Cu") (net 31))
+  (via (at 157.17 67.16) (size 0.8) (drill 0.4) (layers "F.Cu" "B.Cu") (net 31))
   (segment (start 135.92 101.77) (end 135.14 101.77) (width 0.15) (layer "B.Cu") (net 31))
+  (segment (start 137.617852 67.937852) (end 137.64 67.915705) (width 0.15) (layer "B.Cu") (net 31))
+  (segment (start 156.58 67.16) (end 156.099519 67.640481) (width 0.15) (layer "B.Cu") (net 31))
   (segment (start 136.10096 99.55) (end 136.100961 69.454743) (width 0.15) (layer "B.Cu") (net 31))
   (segment (start 136.100961 69.454743) (end 136.305705 69.25) (width 0.15) (layer "B.Cu") (net 31))
+  (segment (start 137.915223 67.640481) (end 137.617852 67.937852) (width 0.15) (layer "B.Cu") (net 31))
   (segment (start 134.99 100.8) (end 135.25 100.54) (width 0.15) (layer "B.Cu") (net 31))
   (segment (start 137.64 67.915705) (end 137.64 67.91) (width 0.15) (layer "B.Cu") (net 31))
   (segment (start 136.10096 99.55) (end 136.100481 99.549521) (width 0.15) (layer "B.Cu") (net 31))
+  (segment (start 156.099519 67.640481) (end 137.915223 67.640481) (width 0.15) (layer "B.Cu") (net 31))
   (segment (start 135.71 100.08) (end 136.10096 99.68904) (width 0.15) (layer "B.Cu") (net 31))
   (segment (start 136.10096 99.68904) (end 136.10096 99.55) (width 0.15) (layer "B.Cu") (net 31))
+  (segment (start 157.17 67.16) (end 156.58 67.16) (width 0.15) (layer "B.Cu") (net 31))
   (segment (start 134.99 101.62) (end 134.99 100.97) (width 0.15) (layer "B.Cu") (net 31))
   (segment (start 135.14 101.77) (end 134.99 101.62) (width 0.15) (layer "B.Cu") (net 31))
   (segment (start 135.25 100.54) (end 135.71 100.08) (width 0.15) (layer "B.Cu") (net 31))
+  (segment (start 136.305705 69.25) (end 137.617852 67.937852) (width 0.15) (layer "B.Cu") (net 31))
   (segment (start 134.99 100.97) (end 134.99 100.8) (width 0.15) (layer "B.Cu") (net 31))
+  (via (at 133.27 99.57) (size 0.8) (drill 0.4) (layers "F.Cu" "B.Cu") (net 32))
+  (via (at 133.27 107.47) (size 0.8) (drill 0.4) (layers "F.Cu" "B.Cu") (net 32))
+  (segment (start 133.27 106.56) (end 133.27 107.29) (width 0.2) (layer "B.Cu") (net 32))
+  (segment (start 133.27 100.48) (end 133.27 99.75) (width 0.2) (layer "B.Cu") (net 32))
+  (zone (net 32) (net_name "GND") (layer "F.Cu") (hatch edge 0.508)
+    (connect_pads (clearance 0.2))
+    (min_thickness 0.2) (filled_areas_thickness no)
+    (fill yes (thermal_gap 0.3) (thermal_bridge_width 0.3))
+    (polygon
+      (pts
+        (xy 177.2 125.98)
+        (xy 132.19 125.98)
+        (xy 132.2 65.98)
+        (xy 177.21 65.97)
+      )
+    )
+  )
   (group "" (id 175babef-1062-40f1-b84d-974a7c04386b)
     (members

Commit message: V2 Updates
Parts:
- added REF**: MountingHole_2.2mm_M2_DIN965, MountingHole:MountingHole_2.2mm_M2_DIN965, F.Cu at (175.2, 68.0)
- added REF**: MountingHole_2.2mm_M2_DIN965, MountingHole:MountingHole_2.2mm_M2_DIN965, F.Cu at (134.2, 124.0)
- added REF**: MountingHole_2.2mm_M2_DIN965, MountingHole:MountingHole_2.2mm_M2_DIN965, F.Cu at (175.2, 124.0)
- added REF**: MountingHole_2.2mm_M2_DIN965, MountingHole:MountingHole_2.2mm_M2_DIN965, F.Cu at (134.2, 68.0)
- added REF**: PinHeader_1x01_P2.00mm_Vertical, Connector_PinHeader_2.00mm:PinHeader_1x01_P2.00mm_Vertical, B.Cu at (160.6, 67.6)
Routing:
- net Net-(D7-Pad2): track 0.00 -> 3.55 mm
- net Net-(D6-Pad2): track 0.00 -> 3.55 mm
- net Net-(D5-Pad2): track 0.00 -> 3.55 mm
- net Net-(D21-Pad2): track 0.00 -> 3.55 mm
- net Net-(D20-Pad2): track 0.00 -> 3.55 mm
- net Net-(D19-Pad2): track 0.00 -> 3.55 mm
- net Net-(D14-Pad2): track 0.00 -> 3.55 mm
- net Net-(D13-Pad2): track 0.00 -> 3.55 mm
- net Net-(D12-Pad2): track 0.00 -> 3.55 mm
- net /Col14: track 121.1 -> 123.6 mm
Other:
- outline, holes or cut-outs redrawn
