File: KiCAD_PCB/Calculator_KeyPad_PCB/KeyPad/KeyPad.kicad_sch (KiCad schematic)
At the start: 43 parts, among them J1 5034801000, SW1 SW_SPST, SW10 SW_SPST, SW11 SW_SPST, SW12 SW_SPST, SW13 SW_SPST, SW14 SW_SPST, SW15 SW_SPST, SW16 SW_SPST, SW17 SW_SPST, SW18 SW_SPST, SW19 SW_SPST, SW2 SW_SPST, SW20 SW_SPST, SW21 SW_SPST, SW3 SW_SPST, SW4 SW_SPST, SW5 SW_SPST, SW6 SW_SPST, SW7 SW_SPST, SW8 SW_SPST, SW9 SW_SPST

Commit message: V2 Updates
Connections:
- net GND: now reaches J1.S1 (SHIELD), J1.S2 (SHIELD)
Other:
- moved on the sheet: J1
Changed lines of the file:
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@@
     (stroke (width 0) (type default) (color 0 0 0 0))
   )
-  (wire (pts (xy 108.712 46.99) (xy 109.728 46.99))
+  (wire (pts (xy 106.68 42.672) (xy 107.696 42.672))
     (stroke (width 0) (type default) (color 0 0 0 0))
   )
@@
     (stroke (width 0) (type default) (color 0 0 0 0))
   )
-  (wire (pts (xy 108.712 41.91) (xy 109.728 41.91))
+  (wire (pts (xy 106.68 37.592) (xy 107.696 37.592))
     (stroke (width 0) (type default) (color 0 0 0 0))
   )
@@
     (stroke (width 0) (type default) (color 0 0 0 0))
   )
+  (wire (pts (xy 105.156 47.752) (xy 107.696 47.752))
+    (stroke (width 0) (type default) (color 0 0 0 0))
+  )
   (wire (pts (xy 52.07 51.816) (xy 53.086 51.816))
     (stroke (width 0) (type default) (color 0 0 0 0))
@@
     (stroke (width 0) (type default) (color 0 0 0 0))
   )
-  (wire (pts (xy 108.712 44.45) (xy 109.728 44.45))
+  (wire (pts (xy 106.68 40.132) (xy 107.696 40.132))
     (stroke (width 0) (type default) (color 0 0 0 0))
   )
@@
     (stroke (width 0) (type default) (color 0 0 0 0))
   )
-  (wire (pts (xy 108.712 31.75) (xy 109.728 31.75))
+  (wire (pts (xy 106.68 27.432) (xy 107.696 27.432))
     (stroke (width 0) (type default) (color 0 0 0 0))
   )
@@
     (stroke (width 0) (type default) (color 0 0 0 0))
   )
-  (wire (pts (xy 108.712 39.37) (xy 109.728 39.37))
+  (wire (pts (xy 106.68 35.052) (xy 107.696 35.052))
     (stroke (width 0) (type default) (color 0 0 0 0))
   )
@@
     (stroke (width 0) (type default) (color 0 0 0 0))
   )
-  (wire (pts (xy 108.712 26.67) (xy 109.728 26.67))
+  (wire (pts (xy 106.68 22.352) (xy 107.696 22.352))
     (stroke (width 0) (type default) (color 0 0 0 0))
   )
@@
     (stroke (width 0) (type default) (color 0 0 0 0))
   )
-  (wire (pts (xy 108.712 34.29) (xy 109.728 34.29))
+  (wire (pts (xy 106.68 29.972) (xy 107.696 29.972))
     (stroke (width 0) (type default) (color 0 0 0 0))
   )
@@
     (stroke (width 0) (type default) (color 0 0 0 0))
   )
-  (wire (pts (xy 108.712 36.83) (xy 109.728 36.83))
+  (wire (pts (xy 105.156 48.768) (xy 105.156 47.752))
+    (stroke (width 0) (type default) (color 0 0 0 0))
+  )
+  (wire (pts (xy 106.68 32.512) (xy 107.696 32.512))
     (stroke (width 0) (type default) (color 0 0 0 0))
   )
@@
     (stroke (width 0) (type default) (color 0 0 0 0))
   )
-  (wire (pts (xy 108.712 24.13) (xy 109.728 24.13))
+  (wire (pts (xy 106.68 19.812) (xy 107.696 19.812))
     (stroke (width 0) (type default) (color 0 0 0 0))
   )
@@
     (stroke (width 0) (type default) (color 0 0 0 0))
   )
-  (wire (pts (xy 108.712 29.21) (xy 109.728 29.21))
+  (wire (pts (xy 106.68 24.892) (xy 107.696 24.892))
     (stroke (width 0) (type default) (color 0 0 0 0))
   )
@@
     (effects (font (size 1.6 1.6)) (justify left bottom))
   )
-  (label "Row6" (at 108.712 26.67 180)
-    (effects (font (size 1.27 1.27)) (justify right bottom))
-  )
-  (label "Col13" (at 108.712 41.91 180)
+  (label "Row6" (at 106.68 22.352 180)
+    (effects (font (size 1.27 1.27)) (justify right bottom))
+  )
+  (label "Col13" (at 106.68 37.592 180)
     (effects (font (size 1.27 1.27)) (justify right bottom))
   )
@@
     (effects (font (size 1.27 1.27)) (justify right bottom))
   )
-  (label "Row4" (at 108.712 31.75 180)
-    (effects (font (size 1.27 1.27)) (justify right bottom))
-  )
-  (label "Row2" (at 108.712 36.83 180)
-    (effects (font (size 1.27 1.27)) (justify right bottom))
-  )
-  (label "Col15" (at 108.712 46.99 180)
+  (label "Row4" (at 106.68 27.432 180)
+    (effects (font (size 1.27 1.27)) (justify right bottom))
+  )
+  (label "Row2" (at 106.68 32.512 180)
+    (effects (font (size 1.27 1.27)) (justify right bottom))
+  )
+  (label "Col15" (at 106.68 42.672 180)
     (effects (font (size 1.27 1.27)) (justify right bottom))
   )
@@
     (effects (font (size 1.27 1.27)) (justify right bottom))
   )
-  (label "Row1" (at 108.712 39.37 180)
-    (effects (font (size 1.27 1.27)) (justify right bottom))
-  )
-  (label "Col14" (at 108.712 44.45 180)
+  (label "Row1" (at 106.68 35.052 180)
+    (effects (font (size 1.27 1.27)) (justify right bottom))
+  )
+  (label "Col14" (at 106.68 40.132 180)
     (effects (font (size 1.27 1.27)) (justify right bottom))
   )
@@
     (effects (font (size 1.27 1.27)) (justify right bottom))
   )
-  (label "Row3" (at 108.712 34.29 180)
-    (effects (font (size 1.27 1.27)) (justify right bottom))
-  )
-  (label "Row7" (at 108.712 24.13 180)
-    (effects (font (size 1.27 1.27)) (justify right bottom))
-  )
-  (label "Row5" (at 108.712 29.21 180)
+  (label "Row3" (at 106.68 29.972 180)
+    (effects (font (size 1.27 1.27)) (justify right bottom))
+  )
+  (label "Row7" (at 106.68 19.812 180)
+    (effects (font (size 1.27 1.27)) (justify right bottom))
+  )
+  (label "Row5" (at 106.68 24.892 180)
     (effects (font (size 1.27 1.27)) (justify right bottom))
   )
@@
     (pin "2")
   )
-  (symbol (lib_id "5034801000:5034801000") (at 119.888 39.37 0) (unit 1)
-    (in_bom yes) (on_board yes) (fields_autoplaced)
-    (property "Reference" "J1" (id 0) (at 126.746 36.8299 0)
+  (symbol (lib_id "power:GND") (at 105.156 48.768 0) (unit 1)
+    (in_bom yes) (on_board yes) (fields_autoplaced)
+    (property "Reference" "#PWR?" (id 0) (at 105.156 55.118 0)
+      (effects (font (size 1.27 1.27)) hide)
+    )
+    (property "Value" "GND" (id 1) (at 105.156 53.34 0))
+    (property "Footprint" "" (id 2) (at 105.156 48.768 0)
+      (effects (font (size 1.27 1.27)) hide)
+    )
+    (property "Datasheet" "" (id 3) (at 105.156 48.768 0)
+      (effects (font (size 1.27 1.27)) hide)
+    )
+    (pin "1")
+  )
+  (symbol (lib_id "5034801000:5034801000") (at 117.856 35.052 0) (unit 1)
+    (in_bom yes) (on_board yes) (fields_autoplaced)
+    (property "Reference" "J1" (id 0) (at 124.714 32.5119 0)
       (effects (font (size 1.27 1.27)) (justify left))
     )
-    (property "Value" "5034801000" (id 1) (at 126.746 39.3699 0)
+    (property "Value" "5034801000" (id 1) (at 124.714 35.0519 0)
       (effects (font (size 1.27 1.27)) (justify left))
     )
-    (property "Footprint" "5034801000:MOLEX_5034801000" (id 2) (at 119.888 39.37 0)
+    (property "Footprint" "5034801000:MOLEX_5034801000" (id 2) (at 117.856 35.052 0)
       (effects (font (size 1.27 1.27)) (justify left bottom) hide)
     )
-    (property "Datasheet" "" (id 3) (at 119.888 39.37 0)
+    (property "Datasheet" "" (id 3) (at 117.856 35.052 0)
       (effects (font (size 1.27 1.27)) (justify left bottom) hide)
     )
-    (property "MANUFACTURER" "MOLEX" (id 4) (at 119.888 39.37 0)
+    (property "MANUFACTURER" "MOLEX" (id 4) (at 117.856 35.052 0)
       (effects (font (size 1.27 1.27)) (justify left bottom) hide)
     )
-    (property "STANDARD" "Manufacturer Recommendation" (id 5) (at 119.888 39.37 0)
+    (property "STANDARD" "Manufacturer Recommendation" (id 5) (at 117.856 35.052 0)
       (effects (font (size 1.27 1.27)) (justify left bottom) hide)
     )
-    (property "PARTREV" "H" (id 6) (at 119.888 39.37 0)
+    (property "PARTREV" "H" (id 6) (at 117.856 35.052 0)
       (effects (font (size 1.27 1.27)) (justify left bottom) hide)
     )
@@
   )
   (symbol_instances
+    (path "/1c408391-fc59-4ea9-a0d9-3d99d381c04f"
+      (reference "#PWR?") (unit 1) (value "GND") (footprint "")
+    )
     (path "/9d3292e9-89ed-435a-b615-fc52a41b2a3d"
       (reference "D1") (unit 1) (value "D_Small") (footprint "Diode_SMD:D_SOD-123")
