File: KiCAD_PCB/Calculator_Joystick_PCB/Joystick-DPAD/_autosave-Joystick-DPAD.kicad_sch (KiCad schematic)
At the start: 10 parts, among them J1 5034801000, SW1 SW_SPST, SW2 SW_SPST, SW3 SW_SPST, SW4 SW_SPST

Commit message: V2 Updates
Connections:
- net XOUT is gone; now on net x_out: JOY1.X (S)
- net YOUT is gone; now on net y_out: JOY1.Y (S)
- net GND: now also J1.S1 (SHIELD), J1.S2 (SHIELD)
- no-connect marks 0 -> 2
Changed lines of the file:
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@@
   (junction (at 55.118 42.926) (diameter 0) (color 0 0 0 0)
   )
+  (no_connect (at 141.224 44.958))
+  (no_connect (at 141.224 42.418))
   (polyline (pts (xy 116.078 68.326) (xy 116.078 11.938))
     (stroke (width 0) (type default) (color 0 0 0 0))
@@
     (stroke (width 0) (type default) (color 0 0 0 0))
   )
+  (wire (pts (xy 141.224 44.958) (xy 143.764 44.958))
+    (stroke (width 0) (type default) (color 0 0 0 0))
+  )
   (wire (pts (xy 56.134 40.386) (xy 55.118 40.386))
     (stroke (width 0) (type default) (color 0 0 0 0))
@@
     (stroke (width 0) (type default) (color 0 0 0 0))
   )
+  (wire (pts (xy 141.224 50.038) (xy 143.764 50.038))
+    (stroke (width 0) (type default) (color 0 0 0 0))
+  )
   (wire (pts (xy 72.39 18.288) (xy 72.39 40.386))
     (stroke (width 0) (type default) (color 0 0 0 0))
@@
   )
   (polyline (pts (xy 46.482 68.326) (xy 116.078 68.326))
+    (stroke (width 0) (type default) (color 0 0 0 0))
+  )
+  (wire (pts (xy 141.224 42.418) (xy 143.764 42.418))
+    (stroke (width 0) (type default) (color 0 0 0 0))
+  )
+  (wire (pts (xy 141.224 51.054) (xy 141.224 50.038))
     (stroke (width 0) (type default) (color 0 0 0 0))
   )
@@
     (effects (font (size 1.27 1.27)) (justify right bottom))
   )
-  (label "XOUT" (at 36.83 35.052 0)
+  (label "x_out" (at 36.83 35.052 0)
     (effects (font (size 1.2446 1.2446)) (justify left bottom))
   )
@@
     (effects (font (size 1.27 1.27)) (justify right bottom))
   )
-  (label "YOUT" (at 36.83 57.15 0)
+  (label "y_out" (at 36.83 57.15 0)
     (effects (font (size 1.2446 1.2446)) (justify left bottom))
   )
@@
     (pin "S2")
   )
+  (symbol (lib_id "power:GND") (at 141.224 51.054 0) (unit 1)
+    (in_bom yes) (on_board yes) (fields_autoplaced)
+    (property "Reference" "#PWR0101" (id 0) (at 141.224 57.404 0)
+      (effects (font (size 1.27 1.27)) hide)
+    )
+    (property "Value" "GND" (id 1) (at 141.224 55.626 0))
+    (property "Footprint" "" (id 2) (at 141.224 51.054 0)
+      (effects (font (size 1.27 1.27)) hide)
+    )
+    (property "Datasheet" "" (id 3) (at 141.224 51.054 0)
+      (effects (font (size 1.27 1.27)) hide)
+    )
+    (pin "1")
+  )
   (sheet_instances
     (path "/" (page "1"))
@@
       (reference "#GND0102") (unit 1) (value "GND") (footprint "Adafruit Mini Analog Thumbstick:")
     )
+    (path "/fee09553-ca13-4e5a-b7ad-f447e7c207ea"
+      (reference "#PWR0101") (unit 1) (value "GND") (footprint "")
+    )
     (path "/66553eac-3edc-435c-bc67-3973452c2abb"
